File: EAGLE Board Designs/Accumulator Management System/AMS Segment/AMS Segment rev18.sch (EAGLE design)
At the start: 165 parts, among them J1 CONNECTOR-2_MICROFIT_SMD_RIGH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, J10 CONNECTOR-2_MICROFIT_SMD_RIGH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, J100 CONNECTOR-1_5222_, J101 CONNECTOR-1_5222_, J102 CONNECTOR-1_5222_, J103 CONNECTOR-1_5222_, J104 CONNECTOR-1_5222_, J105 CONNECTOR-1_5222_, J106 CONNECTOR-1_5222_, J107 CONNECTOR-1_5222_, J108 CONNECTOR-1_5222_, J109 CONNECTOR-1_5222_, J110 CONNECTOR-1_5222_, J111 CONNECTOR-1_5222_, J112 CONNECTOR-1_5222_, J113 CONNECTOR-1_5222_, J114 CONNECTOR-1_5222_, J115 CONNECTOR-1_5222_, J116 CONNECTOR-1_5222_, J117 CONNECTOR-1_5222_, J118 CONNECTOR-1_5222_, J119 CONNECTOR-1_5222_, J120 CONNECTOR-1_5222_, J121 CONNECTOR-1_5222_, J2 CONNECTOR-2_MICROFIT_SMD_RIGH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, J3 CONNECTOR-2_MICROFIT_SMD_RIGH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, J4 CONNECTOR-2_MICROFIT_SMD_RIGH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, J5 CONNECTOR-2_MICROFIT_SMD_RIGH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, J6 CONNECTOR-2_MICROFIT_SMD_RIGH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, J7 CONNECTOR-2_MICROFIT_SMD_RIGH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, J8 CONNECTOR-2_MICROFIT_SMD_RIGH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, J9 CONNECTOR-2_MICROFIT_SMD_RIGH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, T1 TRANSFORMER_HM2112ZNLT, U1 SHT31-ARP-B, U2 LTC6811-2, U3 LT3990-5, U4 LT3990-5, U5 LTC6811-2, U6 SHT31-ARP-B

Commit message: fixed isospi transformer
Connections:
- net IML: now also T1B.TD-; no longer T1B.TD+
- net IMU: now also T1A.TD-; no longer T1A.TD+
- net IPL: now also T1B.TD+; no longer T1B.TD-
- net IPU: now also T1A.TD+; no longer T1A.TD-
- net N$22: now also T1A.MX-; no longer T1A.MX+
- net N$27: now also T1A.MX+; no longer T1A.MX-
- net N$32: now also T1B.MX-; no longer T1B.MX+
- net N$33: now also T1B.MX+; no longer T1B.MX-
Changed lines of the file:
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@@
 <label x="147.32" y="149.86" size="1.27" layer="95" rot="R180" xref="yes"/>
 <pinref part="C18" gate="G$1" pin="2"/>
-<pinref part="T1" gate="A" pin="TD+"/>
+<pinref part="T1" gate="A" pin="TD-"/>
 <junction x="149.86" y="149.86"/>
 </segment>
@@
 <label x="147.32" y="124.46" size="1.27" layer="95" rot="R180" xref="yes"/>
 <pinref part="C16" gate="G$1" pin="2"/>
-<pinref part="T1" gate="B" pin="TD+"/>
+<pinref part="T1" gate="B" pin="TD-"/>
 <junction x="149.86" y="124.46"/>
 </segment>
@@
 <label x="147.32" y="165.1" size="1.27" layer="95" rot="R180" xref="yes"/>
 <pinref part="R25" gate="G$1" pin="2"/>
-<pinref part="T1" gate="A" pin="TD-"/>
+<pinref part="T1" gate="A" pin="TD+"/>
 <junction x="149.86" y="165.1"/>
 </segment>
@@
 <label x="147.32" y="139.7" size="1.27" layer="95" rot="R180" xref="yes"/>
 <pinref part="R23" gate="G$1" pin="2"/>
-<pinref part="T1" gate="B" pin="TD-"/>
+<pinref part="T1" gate="B" pin="TD+"/>
 <junction x="149.86" y="139.7"/>
 </segment>
@@
 <segment>
 <pinref part="R29" gate="G$1" pin="2"/>
+<pinref part="T1" gate="A" pin="MX-"/>
+<wire x1="198.12" y1="147.32" x2="195.58" y2="147.32" width="0.1524" layer="91"/>
+</segment>
+</net>
+<net name="N$27" class="5">
+<segment>
+<pinref part="R28" gate="G$1" pin="2"/>
 <pinref part="T1" gate="A" pin="MX+"/>
-<wire x1="198.12" y1="147.32" x2="195.58" y2="147.32" width="0.1524" layer="91"/>
-</segment>
-</net>
-<net name="N$27" class="5">
-<segment>
-<pinref part="R28" gate="G$1" pin="2"/>
-<pinref part="T1" gate="A" pin="MX-"/>
 <wire x1="198.12" y1="167.64" x2="195.58" y2="167.64" width="0.1524" layer="91"/>
 </segment>
@@
 <segment>
 <pinref part="R26" gate="G$1" pin="2"/>
+<pinref part="T1" gate="B" pin="MX-"/>
+<wire x1="198.12" y1="121.92" x2="195.58" y2="121.92" width="0.1524" layer="91"/>
+</segment>
+</net>
+<net name="N$33" class="5">
+<segment>
+<pinref part="R24" gate="G$1" pin="2"/>
 <pinref part="T1" gate="B" pin="MX+"/>
-<wire x1="198.12" y1="121.92" x2="195.58" y2="121.92" width="0.1524" layer="91"/>
-</segment>
-</net>
-<net name="N$33" class="5">
-<segment>
-<pinref part="R24" gate="G$1" pin="2"/>
-<pinref part="T1" gate="B" pin="MX-"/>
 <wire x1="198.12" y1="142.24" x2="195.58" y2="142.24" width="0.1524" layer="91"/>
 </segment>
