File: EAGLE Board Designs/Accumulator Management System/AMS Segment/AMS Segment rev19.brd (EAGLE design)
At the start: 275.2 x 86 mm, 347 parts, among them J1 CONNECTOR-2_MICROFIT_SMD_RIGH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, J10 CONNECTOR-2_MICROFIT_SMD_RIGH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, J100 CONNECTOR-1_5222_, J101 CONNECTOR-1_5222_, J102 CONNECTOR-1_5222_, J103 CONNECTOR-1_5222_, J104 CONNECTOR-1_5222_, J105 CONNECTOR-1_5222_, J106 CONNECTOR-1_5222_, J107 CONNECTOR-1_5222_, J108 CONNECTOR-1_5222_, J109 CONNECTOR-1_5222_, J110 CONNECTOR-1_5222_, J111 CONNECTOR-1_5222_, J112 CONNECTOR-1_5222_, J113 CONNECTOR-1_5222_, J114 CONNECTOR-1_5222_, J115 CONNECTOR-1_5222_, J116 CONNECTOR-1_5222_, J117 CONNECTOR-1_5222_, J118 CONNECTOR-1_5222_, J119 CONNECTOR-1_5222_, J120 CONNECTOR-1_5222_, J121 CONNECTOR-1_5222_, J2 CONNECTOR-2_MICROFIT_SMD_RIGH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, J3 CONNECTOR-2_MICROFIT_SMD_RIGH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, J4 CONNECTOR-2_MICROFIT_SMD_RIGH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, J5 CONNECTOR-2_MICROFIT_SMD_RIGH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, J6 CONNECTOR-2_MICROFIT_SMD_RIGH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, J7 CONNECTOR-2_MICROFIT_SMD_RIGH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, J8 CONNECTOR-2_MICROFIT_SMD_RIGH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, J9 CONNECTOR-2_MICROFIT_SMD_RIGH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, T1 TRANSFORMER_HM2112ZNLT, U1 SHT31-ARP-B, U2 LTC6811-2, U3 LT3990-5, U4 LT3990-5, U5 LTC6811-2, U6 SHT31-ARP-B

Commit message: Rerouted IsoSPI
Rerouted IsoSPI
Parts:
- moved C23 25.2 mm to (78.6, -59.5), turned to 270 degrees
- moved C25 25.0 mm to (88.9, -36.6), turned to 180 degrees
- moved TP6 18.2 mm to (135.1, -76.7), turned to 0 degrees
- moved TP5 17.2 mm to (139.6, -76.0), turned to 270 degrees
- moved R27 3.87 mm to (135.3, -73.8)
- moved C26 0.76 mm to (77.0, -59.6)
- moved C27 0.76 mm to (75.3, -59.6)
- moved C28 0.76 mm to (73.4, -59.6)
- moved R47 0.76 mm to (71.8, -59.6)
Routing:
- net IM: track 47.9 -> 34.1 mm, vias 2 -> 0
- net IPU: track 61.4 -> 65.5 mm
- net IP: track 40.0 -> 36.6 mm
- net VREGU: track 306.1 -> 304.7 mm
- net IMU: track 67.1 -> 68.1 mm
- net VREF1U: track 3.12 -> 2.28 mm
- net C0U: track 4.29 -> 3.53 mm
- net GPIO4L: track 75.8 -> 75.3 mm
