File: EAGLE Board Designs/Discharge Board/Discharge Board.sch (EAGLE design)
At the start: 7 parts, among them J1 CONNECTOR-2_MICROFIT_SMD_RIGH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, J2 CONNECTOR-2_MICROFIT_SMD_RIGH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, K1 RELAY_SPST_NC_POLARIZED_D_24

Commit message: minor tweaks
Parts:
- renumbered J1 to J101, J2 to J100, R6 to R1, R7 to R2, R8 to R3
Changed lines of the file:
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@@
 <part name="P2" library="HyTechSupplies" deviceset="GND" device=""/>
 <part name="P12" library="HyTechSupplies" deviceset="TS-UNFUSED" device=""/>
-<part name="R6" library="HyTechDevices" deviceset="RESISTOR_?_*" device="B20" technology="15K"/>
-<part name="R7" library="HyTechDevices" deviceset="RESISTOR_?_*" device="B20" technology="15K"/>
-<part name="R8" library="HyTechDevices" deviceset="RESISTOR_?_*" device="B20" technology="15K"/>
+<part name="R1" library="HyTechDevices" deviceset="RESISTOR_?_*" device="B20" technology="15K"/>
+<part name="R2" library="HyTechDevices" deviceset="RESISTOR_?_*" device="B20" technology="15K"/>
+<part name="R3" library="HyTechDevices" deviceset="RESISTOR_?_*" device="B20" technology="15K"/>
 <part name="K1" library="HyTechDevices" deviceset="RELAY_SPST_NC_POLARIZED_?*" device="D_" technology="24"/>
-<part name="J2" library="HyTechDevices" deviceset="CONNECTOR-2_?_*" device="MICROFIT_SMD_RIGHTANGLE_02_SINGLE" technology="BLACK"/>
-<part name="J1" library="HyTechDevices" deviceset="CONNECTOR-2_?_*" device="MICROFIT_SMD_RIGHTANGLE_02_SINGLE" technology="BLACK"/>
+<part name="J100" library="HyTechDevices" deviceset="CONNECTOR-2_?_*" device="MICROFIT_SMD_RIGHTANGLE_02_SINGLE" technology="BLACK"/>
+<part name="J101" library="HyTechDevices" deviceset="CONNECTOR-2_?_*" device="MICROFIT_SMD_RIGHTANGLE_02_SINGLE" technology="BLACK"/>
+<part name="FRAME1" library="HyTechFrames" deviceset="FRAME" device=""/>
 </parts>
 <sheets>
@@
 <attribute name="VALUE" x="48.26" y="7.62" size="1.27" layer="96" align="top-center"/>
 </instance>
-<instance part="R6" gate="G$1" x="40.64" y="17.78" smashed="yes" rot="R90">
+<instance part="R1" gate="G$1" x="40.64" y="17.78" smashed="yes" rot="R90">
 <attribute name="NAME" x="39.37" y="16.51" size="1.27" layer="95" rot="R90" align="bottom-center"/>
 <attribute name="RESISTANCE" x="41.91" y="16.51" size="1.27" layer="96" rot="R90" align="top-center"/>
 </instance>
-<instance part="R7" gate="G$1" x="35.56" y="17.78" smashed="yes" rot="R90">
+<instance part="R2" gate="G$1" x="35.56" y="17.78" smashed="yes" rot="R90">
 <attribute name="NAME" x="34.29" y="16.51" size="1.27" layer="95" rot="R90" align="bottom-center"/>
 <attribute name="RESISTANCE" x="36.83" y="16.51" size="1.27" layer="96" rot="R90" align="top-center"/>
 </instance>
-<instance part="R8" gate="G$1" x="30.48" y="17.78" smashed="yes" rot="R90">
+<instance part="R3" gate="G$1" x="30.48" y="17.78" smashed="yes" rot="R90">
 <attribute name="NAME" x="29.21" y="16.51" size="1.27" layer="95" rot="R90" align="bottom-center"/>
 <attribute name="RESISTANCE" x="31.75" y="16.51" size="1.27" layer="96" rot="R90" align="top-center"/>
@@
 <attribute name="NAME" x="14.478" y="35.56" size="1.27" layer="95" rot="MR270"/>
 </instance>
-<instance part="J2" gate="G$1" x="66.04" y="30.48" smashed="yes" rot="R180">
+<instance part="J100" gate="G$1" x="66.04" y="30.48" smashed="yes" rot="R180">
 <attribute name="MPN" x="66.04" y="38.735" size="1.27" layer="96" rot="R180" align="top-left"/>
 <attribute name="NAME" x="66.04" y="29.718" size="1.27" layer="95" rot="R180"/>
 </instance>
-<instance part="J1" gate="G$1" x="-12.7" y="35.56" smashed="yes">
+<instance part="J101" gate="G$1" x="-12.7" y="35.56" smashed="yes">
 <attribute name="MPN" x="-12.7" y="27.305" size="1.27" layer="96" align="top-left"/>
 <attribute name="NAME" x="-12.7" y="36.322" size="1.27" layer="95"/>
+</instance>
+<instance part="FRAME1" gate="O" x="-101.6" y="-114.3" smashed="yes">
+<attribute name="LAST_DATE_TIME" x="85.09" y="-111.76" size="2.54" layer="95"/>
+<attribute name="DRAWING_NAME" x="105.41" y="-91.44" size="2.54" layer="95"/>
+<attribute name="SHEET" x="157.48" y="-111.76" size="2.54" layer="95"/>
+<attribute name="ENGINEER" x="27.94" y="-91.44" size="2.54" layer="95"/>
+<attribute name="DESIGNER_SCHEMATIC" x="74.93" y="-68.58" size="2.54" layer="95"/>
+<attribute name="DESIGNER_BOARD" x="74.93" y="-76.2" size="2.54" layer="95"/>
+<attribute name="DESIGNER_FURTHER" x="74.93" y="-83.82" size="2.54" layer="95"/>
+<attribute name="REVIEWER_SCHEMATIC" x="125.73" y="-68.58" size="2.54" layer="95"/>
+<attribute name="REVIEWER_BOARD" x="125.73" y="-76.2" size="2.54" layer="95"/>
+<attribute name="REVIEWER_FURTHER" x="125.73" y="-83.82" size="2.54" layer="95"/>
+<attribute name="DESCRIPTION_1" x="95.25" y="-99.06" size="2.54" layer="95"/>
+<attribute name="DESCRIPTION_2" x="74.93" y="-104.14" size="2.54" layer="95"/>
 </instance>
 </instances>
@@
 <junction x="22.86" y="20.32"/>
 <pinref part="K1" gate="G$1" pin="COIL-"/>
-<pinref part="J1" gate="G$1" pin="2"/>
+<pinref part="J101" gate="G$1" pin="2"/>
 <wire x1="-2.54" y1="30.48" x2="-2.54" y2="12.7" width="0.1524" layer="91"/>
 <wire x1="-2.54" y1="12.7" x2="22.86" y2="12.7" width="0.1524" layer="91"/>
@@
 <wire x1="22.86" y1="40.64" x2="22.86" y2="45.72" width="0.1524" layer="91"/>
 <pinref part="K1" gate="G$1" pin="COIL+"/>
-<pinref part="J1" gate="G$1" pin="1"/>
+<pinref part="J101" gate="G$1" pin="1"/>
 <wire x1="-2.54" y1="33.02" x2="-2.54" y2="45.72" width="0.1524" layer="91"/>
 <wire x1="-2.54" y1="45.72" x2="22.86" y2="45.72" width="0.1524" layer="91"/>
@@
 <wire x1="33.02" y1="43.18" x2="33.02" y2="38.1" width="0.6096" layer="91"/>
 <pinref part="K1" gate="G$1" pin="CONTACT1"/>
-<pinref part="J2" gate="G$1" pin="2"/>
+<pinref part="J100" gate="G$1" pin="2"/>
 <wire x1="55.88" y1="35.56" x2="55.88" y2="43.18" width="0.6096" layer="91"/>
 <wire x1="55.88" y1="43.18" x2="33.02" y2="43.18" width="0.6096" layer="91"/>
@@
 <segment>
 <wire x1="35.56" y1="22.86" x2="35.56" y2="20.32" width="0.6096" layer="91"/>
-<pinref part="R7" gate="G$1" pin="2"/>
-<pinref part="R8" gate="G$1" pin="2"/>
+<pinref part="R2" gate="G$1" pin="2"/>
+<pinref part="R3" gate="G$1" pin="2"/>
 <wire x1="30.48" y1="20.32" x2="35.56" y2="20.32" width="0.6096" layer="91"/>
 <junction x="35.56" y="20.32"/>
-<pinref part="R6" gate="G$1" pin="2"/>
+<pinref part="R1" gate="G$1" pin="2"/>
 <wire x1="35.56" y1="20.32" x2="40.64" y2="20.32" width="0.6096" layer="91"/>
 <pinref part="K1" gate="G$1" pin="CONTACT2"/>
@@
 <net name="N$5" class="0">
 <segment>
-<pinref part="R6" gate="G$1" pin="1"/>
-<pinref part="R7" gate="G$1" pin="1"/>
+<pinref part="R1" gate="G$1" pin="1"/>
+<pinref part="R2" gate="G$1" pin="1"/>
 <wire x1="35.56" y1="12.7" x2="40.64" y2="12.7" width="0.6096" layer="91"/>
 <junction x="35.56" y="12.7"/>
-<pinref part="R8" gate="G$1" pin="1"/>
+<pinref part="R3" gate="G$1" pin="1"/>
 <wire x1="30.48" y1="12.7" x2="35.56" y2="12.7" width="0.6096" layer="91"/>
 <pinref part="P12" gate="G$1" pin="TS-UNFUSED"/>
 <wire x1="40.64" y1="12.7" x2="48.26" y2="12.7" width="0.6096" layer="91"/>
-<pinref part="J2" gate="G$1" pin="1"/>
+<pinref part="J100" gate="G$1" pin="1"/>
 <wire x1="55.88" y1="33.02" x2="55.88" y2="12.7" width="0.6096" layer="91"/>
 <wire x1="55.88" y1="12.7" x2="48.26" y2="12.7" width="0.6096" layer="91"/>

Commit message: Replace B20 with B20-SHORTENED
Parts:
- R1, R2, R3: value RESISTOR_B20_15K -> RESISTOR_B20-SHORTENED_15K; device HyTechDevices:RESISTOR_B20_15K -> HyTechDevices:RESISTOR_B20-SHORTENED_15K
Changed lines of the file:
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@@
 <part name="P2" library="HyTechSupplies" deviceset="GND" device=""/>
 <part name="P12" library="HyTechSupplies" deviceset="TS-UNFUSED" device=""/>
-<part name="R1" library="HyTechDevices" deviceset="RESISTOR_?_*" device="B20" technology="15K"/>
-<part name="R2" library="HyTechDevices" deviceset="RESISTOR_?_*" device="B20" technology="15K"/>
-<part name="R3" library="HyTechDevices" deviceset="RESISTOR_?_*" device="B20" technology="15K"/>
+<part name="R1" library="HyTechDevices" deviceset="RESISTOR_?_*" device="B20-SHORTENED" technology="15K" value="RESISTOR_B20-SHORTENED_15K"/>
+<part name="R2" library="HyTechDevices" deviceset="RESISTOR_?_*" device="B20-SHORTENED" technology="15K" value="RESISTOR_B20-SHORTENED_15K"/>
+<part name="R3" library="HyTechDevices" deviceset="RESISTOR_?_*" device="B20-SHORTENED" technology="15K" value="RESISTOR_B20-SHORTENED_15K"/>
 <part name="K1" library="HyTechDevices" deviceset="RELAY_SPST_NC_POLARIZED_?*" device="D_" technology="24"/>
 <part name="J100" library="HyTechDevices" deviceset="CONNECTOR-2_?_*" device="MICROFIT_SMD_RIGHTANGLE_02_SINGLE" technology="BLACK"/>
