File: EAGLE Board Designs/Discharge Board/Discharge Board rev2.sch (EAGLE design)
At the start: 9 parts, among them J100 CONNECTOR-5_MICRO_VS_, J101 CONNECTOR-2_MICROFIT_SMD_RIGH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, K1 RELAY_SPST_NC_POLARIZED_D_24

Commit message: replaced 5-pin connector with new right angle
Parts:
- J100: value CONNECTOR-5_MICRO_VS_ -> CONNECTOR-5_MICRO_R5S_; device HyTechDevices:CONNECTOR-5_MICRO_VS_ -> HyTechDevices:CONNECTOR-5_MICRO_R5S_
Changed lines of the file:
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@@
 <part name="R3" library="HyTechDevices" deviceset="RESISTOR_?_*" device="B20-SHORTENED" technology="15K" value="RESISTOR_B20-SHORTENED_15K"/>
 <part name="K1" library="HyTechDevices" deviceset="RELAY_SPST_NC_POLARIZED_?*" device="D_" technology="24"/>
-<part name="J100" library="HyTechDevices" deviceset="CONNECTOR-5_?_*" device="MICRO_VS"/>
+<part name="J100" library="HyTechDevices" deviceset="CONNECTOR-5_?_*" device="MICRO_R5S" value="CONNECTOR-5_MICRO_R5S_"/>
 <part name="J101" library="HyTechDevices" deviceset="CONNECTOR-2_?_*" device="MICROFIT_SMD_RIGHTANGLE_02_SINGLE" technology="BLACK"/>
 <part name="FRAME1" library="HyTechFrames" deviceset="FRAME" device="">
