File: EAGLE Board Designs/Accumulator Management System/AMS Test Board/AMS Test Board rev2.brd (EAGLE design)
At the start: 386.6 x 87.7 mm, 104 parts, among them J1 CONNECTOR-2__B2B-PH-K, J10 CONNECTOR-2__B2B-PH-K, J11 CONNECTOR-2__B2B-PH-K, J12 CONNECTOR-2__B2B-PH-K, J13 CONNECTOR-2__B2B-PH-K, J14 CONNECTOR-2__B2B-PH-K, J15 CONNECTOR-2__B2B-PH-K, J16 CONNECTOR-2__B2B-PH-K, J17 CONNECTOR-2__B2B-PH-K, J18 CONNECTOR-2__B2B-PH-K, J19 CONNECTOR-2__B2B-PH-K, J2 CONNECTOR-2__B2B-PH-K, J20 CONNECTOR-2__B2B-PH-K, J21 CONNECTOR-2__B2B-PH-K, J22 CONNECTOR-1_5222, J23 CONNECTOR-1_5222, J24 CONNECTOR-1_5222, J25 CONNECTOR-1_5222, J26 CONNECTOR-1_5222, J27 CONNECTOR-1_5222, J28 CONNECTOR-1_5222, J29 CONNECTOR-1_5222, J3 CONNECTOR-2__B2B-PH-K, J30 CONNECTOR-1_5222, J31 CONNECTOR-1_5222, J32 CONNECTOR-1_5222, J33 CONNECTOR-1_5222, J34 CONNECTOR-1_5222, J35 CONNECTOR-1_5222, J36 CONNECTOR-1_5222, J37 CONNECTOR-1_5222, J38 CONNECTOR-1_5222, J39 CONNECTOR-1_5222, J4 CONNECTOR-2__B2B-PH-K, J40 CONNECTOR-1_5222, J41 CONNECTOR-1_5222, J42 CONNECTOR-1_5222, J43 CONNECTOR-1_5222, J44 CONNECTOR-2_MF_T_V_, J5 CONNECTOR-2__B2B-PH-K, J6 CONNECTOR-2__B2B-PH-K, J7 CONNECTOR-2__B2B-PH-K, J8 CONNECTOR-2__B2B-PH-K, J9 CONNECTOR-2__B2B-PH-K, T1 TRANSFORMER_HM2112ZNLT_AIRGAP, U1 LTC6820

Commit message: AMS Test Board rev2 Completed
Parts:
- removed U$6: (no value), HyTechManufacturing:HV_LARGE
- moved U$14 52.1 mm to (267.8, 5.21)
- moved U$17 24.2 mm to (383.5, 58.9)
- moved R1 19.8 mm to (341.6, 13.0), turned to 0 degrees
- moved R2 8.98 mm to (357.4, 16.4)
- moved C1 8.46 mm to (353.1, 34.2), turned to 90 degrees
- moved R25 7.71 mm to (357.5, 18.8)
- moved R33 7.24 mm to (363.1, 20.4), turned to 270 degrees
- moved TD- 7.24 mm to (338.6, 16.6)
- moved R32 7.23 mm to (365.5, 20.4), turned to 270 degrees
- moved TD+ 7.11 mm to (345.7, 16.6)
- moved C5 6.23 mm to (359.9, 29.1)
- moved C6 4.87 mm to (359.9, 26.8)
- moved U$19 2.54 mm to (340.6, 78.1)
Routing:
- net IP: track 118.5 -> 15.7 mm, vias 0 -> 2
- net N$26: track 143.8 -> 50.7 mm
- net N$25: track 118.0 -> 35.8 mm
- net TD-: track 94.1 -> 39.2 mm
- net TD+: track 88.7 -> 52.7 mm
- net N$31: track 27.4 -> 6.78 mm
- net +3V3: track 49.2 -> 36.3 mm
- net N$30: track 13.5 -> 2.49 mm
- net N$23: track 12.4 -> 3.79 mm
- net N$27: track 42.3 -> 44.1 mm
- net 19-: track 140.0 -> 141.2 mm
- net 11-: track 282.7 -> 283.8 mm
- net 9-: track 332.4 -> 333.5 mm
- net 1-: track 360.1 -> 361.2 mm
- net 7-: track 358.8 -> 359.9 mm
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