File: EAGLE Board Designs/Accumulator Management System/AMS Test Board/AMS Test Board rev3.brd (EAGLE design)
At the start: 386.6 x 87.7 mm, 103 parts, among them J1 CONNECTOR-2__B2B-PH-K, J10 CONNECTOR-2__B2B-PH-K, J11 CONNECTOR-2__B2B-PH-K, J12 CONNECTOR-2__B2B-PH-K, J13 CONNECTOR-2__B2B-PH-K, J14 CONNECTOR-2__B2B-PH-K, J15 CONNECTOR-2__B2B-PH-K, J16 CONNECTOR-2__B2B-PH-K, J17 CONNECTOR-2__B2B-PH-K, J18 CONNECTOR-2__B2B-PH-K, J19 CONNECTOR-2__B2B-PH-K, J2 CONNECTOR-2__B2B-PH-K, J20 CONNECTOR-2__B2B-PH-K, J21 CONNECTOR-2__B2B-PH-K, J22 CONNECTOR-1_5222, J23 CONNECTOR-1_5222, J24 CONNECTOR-1_5222, J25 CONNECTOR-1_5222, J26 CONNECTOR-1_5222, J27 CONNECTOR-1_5222, J28 CONNECTOR-1_5222, J29 CONNECTOR-1_5222, J3 CONNECTOR-2__B2B-PH-K, J30 CONNECTOR-1_5222, J31 CONNECTOR-1_5222, J32 CONNECTOR-1_5222, J33 CONNECTOR-1_5222, J34 CONNECTOR-1_5222, J35 CONNECTOR-1_5222, J36 CONNECTOR-1_5222, J37 CONNECTOR-1_5222, J38 CONNECTOR-1_5222, J39 CONNECTOR-1_5222, J4 CONNECTOR-2__B2B-PH-K, J40 CONNECTOR-1_5222, J41 CONNECTOR-1_5222, J42 CONNECTOR-1_5222, J43 CONNECTOR-1_5222, J44 CONNECTOR-2_MF_T_V_, J5 CONNECTOR-2__B2B-PH-K, J6 CONNECTOR-2__B2B-PH-K, J7 CONNECTOR-2__B2B-PH-K, J8 CONNECTOR-2__B2B-PH-K, J9 CONNECTOR-2__B2B-PH-K, T1 TRANSFORMER_HM2112ZNLT_AIRGAP, U1 LTC6820

Commit message: quick update
Routing:
- net GND: track 8.70 -> 11.0 mm, vias 4 -> 5
Changed lines of the file:
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@@
 <?xml version="1.0" encoding="utf-8"?>
 <!DOCTYPE eagle SYSTEM "eagle.dtd">
-<eagle version="7.7.0">
+<eagle version="9.6.2">
 <drawing>
 <settings>
 <setting alwaysvectorfont="no"/>
+<setting keepoldvectorfont="yes"/>
 <setting verticaltext="up"/>
 </settings>
@@
 <contactref element="A1" pad="AGND/GND"/>
 <contactref element="C6" pad="1"/>
-<contactref element="C5" pad="2"/>
-<contactref element="C1" pad="2"/>
-<contactref element="R2" pad="2"/>
 <polygon width="0.1524" layer="16">
 <vertex x="332.74" y="41.91"/>
@@
 <vertex x="386.08" y="41.91"/>
 </polygon>
-<wire x1="356.528" y1="16.383" x2="354.457" y2="16.383" width="0.254" layer="1"/>
-<via x="354.457" y="16.383" extent="1-16" drill="0.381"/>
 <wire x1="359.168" y1="26.797" x2="356.997" y2="26.797" width="0.254" layer="1"/>
 <via x="356.997" y="26.797" extent="1-16" drill="0.381"/>
-<wire x1="359.168" y1="29.083" x2="356.997" y2="29.083" width="0.254" layer="1"/>
-<via x="356.997" y="29.083" extent="1-16" drill="0.381"/>
-<wire x1="353.06" y1="36.703" x2="353.06" y2="34.913" width="0.254" layer="1"/>
-<via x="353.06" y="36.703" extent="1-16" drill="0.381"/>
 <contactref element="U1" pad="13"/>
 <contactref element="U1" pad="14"/>
 <wire x1="356.5425" y1="22.237" x2="356.5425" y2="22.737" width="0.254" layer="1"/>
-<wire x1="356.997" y1="29.083" x2="353.06" y2="34.913" width="0" layer="19" extent="1-1"/>
-<wire x1="359.168" y1="26.797" x2="359.168" y2="29.083" width="0" layer="19" extent="1-1"/>
-<wire x1="356.5425" y1="22.737" x2="356.997" y2="26.797" width="0" layer="19" extent="1-1"/>
-<wire x1="356.528" y1="16.383" x2="356.5425" y2="22.237" width="0" layer="19" extent="1-1"/>
-<wire x1="368.046" y1="6.35" x2="356.528" y2="16.383" width="0" layer="19" extent="1-1"/>
-<wire x1="383.286" y1="3.81" x2="368.046" y2="6.35" width="0" layer="19" extent="1-1"/>
+<contactref element="C1" pad="2"/>
+<contactref element="R2" pad="2"/>
+<contactref element="C5" pad="2"/>
+<wire x1="356.5425" y1="22.237" x2="354.85" y2="22.237" width="0.254" layer="1"/>
+<wire x1="354.85" y1="22.237" x2="354.838" y2="22.225" width="0.254" layer="1"/>
+<wire x1="354.838" y1="22.225" x2="354.457" y2="22.225" width="0.254" layer="1"/>
+<via x="354.457" y="22.225" extent="1-16" drill="0.3556"/>
+<wire x1="359.168" y1="29.083" x2="356.997" y2="29.083" width="0.254" layer="1"/>
+<via x="356.997" y="29.083" extent="1-16" drill="0.3556"/>
+<wire x1="353.06" y1="34.913" x2="355.207" y2="34.913" width="0.254" layer="1"/>
+<wire x1="355.207" y1="34.913" x2="355.219" y2="34.925" width="0.254" layer="1"/>
+<via x="355.219" y="34.925" extent="1-16" drill="0.3556"/>
+<wire x1="356.528" y1="16.383" x2="354.584" y2="16.383" width="0.254" layer="1"/>
+<via x="354.584" y="16.383" extent="1-16" drill="0.3556"/>
 </signal>
 <signal name="N$23">

Commit message: Quick update
Parts:
- moved TD+ 7.62 mm to (338.1, 16.6)
- moved TD- 7.62 mm to (346.2, 16.6)
Routing:
- net TD-: track 39.2 -> 57.8 mm
- net TD+: track 52.7 -> 53.6 mm
Other:
- board text added: "AMS Test Board Rev 3 HyTech Racing 2023 Designed by Ethan Su"
- board text removed: "AMS Test Board Rev 2 HyTech Racing 2023 Designed by Ethan Su"
Changed lines of the file:
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@@
 <wire x1="49.0982" y1="87.5284" x2="49.0982" y2="-0.1016" width="0.508" layer="21"/>
 <wire x1="331.8256" y1="87.5284" x2="331.8256" y2="-0.1016" width="0.508" layer="21"/>
-<text x="340.741" y="68.453" size="1.778" layer="21">AMS Test Board Rev 2
+<text x="340.741" y="68.453" size="1.778" layer="21">AMS Test Board Rev 3
 HyTech Racing 2023
 Designed by Ethan Su</text>
@@
 <attribute name="NAME" x="341.63" y="10.287" size="0.8128" layer="25" align="bottom-center"/>
 </element>
-<element name="TD-" library="HyTechDevices - Copy" package="MICRO_MINIATURE" value="TEST_POINT" x="338.582" y="16.637" smashed="yes">
-<attribute name="DKPN" value="36-5015CT-ND" x="338.582" y="16.637" size="1.778" layer="27" display="off"/>
-<attribute name="MANUFACTURER" value="Keystone Electronics" x="338.582" y="16.637" size="1.778" layer="27" display="off"/>
-<attribute name="MOPN" value="534-5015" x="338.582" y="16.637" size="1.778" layer="27" display="off"/>
-<attribute name="MPN" value="5015" x="338.582" y="16.637" size="1.778" layer="27" display="off"/>
-<attribute name="NAME" x="338.582" y="17.907" size="0.8128" layer="25" font="vector" align="bottom-center"/>
-</element>
-<element name="TD+" library="HyTechDevices - Copy" package="MICRO_MINIATURE" value="TEST_POINT" x="345.694" y="16.637" smashed="yes">
-<attribute name="DKPN" value="36-5015CT-ND" x="345.694" y="16.637" size="1.778" layer="27" display="off"/>
-<attribute name="MANUFACTURER" value="Keystone Electronics" x="345.694" y="16.637" size="1.778" layer="27" display="off"/>
-<attribute name="MOPN" value="534-5015" x="345.694" y="16.637" size="1.778" layer="27" display="off"/>
-<attribute name="MPN" value="5015" x="345.694" y="16.637" size="1.778" layer="27" display="off"/>
-<attribute name="NAME" x="345.694" y="17.907" size="0.8128" layer="25" font="vector" align="bottom-center"/>
+<element name="TD-" library="HyTechDevices - Copy" package="MICRO_MINIATURE" value="TEST_POINT" x="346.202" y="16.637" smashed="yes">
+<attribute name="DKPN" value="36-5015CT-ND" x="346.202" y="16.637" size="1.778" layer="27" display="off"/>
+<attribute name="MANUFACTURER" value="Keystone Electronics" x="346.202" y="16.637" size="1.778" layer="27" display="off"/>
+<attribute name="MOPN" value="534-5015" x="346.202" y="16.637" size="1.778" layer="27" display="off"/>
+<attribute name="MPN" value="5015" x="346.202" y="16.637" size="1.778" layer="27" display="off"/>
+<attribute name="NAME" x="346.202" y="17.907" size="0.8128" layer="25" font="vector" align="bottom-center"/>
+</element>
+<element name="TD+" library="HyTechDevices - Copy" package="MICRO_MINIATURE" value="TEST_POINT" x="338.074" y="16.637" smashed="yes">
+<attribute name="DKPN" value="36-5015CT-ND" x="338.074" y="16.637" size="1.778" layer="27" display="off"/>
+<attribute name="MANUFACTURER" value="Keystone Electronics" x="338.074" y="16.637" size="1.778" layer="27" display="off"/>
+<attribute name="MOPN" value="534-5015" x="338.074" y="16.637" size="1.778" layer="27" display="off"/>
+<attribute name="MPN" value="5015" x="338.074" y="16.637" size="1.778" layer="27" display="off"/>
+<attribute name="NAME" x="338.074" y="17.907" size="0.8128" layer="25" font="vector" align="bottom-center"/>
 </element>
 <element name="R1" library="HyTechDevices" package="0603-RES" value="RESISTOR_0603_120" x="341.63" y="12.954" smashed="yes">
@@
 <wire x1="343.1286" y1="6.3754" x2="340.741" y2="8.763" width="0.254" layer="1"/>
 <wire x1="340.741" y1="8.763" x2="333.413" y2="16.091" width="0.254" layer="1"/>
-<wire x1="338.582" y1="16.637" x2="340.78" y2="14.439" width="0.254" layer="1"/>
-<wire x1="340.78" y1="14.439" x2="340.78" y2="12.954" width="0.254" layer="1"/>
 <wire x1="340.78" y1="12.954" x2="340.78" y2="8.802" width="0.254" layer="1"/>
 <wire x1="340.78" y1="8.802" x2="340.741" y2="8.763" width="0.254" layer="1"/>
 <wire x1="334.993" y1="31.479996875" x2="334.035784375" y2="31.479996875" width="0.254" layer="1"/>
+<wire x1="340.78" y1="12.954" x2="339.764" y2="13.97" width="0.254" layer="1"/>
+<wire x1="334.01" y1="16.51" x2="334.01" y2="17.78" width="0.254" layer="1"/>
+<wire x1="334.01" y1="17.78" x2="335.28" y2="19.05" width="0.254" layer="1"/>
+<wire x1="343.789" y1="19.05" x2="346.202" y2="16.637" width="0.254" layer="1"/>
+<wire x1="339.764" y1="13.97" x2="336.55" y2="13.97" width="0.254" layer="1"/>
+<wire x1="336.55" y1="13.97" x2="334.01" y2="16.51" width="0.254" layer="1"/>
+<wire x1="335.28" y1="19.05" x2="343.789" y2="19.05" width="0.254" layer="1"/>
 </signal>
 <signal name="TD+">
@@
 <wire x1="332.867" y1="15.7474" x2="332.867" y2="34.11651875" width="0.254" layer="1"/>
 <wire x1="340.1314" y1="6.223" x2="340.1314" y2="6.35" width="0.254" layer="1"/>
-<wire x1="345.694" y1="16.637" x2="342.48" y2="13.423" width="0.254" layer="1"/>
-<wire x1="342.48" y1="13.423" x2="342.48" y2="12.954" width="0.254" layer="1"/>
 <wire x1="342.48" y1="12.954" x2="344.678" y2="10.756" width="0.254" layer="1"/>
 <wire x1="344.678" y1="10.756" x2="344.678" y2="5.207" width="0.254" layer="1"/>
@@
 <wire x1="341.7824" y1="4.572" x2="340.1314" y2="6.223" width="0.254" layer="1"/>
 <wire x1="344.043" y1="4.572" x2="341.7824" y2="4.572" width="0.254" layer="1"/>
+<wire x1="342.48" y1="12.954" x2="338.797" y2="16.637" width="0.254" layer="1"/>
+<wire x1="338.797" y1="16.637" x2="338.074" y2="16.637" width="0.254" layer="1"/>
 </signal>
 <signal name="N$30">
