File: EAGLE Board Designs/Accumulator Management System/AMS Test Board/AMS Test Board/AMS Test Board rev1.brd (EAGLE design)
At the start: 386.6 x 87.7 mm, 53 parts, among them J1 CONNECTOR-2__B2B-PH-K, J10 CONNECTOR-2__B2B-PH-K, J11 CONNECTOR-2__B2B-PH-K, J12 CONNECTOR-2__B2B-PH-K, J13 CONNECTOR-2__B2B-PH-K, J14 CONNECTOR-2__B2B-PH-K, J15 CONNECTOR-2__B2B-PH-K, J16 CONNECTOR-2__B2B-PH-K, J17 CONNECTOR-2__B2B-PH-K, J18 CONNECTOR-2__B2B-PH-K, J19 CONNECTOR-2__B2B-PH-K, J2 CONNECTOR-2__B2B-PH-K, J20 CONNECTOR-2__B2B-PH-K, J21 CONNECTOR-2__B2B-PH-K, J22 CONNECTOR-1_5222, J23 CONNECTOR-1_5222, J24 CONNECTOR-1_5222, J25 CONNECTOR-1_5222, J26 CONNECTOR-1_5222, J27 CONNECTOR-1_5222, J28 CONNECTOR-1_5222, J29 CONNECTOR-1_5222, J3 CONNECTOR-2__B2B-PH-K, J30 CONNECTOR-1_5222, J31 CONNECTOR-1_5222, J32 CONNECTOR-1_5222, J33 CONNECTOR-1_5222, J34 CONNECTOR-1_5222, J35 CONNECTOR-1_5222, J36 CONNECTOR-1_5222, J37 CONNECTOR-1_5222, J38 CONNECTOR-1_5222, J39 CONNECTOR-1_5222, J4 CONNECTOR-2__B2B-PH-K, J40 CONNECTOR-1_5222, J41 CONNECTOR-1_5222, J42 CONNECTOR-1_5222, J43 CONNECTOR-1_5222, J5 CONNECTOR-2__B2B-PH-K, J6 CONNECTOR-2__B2B-PH-K, J7 CONNECTOR-2__B2B-PH-K, J8 CONNECTOR-2__B2B-PH-K, J9 CONNECTOR-2__B2B-PH-K

Commit message: Drafted AMS Test Board
Routed all 21 battery connectors on left side (no fuses).
Parts:
- moved J18 121.8 mm to (36.8, 43.2), turned to 180 degrees
- moved J17 116.3 mm to (36.8, 34.3), turned to 180 degrees
- moved J16 111.9 mm to (36.8, 25.4), turned to 180 degrees
- moved J15 108.8 mm to (36.8, 16.5), turned to 180 degrees
- moved J10 104.4 mm to (22.9, 52.1), turned to 180 degrees
- moved J9 94.4 mm to (22.9, 61.0), turned to 180 degrees
- moved J14 90.8 mm to (22.9, 16.5), turned to 180 degrees
- moved J2 90.8 mm to (8.89, 25.4), turned to 180 degrees
- moved J1 85.8 mm to (8.89, 16.5), turned to 180 degrees
- moved J8 85.1 mm to (22.9, 69.8), turned to 180 degrees
- moved J13 78.3 mm to (22.9, 25.4), turned to 180 degrees
- moved J20 67.9 mm to (36.8, 61.0), turned to 180 degrees
- moved J12 65.7 mm to (22.9, 34.3), turned to 180 degrees
- moved J19 63.8 mm to (36.8, 52.1), turned to 180 degrees
- moved J7 62.2 mm to (8.89, 69.8), turned to 180 degrees
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Routing:
- net 2-: track 0.00 -> 388.5 mm
- net 1-: track 0.00 -> 368.0 mm
- net 4-: track 0.00 -> 344.4 mm
- net 3-: track 0.00 -> 324.9 mm
- net 5-: track 0.00 -> 317.7 mm
- net 7-: track 0.00 -> 309.4 mm
- net 6-: track 0.00 -> 300.6 mm
- net 9-: track 0.00 -> 283.1 mm
- net 11-: track 0.00 -> 238.6 mm
- net 8-: track 0.00 -> 237.5 mm
- net 10-: track 0.00 -> 216.7 mm
- net 12-: track 0.00 -> 208.9 mm
- net 13-: track 0.00 -> 203.3 mm
- net 14-: track 0.00 -> 200.7 mm
- net 16-: track 0.00 -> 174.3 mm
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
Commit message: Update AMS Test Board rev1.brd
Routing:
- net 13-: track 203.3 -> 193.6 mm
- net 18-: track 129.4 -> 130.7 mm
- net 12-: track 208.9 -> 209.6 mm
Changed lines of the file:
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@@
 <contactref element="J41" pad="1"/>
 <contactref element="J19" pad="1"/>
-<wire x1="83.82" y1="73.66" x2="33.02" y2="73.66" width="0.254" layer="1"/>
-<wire x1="83.82" y1="73.66" x2="86.36" y2="71.12" width="0.254" layer="1"/>
-<wire x1="86.36" y1="71.12" x2="86.36" y2="64.77" width="0.254" layer="1"/>
-<wire x1="86.36" y1="64.77" x2="86.2584" y2="64.6684" width="0.254" layer="1"/>
-<wire x1="86.2584" y1="64.6684" x2="86.1314" y2="64.6684" width="0.254" layer="1"/>
+<wire x1="84.836" y1="73.66" x2="33.02" y2="73.66" width="0.254" layer="1"/>
+<wire x1="84.836" y1="73.66" x2="86.106" y2="72.39" width="0.254" layer="1"/>
+<wire x1="86.106" y1="72.39" x2="86.106" y2="64.6938" width="0.254" layer="1"/>
+<wire x1="86.1314" y1="64.6684" x2="86.106" y2="64.6938" width="0.254" layer="1"/>
 <wire x1="33.02" y1="73.66" x2="31.496" y2="72.136" width="0.254" layer="1"/>
 <wire x1="31.496" y1="72.136" x2="31.496" y2="64.77" width="0.254" layer="1"/>
@@
 <wire x1="35.83" y1="42.63" x2="35.83" y2="42.714" width="0.254" layer="1"/>
 <wire x1="35.83" y1="42.714" x2="30.861" y2="47.683" width="0.254" layer="1"/>
-<wire x1="110.49" y1="70.358" x2="106.553" y2="74.295" width="0.254" layer="1"/>
-<wire x1="110.49" y1="64.9478" x2="110.7694" y2="64.6684" width="0.254" layer="1"/>
-<wire x1="110.49" y1="70.358" x2="110.49" y2="64.9478" width="0.254" layer="1"/>
+<wire x1="110.744" y1="72.39" x2="108.839" y2="74.295" width="0.254" layer="1"/>
+<wire x1="110.744" y1="64.6938" x2="110.7694" y2="64.6684" width="0.254" layer="1"/>
+<wire x1="110.744" y1="72.39" x2="110.744" y2="64.6938" width="0.254" layer="1"/>
 <wire x1="32.766" y1="74.295" x2="30.861" y2="72.39" width="0.254" layer="1"/>
-<wire x1="106.553" y1="74.295" x2="32.766" y2="74.295" width="0.254" layer="1"/>
+<wire x1="108.839" y1="74.295" x2="32.766" y2="74.295" width="0.254" layer="1"/>
 <wire x1="30.861" y1="72.39" x2="30.861" y2="47.683" width="0.254" layer="1"/>
 <wire x1="35.925" y1="35.677" x2="35.83" y2="35.772" width="0.254" layer="1"/>
@@
 <wire x1="30.226" y1="30.581" x2="30.226" y2="72.644" width="0.254" layer="1"/>
 <wire x1="30.226" y1="72.644" x2="32.512" y2="74.93" width="0.254" layer="1"/>
-<wire x1="32.512" y1="74.93" x2="132.08" y2="74.93" width="0.254" layer="1"/>
-<wire x1="132.08" y1="74.93" x2="135.382" y2="71.628" width="0.254" layer="1"/>
-<wire x1="135.382" y1="71.628" x2="135.382" y2="64.6938" width="0.254" layer="1"/>
-<wire x1="135.382" y1="64.6938" x2="135.4074" y2="64.6684" width="0.254" layer="1"/>
+<wire x1="32.512" y1="74.93" x2="132.715" y2="74.93" width="0.254" layer="1"/>
+<wire x1="132.715" y1="74.93" x2="135.509" y2="72.136" width="0.254" layer="1"/>
+<wire x1="135.509" y1="72.136" x2="135.509" y2="64.77" width="0.254" layer="1"/>
+<wire x1="135.4074" y1="64.6684" x2="135.509" y2="64.77" width="0.254" layer="1"/>
 </signal>
 <signal name="15-">
@@
 <wire x1="23.876" y1="33.724" x2="23.86" y2="33.74" width="0.254" layer="1"/>
 <wire x1="23.876" y1="26.866" x2="23.876" y2="33.724" width="0.254" layer="1"/>
-<wire x1="23.86" y1="33.74" x2="18.288" y2="28.168" width="0.254" layer="1"/>
 <wire x1="180.8734" y1="16.4084" x2="180.8734" y2="24.2824" width="0.254" layer="1"/>
-<wire x1="18.288" y1="28.168" x2="18.288" y2="13.97" width="0.254" layer="1"/>
+<wire x1="18.288" y1="13.97" x2="18.288" y2="21.278" width="0.254" layer="1"/>
 <wire x1="18.288" y1="13.97" x2="178.435" y2="13.97" width="0.254" layer="1"/>
 <wire x1="178.435" y1="13.97" x2="180.8734" y2="16.4084" width="0.254" layer="1"/>
+<wire x1="18.288" y1="21.278" x2="21.86" y2="24.85" width="0.254" layer="1"/>
 </signal>
 <signal name="12-">
@@
 <wire x1="28.956" y1="47.726" x2="23.86" y2="42.63" width="0.254" layer="1"/>
 <wire x1="28.956" y1="73.152" x2="32.004" y2="76.2" width="0.254" layer="1"/>
-<wire x1="180.34" y1="76.2" x2="184.785" y2="71.755" width="0.254" layer="1"/>
-<wire x1="184.785" y1="71.755" x2="184.785" y2="65.278" width="0.254" layer="1"/>
-<wire x1="184.785" y1="65.278" x2="184.404" y2="64.897" width="0.254" layer="1"/>
+<wire x1="181.102" y1="76.2" x2="185.039" y2="72.263" width="0.254" layer="1"/>
+<wire x1="185.039" y1="72.263" x2="185.039" y2="65.532" width="0.254" layer="1"/>
+<wire x1="185.039" y1="65.532" x2="184.404" y2="64.897" width="0.254" layer="1"/>
 <wire x1="184.404" y1="64.897" x2="184.6326" y2="64.6684" width="0.254" layer="1"/>
 <wire x1="184.6326" y1="64.6684" x2="184.9374" y2="64.6684" width="0.254" layer="1"/>
 <wire x1="28.956" y1="47.726" x2="28.956" y2="73.152" width="0.254" layer="1"/>
-<wire x1="32.004" y1="76.2" x2="180.34" y2="76.2" width="0.254" layer="1"/>
+<wire x1="32.004" y1="76.2" x2="181.102" y2="76.2" width="0.254" layer="1"/>
 </signal>
 <signal name="11-">
@@
 <contactref element="J43" pad="1"/>
 <wire x1="59.69" y1="64.6938" x2="59.7154" y2="64.6684" width="0.1524" layer="1"/>
-<wire x1="59.69" y1="71.755" x2="59.69" y2="64.6938" width="0.254" layer="1"/>
-<wire x1="58.42" y1="73.025" x2="59.69" y2="71.755" width="0.254" layer="1"/>
+<wire x1="59.69" y1="72.263" x2="59.69" y2="64.6938" width="0.254" layer="1"/>
+<wire x1="58.928" y1="73.025" x2="59.69" y2="72.263" width="0.254" layer="1"/>
 <wire x1="37.83" y1="69.3" x2="35.687" y2="71.443" width="0.254" layer="1"/>
 <wire x1="35.687" y1="71.443" x2="35.687" y2="72.39" width="0.254" layer="1"/>
 <wire x1="35.687" y1="72.39" x2="36.322" y2="73.025" width="0.254" layer="1"/>
-<wire x1="36.322" y1="73.025" x2="58.42" y2="73.025" width="0.254" layer="1"/>
+<wire x1="36.322" y1="73.025" x2="58.928" y2="73.025" width="0.254" layer="1"/>
 </signal>
 </signals>

Commit message: AMS Test Board Update
Created additional space between battery connectors and added fuses.
Parts:
- added F1, F10, F11, F12, F13, F14, F15, F16, F17, F18, F19, F2, F20, F21, F22, F3, F4, F5, F6, F7, F8, F9: FUSE_OMF_125_.5A, HyTechDevices:OMF_125
- moved J21 8.36 mm to (39.1, 77.9)
- moved J7 8.29 mm to (6.90, 77.9)
- moved J8 8.05 mm to (23.0, 77.9)
- moved J15 7.15 mm to (39.1, 9.73)
- moved J1 7.06 mm to (6.90, 9.73)
- moved J14 6.78 mm to (23.0, 9.73)
- moved J20 6.02 mm to (39.1, 66.5)
- moved J6 5.92 mm to (6.90, 66.5)
- moved J9 5.58 mm to (23.0, 66.5)
- moved J16 4.87 mm to (39.1, 21.1)
- moved J2 4.74 mm to (6.90, 21.1)
- moved J13 4.31 mm to (23.0, 21.1)
- moved J19 3.85 mm to (39.1, 55.2)
- moved J5 3.69 mm to (6.90, 55.2)
- moved J10 3.11 mm to (23.0, 55.2)
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Connections:
- new net N$1: F1.1, J22.1
- new net N$10: F10.1, J31.1
- new net N$11: F11.1, J32.1
- new net N$12: F12.1, J33.1
- new net N$13: F13.1, J34.1
- new net N$14: F14.1, J35.1
- new net N$15: F15.1, J36.1
- new net N$16: F16.1, J37.1
- new net N$17: F17.1, J38.1
- new net N$18: F18.1, J39.1
- new net N$19: F19.1, J40.1
- new net N$2: F2.1, J23.1
- new net N$20: F20.1, J41.1
- new net N$21: F21.1, J42.1
- new net N$22: F22.1, J43.1
- new net N$3: F3.1, J24.1
- new net N$4: F4.1, J25.1
- new net N$5: F5.1, J26.1
- new net N$6: F6.1, J27.1
- new net N$7: F7.1, J28.1
- new net N$8: F8.1, J29.1
- new net N$9: F9.1, J30.1
- net 1-: now also F1.2; no longer J22.1
- net 10-: now also F10.2; no longer J31.1
- net 11-: now also F11.2; no longer J32.1
- net 12-: now also F12.2; no longer J33.1
- net 13-: now also F13.2; no longer J34.1
- net 14-: now also F14.2; no longer J35.1
- net 15-: now also F15.2; no longer J36.1
- net 16-: now also F16.2; no longer J37.1
- net 17-: now also F17.2; no longer J38.1
- net 18-: now also F18.2; no longer J39.1
- net 19-: now also F19.2; no longer J40.1
- net 2-: now also F2.2; no longer J23.1
- net 20-: now also F20.2; no longer J41.1
- net 21+: now also F22.2; no longer J43.1
- net 21-: now also F21.2; no longer J42.1
- net 3-: now also F3.2; no longer J24.1
- net 4-: now also F4.2; no longer J25.1
- net 5-: now also F5.2; no longer J26.1
- net 6-: now also F6.2; no longer J27.1
- net 7-: now also F7.2; no longer J28.1
- net 8-: now also F8.2; no longer J29.1
- net 9-: now also F9.2; no longer J30.1
Routing:
- net 9-: track 283.1 -> 329.4 mm
- net 7-: track 309.4 -> 355.7 mm
- net 14-: track 200.7 -> 245.1 mm
- net 16-: track 174.7 -> 218.8 mm
- net 5-: track 317.7 -> 359.3 mm
- net 11-: track 238.6 -> 279.9 mm
- net N$20: track 0.00 -> 39.8 mm
- net 12-: track 209.6 -> 248.6 mm
- net 18-: track 130.7 -> 169.4 mm
- net N$2: track 0.00 -> 38.4 mm
- net N$12: track 0.00 -> 38.0 mm
- net N$4: track 0.00 -> 37.8 mm
- net N$16: track 0.00 -> 37.7 mm
- net N$9: track 0.00 -> 37.5 mm
- net N$8: track 0.00 -> 37.5 mm
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