File: ESF Schematics/2023/Shutdown Circuit Schematic.sch (EAGLE design)
At the start: 73 parts, among them J1 CONNECTOR-1_LCAX2-14F-E, J2 CONNECTOR-1_LCAX2-14F-E, J3 CONNECTOR-1_LCAX2-14F-E, J4 CONNECTOR-1_LCAX2-14F-E, Q1 MOSFET_N-CHANNEL, Q2 MOSFET_N-CHANNEL, U1 LOGICGATE_INVERTER, U2 LOGICGATE_INVERTER

Commit message: WIP
Parts:
- removed F2, F4: 10A, HyTechSymbolsTemp:FUSE
- removed POWER_ON: BUTTON_NO, HyTechSymbolsTemp:BUTTON_NO
- removed POWER_SWITCHING_RELAY: RELAY_SOLIDSTATE_NO_CMX60D20, HyTechSymbolsTemp:RELAY_SOLIDSTATE_NO_CMX60D20
- removed R1: 10k, HyTechSymbolsTemp:RESISTOR
- removed U$1: DC-DC_CONVERTER_DCM4623TD2J13D0T70, HyTechSymbols:DC-DC_CONVERTER_DCM4623TD2J13D0T70
- removed U$9: POWER_SWITCHING_BOARD, HyTechSymbols:POWER_SWITCHING_BOARD
- added BOTS_SENSE_RELAY: RELAY_DPDT_RT424009, HyTechSymbolsTemp:RELAY_DPDT_RT424009
- D1, D2: value DIODE_SHOTTKY -> DIODE; device HyTechSymbolsTemp:DIODE_SHOTTKY -> HyTechSymbolsTemp:DIODE
Connections:
- removed net DCDC+: F4.1, U$9.V1
- removed net DCDC-: U$1.-OUT
- removed net N$17: D1.C, D2.C, POWER_SWITCHING_RELAY.CONTROL+, R1.2, U$9.!SHDN
- removed net N$18: S9.P, U$9.VOUT
- removed net N$20: F2.1, S9.S
- removed net N$30: F4.2, U$1.+OUT
- new net BOTS_SENSE: BOTS_SENSE_RELAY.COIL+, D2.C
- net GLV_SYSTEMS: now also S9.S; no longer D2.A, F2.2
- net GND: now also BOTS_SENSE_RELAY.4; no longer POWER_SWITCHING_RELAY.CONTROL-, R1.1, U$9.GND
- net N$15: now also BOTS_SENSE_RELAY.6, SOFTWARE_SHDN_RELAY.5; no longer F1.2, POWER_ON.P$1, POWER_SWITCHING_RELAY.CONTACT1
- net N$16: now also BOTS_SENSE_RELAY.3, BOTS_SENSE_RELAY.COIL-, D1.A, D2.A; no longer POWER_SWITCHING_RELAY.CONTACT2, U$9.V2
- net N$19: now also BOTS_SENSE_RELAY.5, S1.P; no longer D1.A, POWER_ON.P$2
- net N$2: now also D1.C
- net N$7: now also F1.2, S9.P; no longer S1.P, SOFTWARE_SHDN_RELAY.5
- net TS+: no longer U$1.+IN
- net TS-UNFUSED: no longer U$1.-IN
Other:
- note removed: "16AWG"
- moved on the sheet: AMS_RELAY, BSPD_RELAY, D10, D3, D4, D5, D6, D7, D8, D9, F1, F3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

Commit message: minor changes
Connections:
- net N$12: no longer S5.P
- net N$13: no longer S6.P
- net N$51: no longer S8.P
- net N$8: no longer S4.P
Changed lines of the file:
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@@
 <net name="N$8" class="0">
 <segment>
-<wire x1="195.58" y1="132.08" x2="187.96" y2="132.08" width="0.1524" layer="91"/>
 <pinref part="S3" gate="SPST" pin="O"/>
 <wire x1="195.58" y1="132.08" x2="195.58" y2="134.62" width="0.1524" layer="91"/>
-<pinref part="S4" gate="SPST" pin="P"/>
 </segment>
 </net>
@@
 <net name="N$12" class="0">
 <segment>
-<wire x1="177.8" y1="132.08" x2="170.18" y2="132.08" width="0.1524" layer="91"/>
 <pinref part="S4" gate="SPST" pin="O"/>
 <wire x1="177.8" y1="134.62" x2="177.8" y2="132.08" width="0.1524" layer="91"/>
-<pinref part="S5" gate="SPST" pin="P"/>
 </segment>
 </net>
 <net name="N$13" class="0">
 <segment>
-<wire x1="152.4" y1="132.08" x2="160.02" y2="132.08" width="0.1524" layer="91"/>
 <pinref part="S5" gate="SPST" pin="O"/>
 <wire x1="160.02" y1="134.62" x2="160.02" y2="132.08" width="0.1524" layer="91"/>
-<pinref part="S6" gate="SPST" pin="P"/>
 </segment>
 </net>
@@
 <net name="N$51" class="0">
 <segment>
-<wire x1="124.46" y1="132.08" x2="116.84" y2="132.08" width="0.1524" layer="91"/>
 <pinref part="S7" gate="SPST" pin="S"/>
 <wire x1="124.46" y1="132.08" x2="124.46" y2="129.54" width="0.1524" layer="91"/>
-<pinref part="S8" gate="SPST" pin="P"/>
-</segment>
-</net>
+</segment>
+</net>

Commit message: more work done
Parts:
- added DISCHARGE_RES1, DISCHARGE_RES2: 15k, HyTechSymbolsTemp:RESISTOR
- added PRECHARGE_RES1: 1.5k, HyTechSymbolsTemp:RESISTOR
- added S10, S11, S12, S13: SWITCH_SPST_, HyTechSymbols:SWITCH_SPST_
- added U$1, U$4: SEGMENT, HyTechSymbols:SEGMENT
- added U$2, U$3, U$5, U$6: MAINTENANCE_PLUG_104742-2, HyTechSymbolsTemp:MAINTENANCE_PLUG_104742-2
- AIR+, AIR-: value RELAY_SPST_NO_GX23BA -> RELAY_SPST_NO_; device HyTechSymbolsTemp:RELAY_SPST_NO_GX23BA -> HyTechSymbols:RELAY_SPST_NO_; MPN (none) -> GX23CA
- AMS_RELAY, BOTS_SENSE_RELAY, BSPD_RELAY, IMD_RELAY, SOFTWARE_SHDN_RELAY: value RELAY_DPDT_RT424009 -> RELAY_DPDT_RT424024; device HyTechSymbolsTemp:RELAY_DPDT_RT424009 -> HyTechSymbols:RELAY_DPDT_RT424024
- DISCHARGE: value RELAY_SPST_NC_3350-4275-126 -> RELAY_SPST_NC_DBR72410; device HyTechSymbolsTemp:RELAY_SPST_NC_3350-4275-126 -> HyTechSymbols:RELAY_SPST_NC_DBR72410
- DISCHARGE_RES: value 10k -> 15k
- PRECHARGE: value RELAY_SPST_NO_3350-1275-126 -> RELAY_SPST_NO_DAR72410; device HyTechSymbolsTemp:RELAY_SPST_NO_3350-1275-126 -> HyTechSymbols:RELAY_SPST_NO_DAR72410
- PRECHARGE_RES: value 750 -> 1.5k
- R3: value 1k -> 2.2k
- S7: MPN HPK Interlock -> Inverter HVP Interlock
Connections:
- new net N$17: S12.P, S13.S
- new net N$18: S11.P, S12.S
- new net N$20: S10.P, S11.S
- new net N$30: S10.S, S2.P
- new net N$54: U$1.+, U$3.1
- new net N$55: U$2.P$1, U$3.P$1
- new net N$56: U$36.1, U$4.-
- new net N$57: U$4.+, U$6.1
- new net N$58: U$5.P$1, U$6.P$1
- net BOTS_SENSE: now also S2.O, S3.P
- net GND: now also LATCHING_BUTTON.P$1; no longer LATCHING_BUTTON.P$2
- net N$12: now also S5.P
- net N$13: now also S6.P
- net N$19: now also S13.P; no longer S1.P
- net N$2: now also LATCHING_BUTTON.P$2; no longer LATCHING_BUTTON.P$1
- net N$21: now also S8.P; no longer S7.P
- net N$23: now also U$1.-, U$5.1; no longer U$15.-, U$36.1
- net N$26: now also PRECHARGE_RES1.1
- net N$29: now also DISCHARGE_RES1.1, DISCHARGE_RES2.1
- net N$4: now also S7.P; no longer S2.P
- net N$51: now also S4.P
- net N$8: now also S1.P
- net N$9: now also U$15.-, U$2.1; no longer S2.O, S3.P
- net TS+UNFUSED: now also PRECHARGE_RES1.2
- net TS-UNFUSED: now also DISCHARGE_RES1.2, DISCHARGE_RES2.2
Other:
- note added: "16AWG"
- note added: "Inverter Enclosure"
- moved on the sheet: AIR+, AIR-, AMS_RELAY, BOTS_SENSE_RELAY, BSPD_RELAY, D1, D10, D2, D3, D4, D5, D6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

Commit message: Many changes
Changed lines of the file:
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@@
 <wire x1="66.04" y1="72.39" x2="6.35" y2="72.39" width="0.8128" layer="97"/>
 <wire x1="6.35" y1="72.39" x2="6.35" y2="127" width="0.8128" layer="97"/>
-<text x="10.16" y="119.38" size="3.81" layer="97">Inverter Enclosure</text>
+<text x="7.62" y="119.38" size="4.572" layer="97">Inverter Enclosure</text>
 <text x="218.44" y="104.14" size="1.27" layer="97" align="top-left">17.5mm^2</text>
 <text x="231.14" y="104.14" size="1.27" layer="97" align="top-left">17.5mm^2</text>
@@
 <attribute name="MPN" x="238.252" y="76.2" size="1.27" layer="95" rot="MR270" align="top-left"/>
 </instance>
-<instance part="J3" gate="G$1" x="147.32" y="50.8" smashed="yes" rot="R180">
-<attribute name="MPN" x="147.32" y="56.515" size="1.27" layer="96" rot="R180" align="top-left"/>
-<attribute name="MANUFACTURER" x="147.32" y="50.038" size="1.27" layer="96" rot="R180"/>
+<instance part="J3" gate="G$1" x="172.72" y="50.8" smashed="yes" rot="R180">
+<attribute name="MPN" x="172.72" y="56.515" size="1.27" layer="96" rot="R180" align="top-left"/>
+<attribute name="MANUFACTURER" x="172.72" y="50.038" size="1.27" layer="96" rot="R180"/>
 </instance>
 <instance part="J4" gate="G$1" x="180.34" y="55.88" smashed="yes">
@@
 <segment>
 <pinref part="J3" gate="G$1" pin="1"/>
-<wire x1="111.76" y1="53.34" x2="137.16" y2="53.34" width="0.4445" layer="91"/>
+<wire x1="111.76" y1="53.34" x2="162.56" y2="53.34" width="0.4445" layer="91"/>
 <junction x="111.76" y="53.34"/>
 <wire x1="111.76" y1="58.42" x2="111.76" y2="53.34" width="0.4445" layer="91"/>

Commit message: minor changes
Parts:
- R3: value 2.2k -> 3.3k
Changed lines of the file:
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@@
 <attribute name="DESCRIPTION_1" value="ESF compliant representation of the HT06"/>
 <attribute name="DESCRIPTION_2" value="shutdown circuit."/>
-<attribute name="DESIGNER_SCHEMATIC" value="Zekun Li"/>
-<attribute name="ENGINEER" value="Zekun Li"/>
-<attribute name="REVIEWER_SCHEMATIC" value="Arvind Srinivasan"/>
+<attribute name="DESIGNER_SCHEMATIC" value="Liwei Sun"/>
+<attribute name="ENGINEER" value="Liwei Sun"/>
 </part>
 <part name="U$20" library="HyTechSymbolsTemp" deviceset="MAINTENANCE_PLUG_*" device="" technology="104742-2"/>
@@
 <part name="P18" library="HyTechSupplies" deviceset="GND" device=""/>
 <part name="R2" library="HyTechSymbolsTemp" deviceset="RESISTOR" device="" value="39"/>
-<part name="R3" library="HyTechSymbolsTemp" deviceset="RESISTOR" device="" value="2.2k"/>
+<part name="R3" library="HyTechSymbolsTemp" deviceset="RESISTOR" device="" value="3.3k"/>
 <part name="S1" library="HyTechSymbols" deviceset="SWITCH_SPST_*" device="" technology="INERTIA_SWITCH"/>
 <part name="S2" library="HyTechSymbols" deviceset="SWITCH_SPST_*" device="">

Commit message: post 1st review, cursed
Parts:
- S7: MPN Inverter HVP Interlock -> Accumulator HVP Interlock
Connections:
- net N$13: now also S7.P; no longer S6.P
- net N$4: now also S4.P; no longer S7.P
- net N$51: now also S6.P; no longer S4.P
Changed lines of the file:
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@@
 </part>
 <part name="S7" library="HyTechSymbols" deviceset="SWITCH_SPST_*" device="">
-<attribute name="MPN" value="Inverter HVP Interlock"/>
+<attribute name="MPN" value="Accumulator HVP Interlock"/>
 </part>
 <part name="S8" library="HyTechSymbols" deviceset="SWITCH_SPST_*" device="" technology="35-210-100-R-900"/>
@@
 <text x="30.48" y="170.18" size="1.27" layer="97" align="bottom-center">GLVMS</text>
 <text x="45.72" y="144.78" size="1.27" layer="97" align="bottom-center">TSMS</text>
-<text x="83.82" y="144.78" size="1.27" layer="97" align="bottom-center">Right BRB</text>
-<text x="101.6" y="144.78" size="1.27" layer="97" align="bottom-center">Left BRB</text>
+<text x="101.6" y="144.78" size="1.27" layer="97" align="bottom-center">Right BRB</text>
+<text x="119.38" y="144.78" size="1.27" layer="97" align="bottom-center">Left BRB</text>
 <text x="154.94" y="144.78" size="1.27" layer="97" align="bottom-center">Cockpit BRB</text>
 <text x="137.16" y="144.78" size="1.27" layer="97" align="bottom-center">Inertia Switch</text>
 <text x="17.78" y="170.18" size="1.27" layer="97" align="top-left">16AWG</text>
 <text x="68.58" y="142.24" size="1.27" layer="97" align="top-left">22AWG</text>
+<text x="104.14" y="142.24" size="1.27" layer="97" align="top-left">22AWG</text>
+<text x="124.46" y="142.24" size="1.27" layer="97" align="top-left">22AWG</text>
 <text x="86.36" y="142.24" size="1.27" layer="97" align="top-left">22AWG</text>
-<text x="106.68" y="142.24" size="1.27" layer="97" align="top-left">22AWG</text>
-<text x="121.92" y="142.24" size="1.27" layer="97" align="top-left">22AWG</text>
 <text x="142.24" y="142.24" size="1.27" layer="97" align="top-left">22AWG</text>
 <text x="182.88" y="142.24" size="1.27" layer="97" align="top-left">22AWG</text>
@@
 <attribute name="MPN" x="154.94" y="136.398" size="1.27" layer="96" rot="MR0" align="top-center"/>
 </instance>
-<instance part="S4" gate="SPST" x="101.6" y="139.7" smashed="yes" rot="MR0">
+<instance part="S4" gate="SPST" x="119.38" y="139.7" smashed="yes" rot="MR0">
+<attribute name="MANUFACTURER" x="119.38" y="143.002" size="1.27" layer="96" rot="MR0" align="bottom-center"/>
+<attribute name="MPN" x="119.38" y="136.398" size="1.27" layer="96" rot="MR0" align="top-center"/>
+</instance>
+<instance part="S5" gate="SPST" x="101.6" y="139.7" smashed="yes" rot="MR0">
 <attribute name="MANUFACTURER" x="101.6" y="143.002" size="1.27" layer="96" rot="MR0" align="bottom-center"/>
 <attribute name="MPN" x="101.6" y="136.398" size="1.27" layer="96" rot="MR0" align="top-center"/>
-</instance>
-<instance part="S5" gate="SPST" x="83.82" y="139.7" smashed="yes" rot="MR0">
-<attribute name="MANUFACTURER" x="83.82" y="143.002" size="1.27" layer="96" rot="MR0" align="bottom-center"/>
-<attribute name="MPN" x="83.82" y="136.398" size="1.27" layer="96" rot="MR0" align="top-center"/>
 </instance>
 <instance part="S6" gate="SPST" x="66.04" y="139.7" smashed="yes" rot="MR0">
@@
 <attribute name="MPN" x="66.04" y="136.398" size="1.27" layer="96" rot="MR0" align="top-center"/>
 </instance>
-<instance part="S7" gate="SPST" x="119.38" y="139.7" smashed="yes" rot="MR0">
-<attribute name="MANUFACTURER" x="119.38" y="143.002" size="1.27" layer="96" rot="MR0" align="bottom-center"/>
-<attribute name="MPN" x="119.38" y="136.398" size="1.27" layer="96" rot="MR0" align="top-center"/>
+<instance part="S7" gate="SPST" x="83.82" y="139.7" smashed="yes" rot="MR0">
+<attribute name="MANUFACTURER" x="83.82" y="143.002" size="1.27" layer="96" rot="MR0" align="bottom-center"/>
+<attribute name="MPN" x="83.82" y="136.398" size="1.27" layer="96" rot="MR0" align="top-center"/>
 </instance>
 <instance part="S8" gate="SPST" x="45.72" y="139.7" smashed="yes" rot="MR0">
@@
 <segment>
 <pinref part="S4" gate="SPST" pin="O"/>
+<wire x1="114.3" y1="142.24" x2="114.3" y2="139.7" width="0.1524" layer="91"/>
+<pinref part="S5" gate="SPST" pin="P"/>
+<wire x1="114.3" y1="139.7" x2="106.68" y2="139.7" width="0.1524" layer="91"/>
+</segment>
+</net>
+<net name="N$13" class="0">
+<segment>
+<pinref part="S5" gate="SPST" pin="O"/>
 <wire x1="96.52" y1="142.24" x2="96.52" y2="139.7" width="0.1524" layer="91"/>
-<pinref part="S5" gate="SPST" pin="P"/>
+<pinref part="S7" gate="SPST" pin="P"/>
 <wire x1="96.52" y1="139.7" x2="88.9" y2="139.7" width="0.1524" layer="91"/>
-</segment>
-</net>
-<net name="N$13" class="0">
-<segment>
-<pinref part="S5" gate="SPST" pin="O"/>
-<wire x1="78.74" y1="142.24" x2="78.74" y2="139.7" width="0.1524" layer="91"/>
-<pinref part="S6" gate="SPST" pin="P"/>
-<wire x1="78.74" y1="139.7" x2="71.12" y2="139.7" width="0.1524" layer="91"/>
 </segment>
 </net>
@@
 <segment>
 <pinref part="S7" gate="SPST" pin="S"/>
-<wire x1="114.3" y1="139.7" x2="114.3" y2="137.16" width="0.1524" layer="91"/>
-<pinref part="S4" gate="SPST" pin="P"/>
-<wire x1="114.3" y1="139.7" x2="106.68" y2="139.7" width="0.1524" layer="91"/>
+<wire x1="78.74" y1="139.7" x2="78.74" y2="137.16" width="0.1524" layer="91"/>
+<pinref part="S6" gate="SPST" pin="P"/>
+<wire x1="78.74" y1="139.7" x2="71.12" y2="139.7" width="0.1524" layer="91"/>
 </segment>
 </net>
@@
 <pinref part="S1" gate="SPST" pin="O"/>
 <wire x1="132.08" y1="142.24" x2="132.08" y2="139.7" width="0.1524" layer="91"/>
-<pinref part="S7" gate="SPST" pin="P"/>
+<pinref part="S4" gate="SPST" pin="P"/>
 <wire x1="132.08" y1="139.7" x2="124.46" y2="139.7" width="0.1524" layer="91"/>
 </segment>

Commit message: minor changes, still cursed
Connections:
- removed net N$30: S10.S, S2.P
- new net N$59: S10.S, S3.P
- net BOTS_SENSE: now also BOTS_SENSE_RELAY.6; no longer S3.P
- net N$15: now also S2.P; no longer BOTS_SENSE_RELAY.6
Other:
- moved on the sheet: BOTS_SENSE_RELAY, D1, D2

Commit message: TS big changes
Connections:
- net BOTS_SENSE: now also IMD_RELAY.6; no longer BOTS_SENSE_RELAY.6
- net N$15: now also BOTS_SENSE_RELAY.6; no longer S2.P
- net N$22: now also S2.P; no longer IMD_RELAY.6
Other:
- moved on the sheet: AMS_RELAY, BOTS_SENSE_RELAY, BSPD_RELAY, D1, D10, D2, D3, D4, D5, D6, D7, D8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
