File: EAGLE Board Designs/Main ECU/MainECU rev12.brd (EAGLE design)
At the start: 127 x 152.4 mm, 365 parts, among them J1 CONNECTOR-40__, J2 ADIS16460, J3 CONNECTOR-40__, K1 RELAY_DPDT_RT424024, K10 RELAY_DPDT_RT424024, K11 RELAY_DPDT_RT424024, K12 RELAY_DPDT_RT424024, K9 RELAY_DPDT_RT424024, Q3 TRANSISTOR_P_MOS_SOT-23_DMP30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, Q4 TRANSISTOR_N_MOS__DMG3406L-7, Q5 TRANSISTOR_P_MOS_SOT-23_DMP30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, Q6 TRANSISTOR_N_MOS__DMG3406L-7, U1 VOLTAGE_REGULATOR_SOT-223_3.3V, U10 OPAMP_1_CHANNEL_OPA991, U11 LOGICGATE_OR, U12 LOGICGATE_OR, U13 LOGICGATE_OR, U14 MAX7400, U15 MAX7400, U16 MAX7400, U17 MAX7400, U18 MAX7400, U19 MAX7400, U2 TCAN1051HQV-Q1, U20 MAX7400, U21 MAX7400, U22 MAX7400, U23 ADC128S022, U24 MAX7400, U25 MAX7400, U3 TCAN1051HQV-Q1, U32 ADC128S022, U33 TCAN1051HQV-Q1, U34 OPAMP_1_CHANNEL_OPA991, U37 OPAMP_1_CHANNEL_OPA991, U38 LOGICGATE_OR, U39 OPAMP_1_CHANNEL_OPA991, U4 TCAN1051HQV-Q1, U41 OPAMP_1_CHANNEL_OPA991, U42 LOGICGATE_AND_DCK3, U43 OPAMP_1_CHANNEL_OPA991, U44 LOGICGATE_NOR, U45 TCAN1051HQV-Q1, U46 TCAN1051HQV-Q1, U5 ADM8316WBX30, U6 ADC128S022, U7 ADC128S022, U8 OPAMP_1_CHANNEL_OPA991, U9 OPAMP_1_CHANNEL_OPA991

Commit message: added jumpers
Parts:
- added JP4, JP5, JP6, JP7: JUMPER__1X02, HyTechDevices:1X02
Connections:
- new net ACCEL_1_PRE: JP4.2, R93.2, U20.2
- new net ACCEL_2_PRE: JP5.2, R95.2, U21.2
- new net BRAKE_1_PRE: JP6.2, R97.2, U22.2
- new net BRAKE_2_PRE: JP7.2, R99.2, U24.2
- net ACCEL_1_EXT: now also JP4.1; no longer R93.2, U20.2
- net ACCEL_2_EXT: now also JP5.1; no longer R95.2, U21.2
- net BRAKE_1_EXT: now also JP6.1; no longer R97.2, U22.2
- net BRAKE_2_EXT: now also JP7.1; no longer R99.2, U24.2
Changed lines of the file:
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@@
 <attribute name="VOLTAGE" value="10V" x="-54.864" y="-323.596" size="1.778" layer="27" display="off"/>
 </element>
+<element name="JP4" library="HyTechDevices" package="1X02" value="JUMPER__1X02" x="-92.456" y="-303.022" smashed="yes">
+<attribute name="DKPN" value="S1011EC-02-ND" x="-92.456" y="-303.022" size="1.778" layer="27" display="off"/>
+<attribute name="MANUFACTURER" value="Sullins Connector Solutions" x="-92.456" y="-303.022" size="1.778" layer="27" display="off"/>
+<attribute name="MOPN" value="" x="-92.456" y="-303.022" size="1.778" layer="27" display="off"/>
+<attribute name="MPN" value="PRPC002SAAN-RC" x="-92.456" y="-303.022" size="1.778" layer="27" display="off"/>
+<attribute name="NAME" x="-92.456" y="-301.498" size="0.8128" layer="25" font="vector" align="bottom-center"/>
+</element>
+<element name="JP5" library="HyTechDevices" package="1X02" value="JUMPER__1X02" x="-92.456" y="-307.34" smashed="yes">
+<attribute name="DKPN" value="S1011EC-02-ND" x="-92.456" y="-307.34" size="1.778" layer="27" display="off"/>
+<attribute name="MANUFACTURER" value="Sullins Connector Solutions" x="-92.456" y="-307.34" size="1.778" layer="27" display="off"/>
+<attribute name="MOPN" value="" x="-92.456" y="-307.34" size="1.778" layer="27" display="off"/>
+<attribute name="MPN" value="PRPC002SAAN-RC" x="-92.456" y="-307.34" size="1.778" layer="27" display="off"/>
+<attribute name="NAME" x="-92.456" y="-305.816" size="0.8128" layer="25" font="vector" align="bottom-center"/>
+</element>
+<element name="JP6" library="HyTechDevices" package="1X02" value="JUMPER__1X02" x="-92.456" y="-311.658" smashed="yes">
+<attribute name="DKPN" value="S1011EC-02-ND" x="-92.456" y="-311.658" size="1.778" layer="27" display="off"/>
+<attribute name="MANUFACTURER" value="Sullins Connector Solutions" x="-92.456" y="-311.658" size="1.778" layer="27" display="off"/>
+<attribute name="MOPN" value="" x="-92.456" y="-311.658" size="1.778" layer="27" display="off"/>
+<attribute name="MPN" value="PRPC002SAAN-RC" x="-92.456" y="-311.658" size="1.778" layer="27" display="off"/>
+<attribute name="NAME" x="-92.456" y="-310.134" size="0.8128" layer="25" font="vector" align="bottom-center"/>
+</element>
+<element name="JP7" library="HyTechDevices" package="1X02" value="JUMPER__1X02" x="-92.456" y="-315.976" smashed="yes">
+<attribute name="DKPN" value="S1011EC-02-ND" x="-92.456" y="-315.976" size="1.778" layer="27" display="off"/>
+<attribute name="MANUFACTURER" value="Sullins Connector Solutions" x="-92.456" y="-315.976" size="1.778" layer="27" display="off"/>
+<attribute name="MOPN" value="" x="-92.456" y="-315.976" size="1.778" layer="27" display="off"/>
+<attribute name="MPN" value="PRPC002SAAN-RC" x="-92.456" y="-315.976" size="1.778" layer="27" display="off"/>
+<attribute name="NAME" x="-92.456" y="-314.452" size="0.8128" layer="25" font="vector" align="bottom-center"/>
+</element>
 </elements>
 <signals>
@@
 <signal name="ACCEL_1_EXT">
 <contactref element="J1" pad="29"/>
-<contactref element="R93" pad="2"/>
-<contactref element="U20" pad="2"/>
-<wire x1="-51.474" y1="-212.852" x2="-53.213" y2="-196.6595" width="0" layer="19" extent="1-1"/>
-<wire x1="27.83" y1="147.05" x2="-53.213" y2="-196.6595" width="0" layer="19" extent="1-1"/>
+<contactref element="JP4" pad="1"/>
+<wire x1="-93.726" y1="-303.022" x2="27.83" y2="147.05" width="0" layer="19" extent="1-1"/>
 </signal>
 <signal name="ACCEL_2_EXT">
 <contactref element="J1" pad="30"/>
-<contactref element="R95" pad="2"/>
-<contactref element="U21" pad="2"/>
-<wire x1="-45.378" y1="-212.852" x2="-45.847" y2="-196.6595" width="0" layer="19" extent="1-1"/>
-<wire x1="27.83" y1="145.05" x2="-45.847" y2="-196.6595" width="0" layer="19" extent="1-1"/>
+<contactref element="JP5" pad="1"/>
+<wire x1="-93.726" y1="-307.34" x2="27.83" y2="145.05" width="0" layer="19" extent="1-1"/>
 </signal>
 <signal name="BRAKE_1_EXT">
 <contactref element="J1" pad="27"/>
-<contactref element="R97" pad="2"/>
-<contactref element="U22" pad="2"/>
-<wire x1="-53.213" y1="-203.7715" x2="-39.282" y2="-212.852" width="0" layer="19" extent="1-1"/>
-<wire x1="29.83" y1="147.05" x2="-53.213" y2="-203.7715" width="0" layer="19" extent="1-1"/>
+<contactref element="JP6" pad="1"/>
+<wire x1="-93.726" y1="-311.658" x2="29.83" y2="147.05" width="0" layer="19" extent="1-1"/>
 </signal>
 <signal name="BRAKE_2_EXT">
 <contactref element="J1" pad="28"/>
-<contactref element="R99" pad="2"/>
-<contactref element="U24" pad="2"/>
-<wire x1="-51.474" y1="-215.9" x2="-45.847" y2="-203.7715" width="0" layer="19" extent="1-1"/>
-<wire x1="29.83" y1="145.05" x2="-45.847" y2="-203.7715" width="0" layer="19" extent="1-1"/>
+<contactref element="JP7" pad="1"/>
+<wire x1="-93.726" y1="-315.976" x2="29.83" y2="145.05" width="0" layer="19" extent="1-1"/>
 </signal>
 <signal name="BRAKE_PRESSURE_F_EXT">
@@
 <wire x1="-49.518" y1="-290.068" x2="-47.918" y2="-299.212" width="0" layer="19" extent="1-1"/>
 </signal>
+<signal name="ACCEL_1_PRE">
+<contactref element="R93" pad="2"/>
+<contactref element="U20" pad="2"/>
+<contactref element="JP4" pad="2"/>
+<wire x1="-51.474" y1="-212.852" x2="-53.213" y2="-196.6595" width="0" layer="19" extent="1-1"/>
+<wire x1="-91.186" y1="-303.022" x2="-51.474" y2="-212.852" width="0" layer="19" extent="1-1"/>
+</signal>
+<signal name="ACCEL_2_PRE">
+<contactref element="R95" pad="2"/>
+<contactref element="U21" pad="2"/>
+<contactref element="JP5" pad="2"/>
+<wire x1="-45.378" y1="-212.852" x2="-45.847" y2="-196.6595" width="0" layer="19" extent="1-1"/>
+<wire x1="-91.186" y1="-307.34" x2="-45.378" y2="-212.852" width="0" layer="19" extent="1-1"/>
+</signal>
+<signal name="BRAKE_1_PRE">
+<contactref element="R97" pad="2"/>
+<contactref element="U22" pad="2"/>
+<contactref element="JP6" pad="2"/>
+<wire x1="-53.213" y1="-203.7715" x2="-39.282" y2="-212.852" width="0" layer="19" extent="1-1"/>
+<wire x1="-91.186" y1="-311.658" x2="-39.282" y2="-212.852" width="0" layer="19" extent="1-1"/>
+</signal>
+<signal name="BRAKE_2_PRE">
+<contactref element="R99" pad="2"/>
+<contactref element="U24" pad="2"/>
+<contactref element="JP7" pad="2"/>
+<wire x1="-51.474" y1="-215.9" x2="-45.847" y2="-203.7715" width="0" layer="19" extent="1-1"/>
+<wire x1="-91.186" y1="-315.976" x2="-51.474" y2="-215.9" width="0" layer="19" extent="1-1"/>
+</signal>
 </signals>

Commit message: fixed BSPD. removed 2 transceivers. routing.
Parts:
- removed C100, C102, C103, C104, C85: CAPACITOR_0603_10V_0.1UF, HyTechDevices:0603-CAP
- removed D10, D11, D12, D13, D14, D15, D9: LED_0603_RED, HyTechDevices:0603-LED
- removed D29, D30, D31, D32, D33, D40, D42, D43, D44, D8: SCHOTTKY_SOD323_30V, HyTechDevices:SOD-323
- removed R101, R94: RESISTOR_0603_13K, HyTechDevices:0603-RES
- removed R102, R96: RESISTOR_0603_3.3K, HyTechDevices:0603-RES
- removed R17, R19, R21, R35, R44, R46, R48, R50, R52: RESISTOR_0603_10K, HyTechDevices:0603-RES
- removed R18, R20, R22, R36, R45, R47, R49, R51, R53: RESISTOR_0603_1.33K, HyTechDevices:0603-RES
- removed R56, R73: RESISTOR_0603_2K, HyTechDevices:0603-RES
- removed R68, R76, R78: RESISTOR_0603_1.13K, HyTechDevices:0603-RES
- removed R69, R77, R79: RESISTOR_0603_10.2K, HyTechDevices:0603-RES
- removed U33, U45, U46: TCAN1051HQV-Q1, HyTechDevices:SOIC-08(NARROW,0.15")
- added C78, C79: CAPACITOR_0603_10V_0.1UF, HyTechDevices:0603-CAP
- added D16, D17, D18, D19, D20, D21, D22, D23, D26, D27: TVS_28VDO-214AA, HyTechDevices:DO-214AA
- added ESP, GPS, LTE, MQTT, RTK: LED_0603_RED, HyTechDevices:0603-LED
- added R129, R131, R133, R135, R137, R139, R141, R143, R145, R147: RESISTOR_0603_4.64K, HyTechDevices:0603-RES
- added R130, R132, R134, R136, R138, R14, R140, R142, R144, R146: RESISTOR_0603_36.5K, HyTechDevices:0603-RES
- added U26: TCAN1051HQV-Q1, HyTechDevices:SOIC-08(NARROW,0.15")
- added U27: OPAMP_1_CHANNEL_OPA991, HyTechDevices:SC-70-5
- added U28: LOGICGATE_OR, HyTechDevices:SC-70-5
- A2: value TEENSY_4.1 -> TEENSY_4.1_SMT; device HyTechDevices:TEENSY_LONG_EXT -> HyTechDevices:TEENSY_LONG_SSM
- D41: value SCHOTTKY_SOD323_30V -> TVS_28VDO-214AA; device HyTechDevices:SOD-323 -> HyTechDevices:DO-214AA
- J1, J3: value CONNECTOR-40__ -> CONNECTOR-34__; device HyTechDevices:EHT-120-01 -> HyTechDevices:EHT-117-01
- JP1, JP2: value JUMPER__1X02 -> JUMPER_0603_; device HyTechDevices:1X02 -> HyTechDevices:0603-RES
- K1, K10, K11, K12, K9: value RELAY_DPDT_RT424024 -> RELAY_DPDT_07DSMT; device HyTechDevices:RT*2* -> HyTechDevices:IM*G
- R10: value RESISTOR_0603_10K -> RESISTOR_0603_1.13K
- R11: value RESISTOR_0603_1.33K -> RESISTOR_0603_10.2K
- R15: value RESISTOR_0603_10K -> RESISTOR_0603_36.5K
- R16: value RESISTOR_0603_1.33K -> RESISTOR_0603_4.64K
- moved JP4 410.1 mm to (3.30, 95.8), turned to 270 degrees
- moved JP5 408.1 mm to (3.30, 89.4), turned to 270 degrees
- moved JP6 406.2 mm to (3.30, 83.1), turned to 270 degrees
- moved JP7 404.2 mm to (3.30, 76.7), turned to 270 degrees
- moved R123 400.7 mm to (24.1, 96.5), flipped to the bottom, turned to 180 degrees
- moved R124 399.4 mm to (21.1, 96.5), flipped to the bottom, turned to 180 degrees
- moved R127 398.5 mm to (24.1, 91.9), flipped to the bottom, turned to 180 degrees
- moved R126 398.3 mm to (27.2, 90.4), flipped to the bottom
- moved R121 397.6 mm to (27.2, 96.5), flipped to the bottom
- moved R128 397.3 mm to (21.1, 91.9), flipped to the bottom, turned to 180 degrees
- moved R119 395.5 mm to (24.1, 101.1), flipped to the bottom, turned to 180 degrees
- moved R122 395.5 mm to (27.2, 95.0), flipped to the bottom
- moved R125 395.5 mm to (27.2, 91.9), flipped to the bottom
- moved R118 395.3 mm to (27.2, 99.6), flipped to the bottom
- moved R120 394.3 mm to (21.1, 101.1), flipped to the bottom, turned to 180 degrees
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Connections:
- net CURRENT_OOR renamed OOR_HI
- net REFERENCE_OOR renamed OOR_LO
- removed net CAN_TCU_RX1: A3.D22, U33.4
- removed net CAN_TCU_RX2: A3.D0, U45.4
- removed net N$10: D41.C, R15.2
- removed net N$11: D42.C, R17.2
- removed net N$12: D43.C, R19.2
- removed net N$14: D44.C, R21.2
- removed net N$27: D8.C, R35.2
- removed net N$3: D40.C, R10.2
- removed net N$31: D9.2, R56.2
- removed net N$33: R62.2, R63.1, U39.1
- removed net N$34: R74.1, R75.2, U8.3
- removed net N$39: D15.2, R73.2
- removed net N$46: R76.2, R77.1, U9.1
- removed net N$48: R78.1, R79.2, U10.3
- removed net N$58: D29.C, R44.2
- removed net N$59: D30.C, R46.2
- removed net N$60: D31.C, R48.2
- removed net N$61: D32.C, R50.2
- removed net N$62: D33.C, R52.2
- removed net N$76: R68.1, R69.2, U43.3
- removed net N$87: R101.2, R102.2, R103.2
- removed net N$90: R94.2, R96.2, R98.2
- new net 0V5: R62.2, R63.1, U27.1, U39.1, U9.1
- new net 4V5: R74.1, R75.2, U10.3, U8.3
- new net 4V5_1: R10.1, R11.2, U43.3
- new net BRAKE_OOR_HI: TP6.1, U28.2, U43.4
- new net BRAKE_OOR_LO: TP5.1, U27.4, U28.1
- net !STEERING_2_CS: no longer J3.12
- net +24V: no longer J3.40
- net +3V3: now also C79.1, U26.5; no longer C102.1, C104.1, C85.1, U33.5, U45.5, U46.5
- net +5V: now also C78.1, R10.2, U26.3, U27.5, U28.5; no longer C100.1, C103.1, J3.38, R68.2, R77.2, R78.2, U33.3, U45.3, U46.3
- net 3.3V: now also A2.3.3V, A2.3.3V@1; no longer A2.3V3, A2.3V3@2, A2.3V3@3
- net ACCEL_1: now also U23.4; no longer U7.6
- net ACCEL_1_EXT: now also J1.1; no longer J1.29
- net ACCEL_2: now also U23.5; no longer U7.7
- net ACCEL_2_EXT: now also J1.2; no longer J1.30
- net BMS_OK: now also J3.31, K10.1; no longer J3.34, K10.A1
- net BRAKELIGHT_EN: no longer J3.9
- net BRAKE_1: now also U23.6, U27.3; no longer U7.8
- net BRAKE_1_EXT: now also J1.3; no longer J1.27
- net BRAKE_2: now also U23.7; no longer U7.11
- net BRAKE_2_EXT: now also J1.4; no longer J1.28
- net BRAKE_MISSING: now also U28.4; no longer TP6.1, U43.4
- net BRAKE_PRESSURE_F: now also U6.10; no longer U6.4
- net BRAKE_PRESSURE_F_EXT: now also J1.18, R98.2; no longer J1.23, R94.1
- net BRAKE_PRESSURE_R: now also U6.9; no longer U6.5
- net BRAKE_PRESSURE_R_EXT: now also J1.19, R103.2; no longer J1.24, R101.1
- net BSPD_OK: now also K11.1; no longer K11.A1
- net CANH_1: now also J1.27; no longer J1.12, U33.7
- net CANH_2: now also J1.31; no longer J1.8, U45.7
- net CANH_3: now also J1.21, U26.7; no longer J1.4, U46.7
- net CANL_1: now also J1.25; no longer J1.10, U33.6
- net CANL_2: now also J1.29; no longer J1.6, U45.6
- net CANL_3: now also J1.23, U26.6; no longer J1.2, U46.6
- net CAN_ECU_RX1: now also A3.D22
- net CAN_ECU_RX2: now also A3.D0
- net CAN_TCU_RX3: now also U26.4; no longer U46.4
- net CAN_TCU_TX1: no longer U33.1
- net CAN_TCU_TX2: no longer U45.1
- net CAN_TCU_TX3: now also U26.1; no longer U46.1
- net CURRENT: now also U23.9; no longer U6.6
- net CURRENT_EXT: now also J1.6; no longer J1.19
- net CURRENT_HIGH: no longer TP5.1
- net CURRENT_OOR_LO: now also U13.1; no longer U11.2
- net ECU_CLK: no longer J3.13
- net ECU_SDI: no longer J3.14
- net ECU_SDO: no longer J3.15
- net FL_INTERLOCK_SENSE: now also R130.1, R131.2; no longer R44.1, R45.2
- net FL_INTERLOCK_SENSE_EXT: now also D17.2, J3.3, R130.2; no longer D29.A, J3.30
- net FR_INTERLOCK_SENSE: now also R132.1, R133.2; no longer R10.1, R11.2
- net FR_INTERLOCK_SENSE_EXT: now also D18.2, J3.4, R132.2; no longer D40.A, J3.28
- net GND: now also A2.GND@1, C78.2, C79.2, D16.1, D17.1, D18.1, D19.1, D20.1, D21.1, D22.1, D23.1, D26.1, D27.1, D41.1, ESP.1, GPS.1, K1.4, K10.4, K11.4, K12.4, K9.4, LTE.1, MQTT.1, R129.1, R131.1, R133.1, R135.1, R137.1, R139.1, R141.1, R143.1, R145.1, R147.1, RTK.1, U26.2, U27.2, U28.3; no longer A2.GND@2, C100.2, C102.2, C103.2, C104.2, C85.2, D10.1, D11.1, D12.1, D13.1, D14.1, D15.1, D9.1, J1.1, J1.11, J1.13, J1.14, J1.17, J1.18, J1.21, J1.22, J1.3, J1.5, J1.7, J1.9, J3.16, J3.17, J3.26, J3.27, J3.3, J3.35, J3.36, J3.37, J3.39, J3.4, J3.7, J3.8, K1.14, K10.14, K11.14, K12.14, K9.14, R102.1, R18.1, R20.1, R22.1, R36.1, R45.1, R47.1, R49.1, R51.1, R53.1, R69.1, R76.1, R79.1, R96.1, U33.2, U45.2, U46.2
- net INERTIA_SENSE: now also R146.1, R147.2; no longer R21.1, R22.2
- net INERTIA_SENSE_EXT: now also D27.2, J3.7, R146.2; no longer D44.A, J3.31
- net INVERTER_24V_EN: no longer J3.10
- net INVERTER_EN: no longer J3.11
- net LATCH_BTN: no longer J3.5, J3.6
- net LOAD_FL: now also U7.8; no longer U23.4
- net LOAD_FL_EXT: now also J1.13; no longer J1.39
- net LOAD_FR: now also U7.9; no longer U23.5
- net LOAD_FR_EXT: now also J1.14; no longer J1.40
- net LOAD_RL: now also U18.5, U23.11; no longer U23.6
- net LOAD_RL_EXT: now also J1.8; no longer J1.37
- net LOAD_RR: now also U7.7; no longer U18.5, U23.7
- net LOAD_RR_EXT: now also J1.12; no longer J1.38
- net N$21: now also K9.3, K9.8; no longer K9.11, K9.A2
- net N$22: now also K11.3, K11.8; no longer K11.11, K11.A2
- net N$23: now also K10.3, K10.8; no longer K10.11, K10.A2
- net N$24: now also K1.3, K1.8; no longer K1.11, K1.A2
- net N$25: now also K12.3, K12.8; no longer K12.11, K12.A2
- net N$32: now also ESP.2; no longer D10.2
- net N$35: now also LTE.2; no longer D11.2
- net N$36: now also MQTT.2; no longer D12.2
- net N$37: now also GPS.2; no longer D13.2
- net N$38: now also RTK.2; no longer D14.2
- net NRF_LTE_OK: no longer R56.1, R73.1
- net OKHS_IN: now also J3.32, K9.1; no longer J3.33, K9.A1
- net REFERENCE: now also U23.10; no longer U6.7
- net REFERENCE_EXT: now also J1.7; no longer J1.20
- net REFERENCE_OOR_HI: now also U11.2; no longer U13.1
- net RL_INTERLOCK_SENSE_EXT: now also D41.2, J3.5, R15.2; no longer D41.A, J3.32
- net RR_INTERLOCK_SENSE: now also R129.2, R14.1; no longer R17.1, R18.2
- net RR_INTERLOCK_SENSE_EXT: now also D16.2, J3.6, R14.2; no longer D42.A, J3.29
- net SHDN_B: now also D19.2, J3.33, J3.34, K1.1, K9.6, R134.2; no longer D30.A, J1.15, J1.16, K1.A1, K9.21
- net SHDN_B_READ: now also R134.1, R135.2; no longer R46.1, R47.2
- net SHDN_C: now also D20.2, K10.6, K9.5, R136.2; no longer D31.A, K10.21, K9.24
- net SHDN_C_READ: now also R136.1, R137.2; no longer R48.1, R49.2
- net SHDN_D: now also D21.2, K10.5, K11.6, R138.2; no longer D32.A, K10.24, K11.21
- net SHDN_D_READ: now also R138.1, R139.2; no longer R50.1, R51.2
- net SHDN_E: now also D22.2, K11.5, K12.6, R140.2; no longer D33.A, K11.24, K12.21
- net SHDN_E_READ: now also R140.1, R141.2; no longer R52.1, R53.2
- net SHDN_F: now also D23.2, K1.6, K12.5, R142.2; no longer D43.A, K1.21, K12.24
- net SHDN_F_READ: now also R142.1, R143.2; no longer R19.1, R20.2
- net SHDN_G: now also D26.2, K1.5, R144.2; no longer D8.A, K1.24
- net SHDN_G_READ: now also R144.1, R145.2; no longer R35.1, R36.2
- net SPN_POT_1: now also U7.10; no longer U23.8
- net SPN_POT_1_EXT: now also J1.15; no longer J1.35
- net SPN_POT_2: now also U7.11; no longer U23.11
- net SPN_POT_2_EXT: now also J1.16; no longer J1.36
- net SPN_POT_3: now also U6.11; no longer U23.10
- net SPN_POT_3_EXT: now also J1.17; no longer J1.33
- net SPN_POT_4: now also U7.4; no longer U23.9
- net SPN_POT_4_EXT: now also J1.9; no longer J1.34
- net SPN_POT_5: now also U7.5; no longer U7.4
- net SPN_POT_5_EXT: now also J1.10; no longer J1.31
- net SPN_POT_6: now also U7.6; no longer U7.5
- net SPN_POT_6_EXT: now also J1.11; no longer J1.32
- net STEERING_1: now also U23.8; no longer U7.10
- net STEERING_1_EXT: now also J1.5; no longer J1.25
- net TCU_RX4: no longer J3.21
- net TCU_RX5: no longer J3.18
- net TCU_RX6: no longer J3.23
- net TCU_RX7: no longer J3.24
- net TCU_TX4: no longer J3.20
- net TCU_TX5: no longer J3.19
- net TCU_TX6: no longer J3.22
- net TCU_TX7: no longer J3.25
- net VBAT: no longer A2.VBAT
- net WATCHDOG_OK: now also K12.1; no longer K12.A1
Routing:
- net +3V3: track 222.1 -> 22.3 mm, vias 6 -> 0
- net +24V: track 190.3 -> 17.0 mm, vias 5 -> 0
- net SHDN_B: track 173.6 -> 20.6 mm, vias 8 -> 0
- net BMS_OK: track 135.3 -> 3.32 mm, vias 2 -> 0
- net TCU_RX5: track 119.3 -> 0.00 mm
- net TCU_TX5: track 118.2 -> 0.00 mm
- net OKHS_IN: track 126.4 -> 11.1 mm, vias 1 -> 0
- net TCU_TX4: track 111.2 -> 0.00 mm
- net TCU_RX4: track 110.9 -> 0.00 mm
- net TCU_TX7: track 104.1 -> 0.00 mm
- net TCU_RX7: track 100.4 -> 0.00 mm
- net TCU_RX6: track 96.5 -> 0.00 mm
- net TCU_TX6: track 93.8 -> 0.00 mm
- net ECU_CLK: track 136.0 -> 44.8 mm, vias 4 -> 2
- net ECU_SDI: track 131.8 -> 45.2 mm, vias 5 -> 2
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Other:
- board size 127 x 152.4 mm -> 109.2 x 115.6 mm
- board text added: "U23"

Commit message: routing progress
Parts:
- added U$3: (no value), HyTechManufacturing:LOGO_HYTECH_MEDIUM
- U$5: device HyTechManufacturing:LOGO_HYTECH_LARGE -> HyTechManufacturing:LOGO_GT_SMALL
- moved U$5 142.8 mm to (78.0, 5.33)
- moved TP2 137.6 mm to (54.4, 121.4)
- moved C26 135.5 mm to (37.1, 97.3), turned to 135 degrees
- moved C2 130.5 mm to (45.2, 98.3), flipped to the bottom
- moved A1 128.2 mm to (48.0, 100.8), turned to 270 degrees
- moved D3 125.3 mm to (34.8, 105.4)
- moved C1 124.8 mm to (45.0, 103.4), flipped to the bottom, turned to 0 degrees
- moved D1 116.0 mm to (36.8, 105.4), flipped to the top
- moved D2 116.0 mm to (40.9, 105.4), flipped to the top
- moved SWOK 83.6 mm to (59.9, 81.8), turned to 180 degrees
- moved R34 81.0 mm to (59.9, 83.8), turned to 180 degrees
- moved C8 73.7 mm to (105.7, 61.7), turned to 180 degrees
- moved WDOG 73.7 mm to (69.1, 81.8), turned to 180 degrees
- moved R32 71.1 mm to (69.1, 83.8), turned to 180 degrees
- moved C10 70.4 mm to (105.7, 60.2)
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Connections:
- net !AD1_CS: now also A2.D33; no longer A2.D41
- net !AD2_CS: now also A2.D29; no longer A2.D40
- net !AD3_CS: now also A2.D34; no longer A2.D39
- net !IMU_CS: now also A2.D38; no longer A2.D3
- net !IMU_RESET: now also A2.D36; no longer A2.D2
- net !STEERING_2_CS: now also A2.D10, J3.15; no longer A2.D9
- net +24V: now also J1.34
- net +5V: now also J1.33
- net BRAKELIGHT_EN: now also A2.D7, J3.21; no longer A2.D6
- net ECU_CLK: now also J3.13
- net ECU_SDI: now also J3.9
- net ECU_SDO: now also J3.11
- net FL_INTERLOCK_SENSE: now also A2.D39; no longer A2.D25
- net FR_INTERLOCK_SENSE: now also A2.D40; no longer A2.D24
- net GND: now also J1.20, J1.22, J1.24, J1.26, J1.28, J1.30, J1.32
- net IMU_DATAREADY: now also A2.D35; no longer A2.D5
- net IMU_SYNC: now also A2.D37; no longer A2.D4
- net INERTIA_SENSE: now also A2.D20; no longer A2.D28
- net INVERTER_24V_EN: now also A2.D8, J3.19; no longer A2.D7
- net INVERTER_EN: now also A2.D9, J3.17; no longer A2.D8
- net RL_INTERLOCK_SENSE: now also A2.D14; no longer A2.D27
- net RR_INTERLOCK_SENSE: now also A2.D16; no longer A2.D26
- net SHDN_B_READ: now also A2.D3; no longer A2.D33
- net SHDN_C_READ: now also A2.D4; no longer A2.D34
- net SHDN_D_READ: now also A2.D5; no longer A2.D35
- net SHDN_E_READ: now also A2.D6; no longer A2.D36
- net SHDN_F_READ: now also A2.D25; no longer A2.D18, A2.D29
- net SHDN_G_READ: now also A2.D26; no longer A2.D19, A2.D32
- net SOFTWARE_OK: now also A2.D28; no longer A2.D20
- net WATCHDOG: now also A2.D32; no longer A2.D21
Routing:
- net ECU_CLK: track 44.8 -> 235.2 mm, vias 2 -> 10
- net ECU_SDO: track 45.7 -> 210.2 mm, vias 2 -> 11
- net ECU_SDI: track 45.2 -> 196.0 mm, vias 2 -> 9
- net !IMU_CS: track 0.00 -> 69.3 mm, vias 0 -> 2
- net IMU_SYNC: track 0.00 -> 66.7 mm, vias 0 -> 2
- net IMU_DATAREADY: track 0.00 -> 65.2 mm, vias 0 -> 2
- net !IMU_RESET: track 0.00 -> 63.7 mm, vias 0 -> 2
- net RR_INTERLOCK_SENSE_EXT: track 0.00 -> 56.5 mm, vias 0 -> 1
- net INERTIA_SENSE_EXT: track 0.00 -> 54.7 mm, vias 0 -> 1
- net FL_INTERLOCK_SENSE_EXT: track 0.00 -> 52.4 mm, vias 0 -> 1
- net FR_INTERLOCK_SENSE_EXT: track 0.00 -> 49.7 mm, vias 0 -> 1
- net RL_INTERLOCK_SENSE_EXT: track 0.00 -> 48.6 mm, vias 0 -> 1
- net !STEERING_2_CS: track 0.00 -> 42.0 mm, vias 0 -> 1
- net !AD3_CS: track 0.00 -> 41.2 mm, vias 0 -> 2
- net INVERTER_24V_EN: track 0.00 -> 39.5 mm, vias 0 -> 1
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