File: EAGLE Board Designs/Main ECU/MainECU rev15.sch (EAGLE design)
At the start: 338 parts, among them J1 CONNECTOR-24_CONNECTOR-24_, J2 CONNECTOR-24_CONNECTOR-24_, K1 RELAY_DPDT_07DSMT, K2 RELAY_DPDT_07DSMT, K3 RELAY_DPDT_07DSMT, K4 RELAY_DPDT_07DSMT, K5 RELAY_DPDT_07DSMT, Q1 TRANSISTOR_N_MOS__DMG3406L-7, Q2 TRANSISTOR_P_MOS_SOT-23_DMP30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, Q3 TRANSISTOR_P_MOS_SOT-23_DMP30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, Q4 TRANSISTOR_N_MOS__DMG3406L-7, T1 TRANSFORMER_HM2112ZNLT, U1 VOLTAGE_REGULATOR_SOT-223_3.3V, U10 LOGICGATE_OR, U11 LOGICGATE_OR, U12 LOGICGATE_OR, U13 LOGICGATE_NOR, U14 TCAN1051HQV-Q1, U15 LOGICGATE_AND_DCK3, U16 MAX3074EESA+, U17 LTC1563, U18 LTC1563, U19 LTC1563, U2 LTC6820, U20 LTC1563, U21 LTC1563, U22 LTC1563, U23 LTC1563, U24 OPAMP_2_CHANNEL_OPA_2991, U25 OPAMP_2_CHANNEL_OPA_2991, U26 OPAMP_2_CHANNEL_OPA_2991, U27 OPAMP_2_CHANNEL_OPA_2991, U28 LTC1563, U29 TCAN1051HQV-Q1, U3 LTC6820, U30 TCAN1051HQV-Q1, U31 ADM8316WBX30, U4 TCAN1051HQV-Q1, U5 LTC1563, U6 MCP3208, U7 OPAMP_1_CHANNEL_OPA991, U8 LOGICGATE_OR, U9 LOGICGATE_OR

Commit message: fixing stuff from brd review
Other:
- note added: "add decoupling"
- note added: "check the beta value"
- note removed: "wait a minute?"
- note removed: "wait a minute?, this is affecting impedance at high frequencies! so i added jumpers"
Changed lines of the file:
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@@
 <pinref part="J1" gate="G$1" pin="1"/>
 <wire x1="58.42" y1="167.64" x2="63.5" y2="167.64" width="0.1524" layer="91"/>
-<label x="63.5" y="167.64" size="1.27" layer="95" xref="yes"/>
+<label x="63.5" y="167.64" size="1.27" layer="95" font="vector" xref="yes"/>
 </segment>
 </net>
@@
 <wire x1="134.62" y1="101.6" x2="10.16" y2="101.6" width="0.1524" layer="97"/>
 <text x="12.7" y="99.06" size="1.778" layer="97" font="vector">CAN Termination Jumpers + TVS Protection</text>
-<text x="15.24" y="93.98" size="1.778" layer="97" font="vector">wait a minute?, this is affecting impedance at high frequencies! so i added jumpers</text>
-<text x="15.24" y="66.04" size="1.778" layer="97" font="vector">wait a minute?</text>
 </plain>
 <instances>
@@
 <wire x1="214.122" y1="172.466" x2="274.32" y2="172.466" width="0.1524" layer="97"/>
 <text x="261.62" y="205.74" size="1.27" layer="97" font="vector">remove this</text>
+<text x="68.58" y="66.04" size="1.778" layer="97">add decoupling</text>
 </plain>
 <instances>
@@
 .1103 gain</text>
 <text x="142.24" y="134.62" size="1.778" layer="97">Filter Stage</text>
+<text x="78.74" y="203.2" size="1.778" layer="97">check the beta value</text>
 </plain>
 <instances>
