File: EAGLE Board Designs/Main ECU/MainECU rev16.brd (EAGLE design)
At the start: 97.5 x 115.6 mm, 373 parts, among them J1 CONNECTOR-24_CONNECTOR-24_, J2 CONNECTOR-24_CONNECTOR-24_, K1 RELAY_DPDT_07DSMT, K2 RELAY_DPDT_07DSMT, K3 RELAY_DPDT_07DSMT, K4 RELAY_DPDT_07DSMT, K5 RELAY_DPDT_07DSMT, Q1 TRANSISTOR_N_MOS__DMG3406L-7, Q2 TRANSISTOR_P_MOS_SOT-23_DMP30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, Q3 TRANSISTOR_P_MOS_SOT-23_DMP30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, Q4 TRANSISTOR_N_MOS__DMG3406L-7, Q5 TRANSISTOR_P_MOS_SOT-23_DMP30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, U1 VOLTAGE_REGULATOR_SOT-223_3.3V, U10 LOGICGATE_OR, U11 LOGICGATE_OR, U12 LOGICGATE_OR, U13 LOGICGATE_NOR, U14 TCAN1051HQV-Q1, U15 LOGICGATE_AND_DCK3, U16 MAX3074EESA+, U17 MAX7400, U18 MAX7400, U19 OPAMP_2_CHANNEL_OPA_2991, U2 MCP3208, U20 OPAMP_2_CHANNEL_OPA_2991, U21 OPAMP_2_CHANNEL_OPA_2991, U22 OPAMP_2_CHANNEL_OPA_2991, U23 OPAMP_2_CHANNEL_OPA_2991, U24 OPAMP_2_CHANNEL_OPA_2991, U25 OPAMP_2_CHANNEL_OPA_2991, U26 OPAMP_2_CHANNEL_OPA_2991, U27 OPAMP_2_CHANNEL_OPA_2991, U28 OPAMP_1_CHANNEL_OPA991, U29 TCAN1051HQV-Q1, U3 OPAMP_1_CHANNEL_OPA991, U30 TCAN1051HQV-Q1, U31 ADM8316WBX30, U32 OPAMP_2_CHANNEL_OPA_2991, U33 OPAMP_1_CHANNEL_OPA991, U34 OPAMP_1_CHANNEL_OPA991, U35 OPAMP_1_CHANNEL_OPA991, U4 TCAN1051HQV-Q1, U5 OPAMP_1_CHANNEL_OPA991, U6 MCP3208, U7 OPAMP_1_CHANNEL_OPA991, U8 LOGICGATE_OR, U9 LOGICGATE_OR

Commit message: nice
Parts:
- removed C55, C66: CAPACITOR_0603_10V_0.1UF, HyTechDevices:0603-CAP
- removed U34, U35: OPAMP_1_CHANNEL_OPA991, HyTechDevices:SC-70-5
- U28, U33: value OPAMP_1_CHANNEL_OPA991 -> OPAMP_2_CHANNEL_OPA_2991; device HyTechDevices:SC-70-5 -> HyTechDevices:SOT-23-8
- moved R126 224.6 mm to (15.2, 95.5), flipped to the bottom, turned to 90 degrees
- moved C90 220.8 mm to (14.5, 97.8), flipped to the bottom
- moved R125 218.1 mm to (11.3, 92.6), flipped to the bottom
- moved C91 213.1 mm to (11.3, 90.9), flipped to the bottom, turned to 180 degrees
- moved R56 207.7 mm to (8.51, 97.8), flipped to the bottom, turned to 180 degrees
- moved R124 205.0 mm to (15.1, 84.8), flipped to the bottom, turned to 90 degrees
- moved C88 201.4 mm to (14.5, 87.2), flipped to the bottom
- moved R81 198.6 mm to (11.2, 82.0), flipped to the bottom
- moved R78 194.3 mm to (8.51, 87.2), flipped to the bottom, turned to 180 degrees
- moved C89 193.7 mm to (11.2, 80.5), flipped to the bottom, turned to 180 degrees
- moved R77 191.7 mm to (11.6, 87.2), flipped to the bottom, turned to 180 degrees
- moved R75 187.1 mm to (5.97, 95.5), flipped to the bottom, turned to 90 degrees
- moved R55 187.1 mm to (11.6, 97.8), flipped to the bottom
- moved R76 186.1 mm to (8.26, 94.6), flipped to the bottom, turned to 180 degrees
- moved R79 185.7 mm to (5.97, 85.0), flipped to the bottom, turned to 90 degrees
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Connections:
- net N$55 renamed FL_CORNER_PRE
- net REFERNECE_PRE1 renamed FR_CORNER_PRE
- removed net REFERNECE_PRE2: C87.1, R81.2, U28.3, U28.4
- new net FR_CORNER_STAGE1: C87.1, R81.2, U33.1, U33.2
- net +3V3: now also U28.8, U33.8; no longer C55.1, C66.1, U28.5, U33.5, U34.5, U35.5
- net FL_CORNER: now also U28.6, U28.7; no longer U35.3, U35.4
- net FR_CORNER: now also U33.6, U33.7; no longer U33.3, U33.4
- net GND: now also U28.4, U33.4; no longer C55.2, C66.2, U28.2, U33.2, U34.2, U35.2
- net N$101: now also U28.1, U28.2; no longer U34.3, U34.4
- net N$12: now also U28.3; no longer U34.1
- net N$59: now also U33.3; no longer U28.1
- net N$70: now also U33.5; no longer U33.1
- net N$76: now also U28.5; no longer U35.1
Routing:
- net SUS_POT_1_EXT: track 0.00 -> 44.0 mm, vias 0 -> 1
- net STEERING_1_EXT: track 0.00 -> 42.6 mm, vias 0 -> 1
- net SUS_POT_2_EXT: track 0.00 -> 37.1 mm, vias 0 -> 1
- net STEERING_2_EXT: track 0.00 -> 36.1 mm, vias 0 -> 1
- net +5V: track 503.2 -> 473.7 mm, vias 11 -> 7
- net FR_CORNER_EXT: track 0.00 -> 27.2 mm, vias 0 -> 1
- net CURRENT_EXT: track 0.00 -> 23.0 mm
- net CURRENT: track 106.5 -> 85.2 mm, vias 5 -> 4
- net N$103: track 0.00 -> 21.1 mm
- net N$105: track 0.00 -> 20.6 mm
- net FL_CORNER_EXT: track 0.00 -> 13.1 mm
- net ACCEL_2_EXT: track 0.00 -> 10.1 mm
- net REFERENCE_EXT: track 0.00 -> 9.14 mm
- net ACCEL_1_EXT: track 0.00 -> 9.11 mm
- net STEERING_1: track 9.07 -> 0.00 mm
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
Commit message: more nice
Connections:
- new net N$107: U2.2
- new net N$108: U2.3
- new net N$109: U2.4
- new net N$110: U2.5
- new net N$111: U2.6
- new net N$112: U2.7
- new net N$113: U2.8
- new net N$55: U2.1
- net 24V_SENSE_ECU: no longer U6.5
- net ACCEL_1: no longer U6.3
- net ACCEL_2: no longer U6.2
- net BRAKE_1: now also U6.4; no longer U6.6
- net BRAKE_2: now also U6.6; no longer U6.4
- net CURRENT: now also U6.3
- net CURRENT_3V3: no longer U6.7
- net REFERENCE: now also U6.5
- net REFERENCE_3V3: no longer U6.1
- net STEERING_1: no longer U6.8
- net STEERING_2: now also U6.1
- net SUS_POT_2: now also U6.2
- net THERM_FL: now also U6.7
- net THERM_FR: now also U6.8
Routing:
- net SUS_POT_1_EXT: track 44.0 -> 0.00 mm, vias 1 -> 0
- net STEERING_1_EXT: track 42.6 -> 0.00 mm, vias 1 -> 0
- net SUS_POT_2_EXT: track 37.1 -> 0.00 mm, vias 1 -> 0
- net STEERING_2_EXT: track 36.1 -> 0.00 mm, vias 1 -> 0
- net FR_CORNER_EXT: track 27.2 -> 0.00 mm, vias 1 -> 0
- net BRAKE_1: track 31.1 -> 35.0 mm
- net BRAKE_2: track 3.83 -> 0.00 mm
