File: EAGLE Board Designs/Dashboard/Dashboard rev6.brd (EAGLE design)
At the start: 14.1 x 15.5 mm, 80 parts, among them J1 JUMPER__1X02, J2 CONNECTOR-8_μF_S_RA_, J3 CONNECTOR-CAN_μF_S_RA_, J4 CONNECTOR-6_μF_S_RA_, J6 CONNECTOR-6_μF_S_RA_, U10 NEOPIXEL, U11 NEOPIXEL, U12 NEOPIXEL, U13 NEOPIXEL, U14 NEOPIXEL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

Commit message: Began placement
Parts:
- removed U17, U18: NEOPIXEL, HyTechDevices:NEOPIXEL
- added U1, U2: NEOPIXEL, HyTechDevices:NEOPIXEL
- moved R5 967.1 mm to (408.9, 490.2)
- moved R4 965.9 mm to (412.8, 490.2)
- moved R3 964.7 mm to (416.6, 490.2)
- moved D5 952.8 mm to (434.3, 475.0)
- moved R15 939.0 mm to (374.6, 490.2)
- moved R8 921.6 mm to (401.3, 490.2)
- moved R7 920.4 mm to (405.1, 490.2)
- moved C38 917.3 mm to (435.6, 490.2)
- moved R12 916.6 mm to (386.1, 490.2)
- moved R14 915.9 mm to (378.5, 490.2)
- moved C39 912.9 mm to (431.8, 490.2)
- moved J1 911.8 mm to (434.3, 486.4)
- moved D1 901.9 mm to (428.0, 490.2)
- moved D4 896.1 mm to (358.1, 462.3)
- moved D3 894.5 mm to (365.8, 462.3)
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Connections:
- removed net N$11: U18.2, U4.4
- removed net N$23 (its old number): U17.2, U18.4
- removed net N$4 (its old number): U12.2, U17.4
- new net N$5: U1.2, U2.4
- new net N$6: U2.2, U4.4
- new net N$8: U6.2, U7.4
- net +5V: now also U1.1, U2.1; no longer U17.1, U18.1
- net GND: now also U1.3, U2.3; no longer U17.3, U18.3
- net N$27: now also U12.2; no longer U6.2
- net NEOPIXEL_CTRL: now also U1.4; no longer U7.4
Other:
- board size 14.1 x 15.5 mm -> 247.6 x 47.3 mm

Commit message: More placements
Parts:
- removed XF2: FUSE_HOLDER_MINIBLADEPTH, HyTechDevices:3568
- added XF1: FUSE_HOLDER_MINIBLADESMD, HyTechDevices:3588
- moved J2 292.4 mm to (678.2, 448.3), turned to 180 degrees
- moved A3 287.0 mm to (646.4, 426.7)
- moved J4 276.9 mm to (640.1, 453.4), turned to 180 degrees
- moved A4 228.0 mm to (659.1, 447.0)
- moved A2 204.5 mm to (595.6, 444.5), turned to 180 degrees
- moved J6 120.8 mm to (548.6, 453.4), turned to 180 degrees
- moved D101 119.4 mm to (492.8, 435.6), flipped to the bottom
- moved U9 111.0 mm to (675.6, 442.0)
- moved J3 104.1 mm to (514.4, 448.3), turned to 180 degrees
- moved U7 93.3 mm to (694.7, 428.0)
- moved U8 93.3 mm to (675.6, 428.0)
- moved LS100 88.2 mm to (506.7, 389.9), flipped to the bottom
- moved U6 70.6 mm to (694.7, 442.0)
- moved U12 36.4 mm to (562.6, 457.2)
- moved U10 17.7 mm to (627.4, 455.9)
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Connections:
- net +24V: now also XF1.3, XF1.4; no longer XF2.3, XF2.4
- net 24VIN: now also XF1.1, XF1.2; no longer XF2.1, XF2.2
Other:
- board text added: "AMS"

Commit message: Added layers
Routing:
- added copper zone on layer 15, net +5V
- added copper zone on layer 2, net GND

Commit message: Approx placements done
Parts:
- removed J1: JUMPER__1X02, HyTechDevices:1X02
- removed RN3: RESISTOR_NETWORK_4_1K, HyTechDevices:1206-RES-ARRAY
- removed TP1_24V: TEST_POINT, HyTechDevices:5015
- added JP1: JUMPER_0603_, HyTechDevices:0603-RES
- added R6: RESISTOR_0603_1K, HyTechDevices:0603-RES
- added TP_24V: TEST_POINT, HyTechDevices:5015
- moved TP_BRB 333.2 mm to (694.7, 428.0)
- moved TP_BOTS 319.7 mm to (694.7, 434.3)
- moved D3 317.8 mm to (682.0, 430.5), turned to 180 degrees
- moved D4 317.8 mm to (674.4, 430.5), turned to 180 degrees
- moved R15 317.6 mm to (682.0, 410.2)
- moved TP_INERTIA 314.5 mm to (694.7, 440.7)
- moved TP_SSOK 311.8 mm to (694.7, 447.0)
- moved D2 311.0 mm to (682.0, 424.2), turned to 180 degrees
- moved R14 310.3 mm to (676.9, 405.1)
- moved R12 306.7 mm to (680.7, 405.1)
- moved C33 304.6 mm to (654.0, 424.2)
- moved R7 295.7 mm to (688.3, 405.1)
- moved R8 295.7 mm to (684.5, 405.1)
- moved R3 289.4 mm to (694.7, 410.2)
- moved R5 289.4 mm to (687.1, 410.2)
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Connections:
- net N$13 renamed A
- net N$14 renamed B
- net N$15 renamed C
- net N$17 renamed F
- net N$19 renamed D
- net N$2 renamed TEENSY_ON
- net N$25 renamed CRX
- net N$28 renamed HORNS
- net N$29 renamed CTX
- net N$39 renamed HORNB
- net N$50 renamed FEED
- removed net N$16: D101.10, RN4.6
- removed net N$18: D101.1, RN4.8
- removed net N$24: J1.2, R36.2
- new net E: D101.1, RN4.6
- new net G: D101.10, RN4.8
- new net N$10: JP1.2, R36.2
- net +24V: now also TP_24V.1; no longer TP1_24V.1
- net CANH: now also JP1.1; no longer J1.1
- net E2: now also RN4.3; no longer RN4.1
- net G2: now also RN4.1; no longer RN4.3
- net GND: now also R6.1; no longer RN3.3
- net N$3: now also R6.2; no longer RN3.6
Other:
- board text added: "+24V"
- board text added: "SHUTDOWN_I"

Commit message: Continued routing
Parts:
- moved LS100 130.7 mm to (602.0, 438.1), turned to 270 degrees
- moved R1 27.4 mm to (622.4, 426.2)
- moved R2 23.6 mm to (622.3, 439.0)
- moved 3.3V 22.5 mm to (623.6, 429.3), turned to 90 degrees
- moved R15 19.8 mm to (666.8, 422.9), turned to 180 degrees
- moved 5V 17.8 mm to (623.6, 435.6), turned to 90 degrees
- moved 24V 16.3 mm to (623.6, 448.3), turned to 90 degrees
- moved 12V 15.3 mm to (623.6, 442.0), turned to 90 degrees
- moved R83 14.9 mm to (622.4, 445.1)
- moved R10 14.0 mm to (622.3, 432.6)
- moved C33 13.5 mm to (643.9, 433.1), turned to 90 degrees
- moved C24 6.35 mm to (650.2, 433.1), turned to 90 degrees
- moved C10 4.02 mm to (574.0, 431.8), turned to 270 degrees
- moved C12 3.59 mm to (494.0, 440.7), turned to 270 degrees
- moved C16 3.59 mm to (491.5, 440.7), turned to 270 degrees
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Connections:
- net A: now also RN2.5; no longer RN2.8
- net A2: now also RN2.4; no longer RN2.1
- net B: now also RN2.6; no longer RN2.7
- net B2: now also RN2.3; no longer RN2.2
- net C: now also RN2.7; no longer RN2.6
- net C2: now also RN2.2; no longer RN2.3
- net D: now also RN2.8; no longer RN2.5
- net D2: now also RN2.1; no longer RN2.4
Routing:
- net GND: track 0.00 -> 47.6 mm, vias 0 -> 20
- net BOTS: track 0.00 -> 39.6 mm
- net +24V: track 0.00 -> 30.0 mm
- net +5V: track 0.00 -> 25.4 mm, vias 0 -> 3
- net BRB: track 0.00 -> 20.4 mm
- net SSOK: track 0.00 -> 15.0 mm
- net +12V: track 0.00 -> 13.0 mm
- net INERTIA: track 0.00 -> 9.06 mm
- net 24VIN: track 0.00 -> 6.07 mm
- net G2: track 0.00 -> 4.00 mm
- net +3V3: track 0.00 -> 3.99 mm
- net F2: track 0.00 -> 3.93 mm
- net E2: track 0.00 -> 3.87 mm
- net A2: track 0.00 -> 3.73 mm
- net B2: track 0.00 -> 3.66 mm
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Other:
- board text added: "IMD"
- board text added: "MCU"

Commit message: RIght side routing
Parts:
- moved R7 36.3 mm to (659.1, 426.7), turned to 180 degrees
- moved R12 36.3 mm to (659.1, 434.3), turned to 180 degrees
- moved R4 36.0 mm to (664.2, 434.3), turned to 180 degrees
- moved R3 35.9 mm to (664.2, 429.3), turned to 180 degrees
- moved R8 35.0 mm to (659.1, 429.3), turned to 180 degrees
- moved R14 32.1 mm to (659.1, 431.8), turned to 180 degrees
- moved R5 31.4 mm to (664.2, 431.8), turned to 180 degrees
- moved D6 29.2 mm to (636.3, 430.5)
- moved TP_SSOK 19.7 mm to (699.8, 428.0)
- moved TP_BOTS 13.7 mm to (699.8, 447.0)
- moved TP_BRB 13.7 mm to (699.8, 440.7)
- moved TP_INERTIA 8.13 mm to (699.8, 434.3)
- moved D2 6.84 mm to (688.3, 426.7), turned to 90 degrees
- moved D4 6.35 mm to (669.3, 426.7), turned to 90 degrees
- moved R6 5.24 mm to (607.1, 458.5)
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Routing:
- net 24VIN: track 6.07 -> 119.6 mm
- net C: track 0.00 -> 85.8 mm, vias 0 -> 1
- net G: track 0.00 -> 85.3 mm, vias 0 -> 1
- net B: track 0.00 -> 84.1 mm, vias 0 -> 1
- net A: track 0.00 -> 81.6 mm, vias 0 -> 1
- net D: track 0.00 -> 80.9 mm, vias 0 -> 1
- net E: track 0.00 -> 76.9 mm, vias 0 -> 1
- net F: track 0.00 -> 76.9 mm, vias 0 -> 1
- net BRB_READ: track 0.00 -> 69.9 mm, vias 0 -> 2
- net BOTS_READ: track 0.00 -> 66.4 mm, vias 0 -> 2
- net SSOK_READ: track 0.00 -> 66.4 mm, vias 0 -> 2
- net INERTIA_READ: track 0.00 -> 62.9 mm, vias 0 -> 2
- net INERTIA: track 9.06 -> 57.2 mm
- net BTN_MC_CYCLE_READ: track 0.00 -> 44.0 mm, vias 0 -> 2
- net BTN_DIM_READ: track 0.00 -> 41.4 mm, vias 0 -> 2
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
Commit message: Left side routing
Parts:
- moved R36 21.6 mm to (565.0, 452.1)
- moved R13 19.3 mm to (580.4, 442.0)
- moved R60 14.8 mm to (569.0, 454.7)
- moved R11 14.5 mm to (580.4, 445.8), turned to 180 degrees
- moved C25 6.48 mm to (565.1, 454.7)
- moved C38 3.81 mm to (576.6, 459.7), turned to 270 degrees
- moved C34 3.59 mm to (569.0, 457.2)
- moved C17 3.58 mm to (571.9, 450.2), turned to 180 degrees
- moved RN4 2.84 mm to (566.4, 434.3)
- moved RN2 2.84 mm to (566.4, 439.4)
- moved U27 2.84 mm to (575.3, 454.7)
- moved U3 2.84 mm to (574.0, 436.9)
- moved U5 2.84 mm to (574.0, 444.5)
- moved C10 2.84 mm to (571.5, 430.5)
- moved C11 2.84 mm to (569.0, 430.5)
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Routing:
- net CANL: track 0.00 -> 68.4 mm, vias 0 -> 2
- net CANH: track 0.00 -> 64.6 mm, vias 0 -> 2
- net N$54: track 0.00 -> 36.4 mm
- net +3V3: track 3.99 -> 39.6 mm
- net CLK: track 0.00 -> 29.7 mm
- net FEED: track 0.00 -> 22.6 mm
- net CIPO: track 0.00 -> 14.6 mm
- net +5V: track 28.6 -> 41.8 mm, vias 4 -> 5
- net BUZZER_CTRL: track 0.00 -> 12.9 mm
- net CS_CAN: track 0.00 -> 12.9 mm
- net GND: track 59.1 -> 70.1 mm, vias 23 -> 27
- net COPI: track 0.00 -> 9.01 mm
- net CTX: track 0.00 -> 8.36 mm
- net HORNS: track 0.00 -> 7.90 mm
- net N$21: track 0.00 -> 5.47 mm
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
Commit message: Continued changes
Parts:
- moved LS100 7.73 mm to (594.4, 436.9), turned to 180 degrees
- moved U15 5.24 mm to (626.1, 431.8)
- moved U11 4.22 mm to (626.1, 444.5)
- moved U14 2.54 mm to (562.6, 431.8), turned to 90 degrees
- moved U10 1.80 mm to (626.1, 457.2)
- moved R11 1.27 mm to (580.4, 447.0)
- moved U13 1.27 mm to (562.6, 444.5), turned to 90 degrees
- turned U1 to 90 degrees
- turned U12 to 90 degrees
- turned U2 to 90 degrees
- turned U4 to 90 degrees
Routing:
- net NEOPIXEL_CTRL: track 0.00 -> 82.0 mm, vias 0 -> 1
- net N$12: track 0.00 -> 67.9 mm
- net DIAL_MODE_1: track 0.00 -> 55.7 mm, vias 0 -> 2
- net +12V: track 13.0 -> 66.6 mm, vias 0 -> 2
- net DIAL_MODE_2: track 0.00 -> 52.1 mm, vias 0 -> 2
- net N$54: track 36.4 -> 12.3 mm
- net CRX: track 0.00 -> 11.4 mm
- net N$27: track 0.00 -> 9.33 mm
- net N$20: track 0.00 -> 9.33 mm
- net G: track 83.3 -> 74.5 mm
- net BTN_START_READ: track 39.3 -> 46.5 mm
- net N$6: track 0.00 -> 6.79 mm
- net BTN_MODE_READ: track 36.5 -> 42.8 mm
- net DIAL_AUTOCROSS: track 0.00 -> 5.59 mm, vias 0 -> 1
- net +5V: track 41.8 -> 45.8 mm, vias 5 -> 7
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