File: EAGLE Board Designs/Connector Board/Connector Board rev1.sch (EAGLE design)
At the start: 14 parts, among them J1 CONNECTOR-37__, J2 CONNECTOR-8_AMPHENOL_M12A_08P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, J3 CONNECTOR-8_AMPHENOL_M12A_08P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, J4 CONNECTOR-6_AS_PCT_, J5 CONNECTOR-13_SOURIAU_, J6 CONNECTOR-40__, J7 CONNECTOR-40__

Commit message: some definitions
Connections:
- new net !STEERING_2_CS: J7.12
- new net +24V: J1.14, J1.24, J1.33, J1.34, J7.40
- new net +5V: J7.38
- new net ACCEL_1_EXT: J6.29
- new net ACCEL_2_EXT: J6.30
- new net BMS_OK: J1.28, J7.34
- new net BRAKELIGHT_12V: J1.9
- new net BRAKELIGHT_EN: J7.9
- new net BRAKE_1_EXT: J6.27
- new net BRAKE_2_EXT: J6.28
- new net BRAKE_PRESSURE_F_EXT: J6.23
- new net BRAKE_PRESSURE_R_EXT: J6.24
- new net CANH_1: J1.15, J6.12
- new net CANH_2: J1.17, J6.8
- new net CANH_3: J1.1, J6.4
- new net CANL_1: J1.16, J6.10
- new net CANL_2: J1.18, J6.6
- new net CANL_3: J1.2, J6.2
- new net CURRENT_EXT: J1.3, J6.19
- new net ECU_CLK: J7.13
- new net ECU_SDI: J7.14
- new net ECU_SDO: J7.15
- new net FL_INTERLOCK_SENSE_EXT: J7.30
- new net FR_INTERLOCK_SENSE_EXT: J7.28
- new net GND: J1.10, J1.13, J1.32, J1.35, J1.37, J1.8, J6.1, J6.11, J6.13, J6.14, J6.17, J6.18, J6.21, J6.22, J6.26, J6.3, J6.5, J6.7, J6.9, J7.16, J7.17, J7.26, J7.27, J7.3, J7.35, J7.36, J7.37, J7.39, J7.4, J7.7, J7.8
- new net INERTIA_SENSE_EXT: J7.31
- new net INVERTER_24V_EN: J1.19, J7.10
- new net INVERTER_EN: J1.30, J7.11
- new net LATCH: J1.21
- new net LATCH_BTN: J7.5, J7.6
- new net LOAD_FL_EXT: J6.39
- new net LOAD_FR_EXT: J6.40
- new net LOAD_RL_EXT: J1.27, J6.37
- new net LOAD_RR_EXT: J1.23, J6.38
- new net N$1: J1.5
- new net N$4: J1.31
- new net N$5: J1.36
- new net OKHS_IN: J1.29, J7.33
- new net REFERENCE_EXT: J1.4, J6.20
- new net RL_INTERLOCK_SENSE_EXT: J7.32
- new net RR_INTERLOCK_SENSE_EXT: J7.29
- new net SHDN_B: J6.15, J6.16
- new net SHDN_G: J7.1, J7.2
- new net SHDN_I: J1.11
- new net SHDN_J: J1.12, J1.6
- new net SHDN_K: J1.7
- new net SHDN_M: J1.20
- new net SPN_POT_1_EXT: J6.35
- new net SPN_POT_2_EXT: J6.36
- new net SPN_POT_3_EXT: J6.33
- new net SPN_POT_4_EXT: J1.26, J6.34
- new net SPN_POT_5_EXT: J1.25, J6.31
- new net SPN_POT_6_EXT: J1.22, J6.32
- new net STEERING_1_EXT: J6.25
- new net TCU_RX5: J7.18
- new net TCU_RX6: J7.23
- new net TCU_RX7: J7.24
- new net TCU_TX4: J7.20
- new net TCU_TX5: J7.19
- new net TCU_TX6: J7.22
- new net TCU_TX7: J7.25
- new net TXU_RX4: J7.21
Other:
- note added: "Accumulator Current Sense"
- note added: "Brake Light"
- note added: "CAN Front"
- note added: "CAN Peripheral"
- note added: "CAN Rear"
- note added: "Digital Signals"
- note added: "Power"
- note added: "RL Corner"
- note added: "RR Corner"
- note added: "Suspension Potentiometers: 1,2 - FL 3 - FR 4,5 - RL 6 - RR"
- moved on the sheet: J1, J2, J3, J4, J6, J7, S1, S2, S3, S4, S5, S6

Commit message: schema progress
Connections:
- new net N$6: J3.4
- new net SHDN_H: J2.6, J3.5
- net +24V: now also J2.1, J3.1
- net GND: now also J2.7, J3.7
- net LOAD_FL_EXT: now also J2.2
- net LOAD_FR_EXT: now also J3.2
- net SHDN_G: now also J2.5
- net SHDN_I: now also J3.6
- net SPN_POT_1_EXT: now also J2.3
- net SPN_POT_2_EXT: now also J2.4
- net SPN_POT_3_EXT: now also J3.3
Other:
- moved on the sheet: J2, J3, J4
Changed lines of the file:
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@@
 <part name="P2" library="HyTechSupplies" deviceset="+5V" device=""/>
 <part name="P3" library="HyTechSupplies" deviceset="GND" device=""/>
+<part name="U$2" library="HyTechSupplies" deviceset="+24V" device=""/>
+<part name="P4" library="HyTechSupplies" deviceset="GND" device=""/>
+<part name="U$3" library="HyTechSupplies" deviceset="+24V" device=""/>
+<part name="P5" library="HyTechSupplies" deviceset="GND" device=""/>
 </parts>
 <sheets>
@@
 <attribute name="MPN" x="12.7" y="88.265" size="1.27" layer="96" align="top-left"/>
 </instance>
-<instance part="J2" gate="G$1" x="210.82" y="203.2" smashed="yes">
-<attribute name="NAME" x="210.82" y="203.962" size="1.27" layer="95"/>
-<attribute name="MPN" x="210.82" y="179.705" size="1.27" layer="96" align="top-left"/>
-</instance>
-<instance part="J3" gate="G$1" x="226.06" y="203.2" smashed="yes">
-<attribute name="NAME" x="226.06" y="203.962" size="1.27" layer="95"/>
-<attribute name="MPN" x="226.06" y="179.705" size="1.27" layer="96" align="top-left"/>
-</instance>
-<instance part="J4" gate="G$1" x="241.3" y="203.2" smashed="yes">
-<attribute name="NAME" x="241.3" y="203.962" size="1.27" layer="95"/>
-<attribute name="MPN" x="241.3" y="184.785" size="1.27" layer="96" align="top-left"/>
+<instance part="J2" gate="G$1" x="170.18" y="190.5" smashed="yes">
+<attribute name="NAME" x="170.18" y="191.262" size="1.27" layer="95"/>
+<attribute name="MPN" x="170.18" y="167.005" size="1.27" layer="96" align="top-left"/>
+</instance>
+<instance part="J3" gate="G$1" x="170.18" y="149.86" smashed="yes">
+<attribute name="NAME" x="170.18" y="150.622" size="1.27" layer="95"/>
+<attribute name="MPN" x="170.18" y="126.365" size="1.27" layer="96" align="top-left"/>
+</instance>
+<instance part="J4" gate="G$1" x="210.82" y="190.5" smashed="yes">
+<attribute name="NAME" x="210.82" y="191.262" size="1.27" layer="95"/>
+<attribute name="MPN" x="210.82" y="172.085" size="1.27" layer="96" align="top-left"/>
 </instance>
 <instance part="J5" gate="G$1" x="256.54" y="203.2" smashed="yes">
@@
 <instance part="P3" gate="1" x="165.1" y="81.28" smashed="yes">
 <attribute name="VALUE" x="165.1" y="80.01" size="1.27" layer="96" align="top-center"/>
+</instance>
+<instance part="U$2" gate="G$1" x="182.88" y="193.04" smashed="yes">
+<attribute name="VALUE" x="182.88" y="198.12" size="1.778" layer="96" align="bottom-center"/>
+</instance>
+<instance part="P4" gate="1" x="182.88" y="167.64" smashed="yes">
+<attribute name="VALUE" x="182.88" y="166.37" size="1.27" layer="96" align="top-center"/>
+</instance>
+<instance part="U$3" gate="G$1" x="182.88" y="152.4" smashed="yes">
+<attribute name="VALUE" x="182.88" y="157.48" size="1.778" layer="96" align="bottom-center"/>
+</instance>
+<instance part="P5" gate="1" x="182.88" y="127" smashed="yes">
+<attribute name="VALUE" x="182.88" y="125.73" size="1.27" layer="96" align="top-center"/>
 </instance>
 </instances>
@@
 <label x="83.82" y="106.68" size="1.27" layer="95" xref="yes"/>
 </segment>
+<segment>
+<pinref part="J3" gate="G$1" pin="3"/>
+<wire x1="180.34" y1="142.24" x2="187.96" y2="142.24" width="0.1524" layer="91"/>
+<label x="187.96" y="142.24" size="1.27" layer="95" xref="yes"/>
+</segment>
 </net>
 <net name="SPN_POT_4_EXT" class="0">
@@
 <label x="83.82" y="101.6" size="1.27" layer="95" xref="yes"/>
 </segment>
+<segment>
+<pinref part="J2" gate="G$1" pin="3"/>
+<wire x1="180.34" y1="182.88" x2="187.96" y2="182.88" width="0.1524" layer="91"/>
+<label x="187.96" y="182.88" size="1.27" layer="95" xref="yes"/>
+</segment>
 </net>
 <net name="SPN_POT_2_EXT" class="0">
@@
 <label x="83.82" y="99.06" size="1.27" layer="95" xref="yes"/>
 </segment>
+<segment>
+<pinref part="J2" gate="G$1" pin="4"/>
+<wire x1="180.34" y1="180.34" x2="187.96" y2="180.34" width="0.1524" layer="91"/>
+<label x="187.96" y="180.34" size="1.27" layer="95" xref="yes"/>
+</segment>
 </net>
 <net name="LOAD_RL_EXT" class="0">
@@
 <label x="83.82" y="91.44" size="1.27" layer="95" xref="yes"/>
 </segment>
+<segment>
+<pinref part="J2" gate="G$1" pin="2"/>
+<wire x1="180.34" y1="185.42" x2="187.96" y2="185.42" width="0.1524" layer="91"/>
+<label x="187.96" y="185.42" size="1.27" layer="95" xref="yes"/>
+</segment>
 </net>
 <net name="LOAD_FR_EXT" class="0">
@@
 <wire x1="76.2" y1="88.9" x2="83.82" y2="88.9" width="0.1524" layer="91"/>
 <label x="83.82" y="88.9" size="1.27" layer="95" xref="yes"/>
+</segment>
+<segment>
+<pinref part="J3" gate="G$1" pin="2"/>
+<wire x1="180.34" y1="144.78" x2="187.96" y2="144.78" width="0.1524" layer="91"/>
+<label x="187.96" y="144.78" size="1.27" layer="95" xref="yes"/>
 </segment>
 </net>
@@
 <label x="45.72" y="160.02" size="1.27" layer="95" xref="yes"/>
 </segment>
+<segment>
+<pinref part="J2" gate="G$1" pin="7"/>
+<pinref part="P4" gate="1" pin="GND"/>
+<wire x1="180.34" y1="172.72" x2="182.88" y2="172.72" width="0.1524" layer="91"/>
+<wire x1="182.88" y1="172.72" x2="182.88" y2="170.18" width="0.1524" layer="91"/>
+</segment>
+<segment>
+<pinref part="J3" gate="G$1" pin="7"/>
+<pinref part="P5" gate="1" pin="GND"/>
+<wire x1="180.34" y1="132.08" x2="182.88" y2="132.08" width="0.1524" layer="91"/>
+<wire x1="182.88" y1="132.08" x2="182.88" y2="129.54" width="0.1524" layer="91"/>
+</segment>
 </net>
 <net name="SHDN_G" class="0">
@@
 <label x="137.16" y="187.96" size="1.27" layer="95" xref="yes"/>
 </segment>
+<segment>
+<pinref part="J2" gate="G$1" pin="5"/>
+<wire x1="180.34" y1="177.8" x2="187.96" y2="177.8" width="0.1524" layer="91"/>
+<label x="187.96" y="177.8" size="1.27" layer="95" xref="yes"/>
+</segment>
 </net>
 <net name="LATCH_BTN" class="0">
@@
 <label x="43.18" y="124.46" size="1.27" layer="95" xref="yes"/>
 </segment>
+<segment>
+<pinref part="J2" gate="G$1" pin="1"/>
+<pinref part="U$2" gate="G$1" pin="+24V"/>
+<wire x1="180.34" y1="187.96" x2="182.88" y2="187.96" width="0.1524" layer="91"/>
+<wire x1="182.88" y1="187.96" x2="182.88" y2="190.5" width="0.1524" layer="91"/>
+</segment>
+<segment>
+<pinref part="J3" gate="G$1" pin="1"/>
+<pinref part="U$3" gate="G$1" pin="+24V"/>
+<wire x1="180.34" y1="147.32" x2="182.88" y2="147.32" width="0.1524" layer="91"/>
+<wire x1="182.88" y1="147.32" x2="182.88" y2="149.86" width="0.1524" layer="91"/>
+</segment>
 </net>
 <net name="SHDN_M" class="0">
@@
 <label x="38.1" y="157.48" size="1.27" layer="95" xref="yes"/>
 </segment>
+<segment>
+<pinref part="J3" gate="G$1" pin="6"/>
+<wire x1="180.34" y1="134.62" x2="187.96" y2="134.62" width="0.1524" layer="91"/>
+<label x="187.96" y="134.62" size="1.27" layer="95" xref="yes"/>
+</segment>
 </net>
 <net name="SHDN_J" class="0">
@@
 </segment>
 </net>
+<net name="SHDN_H" class="0">
+<segment>
+<pinref part="J2" gate="G$1" pin="6"/>
+<wire x1="180.34" y1="175.26" x2="187.96" y2="175.26" width="0.1524" layer="91"/>
+<label x="187.96" y="175.26" size="1.27" layer="95" xref="yes"/>
+</segment>
+<segment>
+<pinref part="J3" gate="G$1" pin="5"/>
+<wire x1="180.34" y1="137.16" x2="187.96" y2="137.16" width="0.1524" layer="91"/>
+<label x="187.96" y="137.16" size="1.27" layer="95" xref="yes"/>
+</segment>
+</net>
+<net name="N$6" class="0">
+<segment>
+<pinref part="J3" gate="G$1" pin="4"/>
+<wire x1="180.34" y1="139.7" x2="187.96" y2="139.7" width="0.1524" layer="91"/>
+</segment>
+</net>

Commit message: schematic progress
Parts:
- removed S1, S2, S3, S4, S5, S6: SWITCH_SPDT_CS12ANW03, HyTechDevices:SWITCH_SPDT_CS12ANW03
- added D1, D2, D3, D4, D5, D6: TVS_15V, HyTechDevices:TVS_15V
- added J10, J11: CONNECTOR-18_MF_T_V_, HyTechDevices:CONNECTOR-18_MF_T_V_
- added J12: CONNECTOR-10_MF_T_V_, HyTechDevices:CONNECTOR-10_MF_T_V_
- added J8, J9: CONNECTOR-4_μF_T_V_BLACK, HyTechDevices:CONNECTOR-4_μF_T_V_BLACK
- added JP1, JP2, JP3, JP4: JUMPER__1X02, HyTechDevices:JUMPER__1X02
- added Q1, Q3, Q5: TRANSISTOR_N_MOS__DMG3406L-7, HyTechDevices:TRANSISTOR_N_MOS__DMG3406L-7
- added Q2, Q4, Q6: TRANSISTOR_P_MOS_SOT-23_DMP3056L-7, HyTechDevices:TRANSISTOR_P_MOS_SOT-23_DMP3056L-7
- added R1, R13, R14, R15, R2, R3, R4: RESISTOR_0603_100K, HyTechDevices:RESISTOR_0603_100K
- added R10, R6, R7, R9: RESISTOR_0603_5.1K, HyTechDevices:RESISTOR_0603_5.1K
- added R11, R12, R5, R8: RESISTOR_0603_10K, HyTechDevices:RESISTOR_0603_10K
- added XF1: FUSE_HOLDER_MINIBLADESMD, HyTechDevices:FUSE_HOLDER_MINIBLADESMD
- J1: value CONNECTOR-37__ -> CONNECTOR-8_μF_T_V_BLACK; device HyTechDevices:CONNECTOR-37__ -> HyTechDevices:CONNECTOR-8_μF_T_V_BLACK
- J2, J3: value CONNECTOR-8_AMPHENOL_M12A_08PMMP_ -> CONNECTOR-8_μF_T_V_BLACK; device HyTechDevices:CONNECTOR-8_AMPHENOL_M12A_08PMMP_ -> HyTechDevices:CONNECTOR-8_μF_T_V_BLACK
- J4: value CONNECTOR-6_AS_PCT_ -> CONNECTOR-8_μF_T_V_BLACK; device HyTechDevices:CONNECTOR-6_AS_PCT_ -> HyTechDevices:CONNECTOR-8_μF_T_V_BLACK
- J5: value CONNECTOR-13_SOURIAU_ -> CONNECTOR-4_μF_T_V_BLACK; device HyTechDevices:CONNECTOR-13_SOURIAU_ -> HyTechDevices:CONNECTOR-4_μF_T_V_BLACK
Connections:
- removed net LATCH: J1.21
- removed net N$1: J1.5
- removed net N$4: J1.31
- removed net N$6: J3.4
- removed net SHDN_J: J1.12, J1.6
- new net +12V: A1.OUT, D5.C, Q6.S, R11.2
- new net ACCEL_1_RAW: JP3.1
- new net ACCEL_2_RAW: JP4.1
- new net BRAKE_1_RAW: JP1.1
- new net BRAKE_2_RAW: JP2.1
- new net INVERTER_24V_EN_BOOSTED: Q2.D
- new net INVERTER_EN_BOOSTED: Q4.D
- new net N$11: D5.A, Q5.D, Q6.G, R11.1
- new net N$7: Q1.D, R6.1
- new net N$8: D4.A, Q4.G, R10.1, R9.2
- new net N$9: Q3.D, R9.1
- new net SHDN_A: J5.1, J5.2, XF1.2
- new net SHDN_L: J8.3, J8.4, J9.1, J9.2
- net +24V: now also A1.IN, D2.C, D4.C, Q2.S, Q4.S, R1.2, R10.2, R2.2, R3.2, R4.2, R7.2, XF1.1; no longer J1.14, J1.24, J1.33, J1.34
- net +5V: now also R13.2, R14.2, R15.2
- net ACCEL_1_EXT: now also JP3.2, R3.1
- net ACCEL_2_EXT: now also JP4.2, R4.1
- net BMS_OK: no longer J1.28
- net BRAKELIGHT_12V: now also Q6.D; no longer J1.9
- net BRAKELIGHT_EN: now also D6.C, Q5.G, R12.2
- net BRAKE_1_EXT: now also JP1.2, R1.1
- net BRAKE_2_EXT: now also JP2.2, R2.1
- net BRAKE_PRESSURE_F_EXT: now also R14.1
- net BRAKE_PRESSURE_R_EXT: now also R15.1
- net CANH_1: no longer J1.15
- net CANH_2: no longer J1.17
- net CANH_3: no longer J1.1
- net CANL_1: no longer J1.16
- net CANL_2: no longer J1.18
- net CANL_3: no longer J1.2
- net CURRENT_EXT: no longer J1.3
- net GND: now also A1.GND, D1.A, D3.A, D6.A, Q1.S, Q3.S, Q5.S, R12.1, R5.1, R8.1; no longer J1.10, J1.13, J1.32, J1.35, J1.37, J1.8
- net INVERTER_24V_EN: now also D1.C, Q1.G, R5.2; no longer J1.19
- net INVERTER_EN: now also D3.C, Q3.G, R8.2; no longer J1.30
- net LOAD_RL_EXT: no longer J1.27
- net LOAD_RR_EXT: no longer J1.23
- net N$5: now also D2.A, Q2.G, R6.2, R7.1; no longer J1.36
- net OKHS_IN: no longer J1.29
- net REFERENCE_EXT: no longer J1.4
- net SHDN_B: now also J5.3, J5.4
- net SHDN_I: no longer J1.11
- net SHDN_K: now also J8.1, J8.2; no longer J1.7
- net SHDN_M: now also J9.3, J9.4; no longer J1.20
- net SPN_POT_4_EXT: no longer J1.26
- net SPN_POT_5_EXT: no longer J1.25
- net SPN_POT_6_EXT: no longer J1.22
- net STEERING_1_EXT: now also R13.1
Other:
- note added: "BOTS"
- note added: "BRB"
- note added: "Inertia"
- note removed: "Accumulator Current Sense"
- note removed: "Brake Light"
- note removed: "CAN Front"
- note removed: "CAN Peripheral"
- note removed: "CAN Rear"
- note removed: "Digital Signals"
- note removed: "Power"
- note removed: "RL Corner"
- note removed: "RR Corner"

Commit message: routing progress. added 100 ohm SPI resistors
Parts:
- removed JP1, JP2, JP3, JP4: JUMPER__1X02, HyTechDevices:JUMPER__1X02
- removed R13, R4: RESISTOR_0603_100K, HyTechDevices:RESISTOR_0603_100K
- J10: value CONNECTOR-18_MF_T_V_ -> CONNECTOR-16_MF_T_V_; device HyTechDevices:CONNECTOR-18_MF_T_V_ -> HyTechDevices:CONNECTOR-16_MF_T_V_
- J12: value CONNECTOR-10_MF_T_V_ -> CONNECTOR-8_μF_T_V_BLACK; device HyTechDevices:CONNECTOR-10_MF_T_V_ -> HyTechDevices:CONNECTOR-8_μF_T_V_BLACK
- J6, J7: value CONNECTOR-40__ -> CONNECTOR-34__; device HyTechDevices:CONNECTOR-40__ -> HyTechDevices:CONNECTOR-34__
- R1, R2, R3: value RESISTOR_0603_100K -> RESISTOR_0603_100; device HyTechDevices:RESISTOR_0603_100K -> HyTechDevices:RESISTOR_0603_100
Connections:
- removed net ACCEL_1_RAW: JP3.1
- removed net ACCEL_2_RAW: JP4.1
- removed net BRAKE_1_RAW: JP1.1
- removed net BRAKE_2_RAW: JP2.1
- removed net FL_INTERLOCK_SENSE_EXT: J7.30
- removed net FR_INTERLOCK_SENSE_EXT: J7.28
- removed net INERTIA_SENSE_EXT: J7.31
- removed net RL_INTERLOCK_SENSE_EXT: J7.32
- removed net RR_INTERLOCK_SENSE_EXT: J7.29
- removed net TCU_RX5: J7.18
- removed net TCU_RX6: J7.23
- removed net TCU_RX7: J7.24
- removed net TCU_TX4: J7.20
- removed net TCU_TX5: J7.19
- removed net TCU_TX6: J7.22
- removed net TCU_TX7: J7.25
- removed net TXU_RX4: J7.21
- new net N$1: J1.2, R1.1
- new net N$2: J1.3, R2.1
- new net N$3: J1.4, R3.1
- new net SHDN_J: J11.11, J11.16, J7.5
- net !STEERING_2_CS: now also J1.5, J7.15; no longer J7.12
- net +24V: now also J11.1, J11.13, J11.2, J11.6, J12.1, J6.34; no longer J7.40, R1.2, R2.2, R3.2, R4.2
- net +5V: now also J1.1, J4.1, J6.33; no longer J7.38, R13.2, R14.2, R15.2
- net ACCEL_1_EXT: now also J4.2, J6.1; no longer J6.29, JP3.2, R3.1
- net ACCEL_2_EXT: now also J4.3, J6.2; no longer J6.30, JP4.2, R4.1
- net BMS_OK: now also J10.10, J7.31; no longer J7.34
- net BRAKELIGHT_12V: now also J10.15
- net BRAKELIGHT_EN: now also J7.21; no longer J7.9
- net BRAKE_1_EXT: now also J4.4, J6.3; no longer J6.27, JP1.2, R1.1
- net BRAKE_2_EXT: now also J4.5, J6.4; no longer J6.28, JP2.2, R2.1
- net BRAKE_PRESSURE_F_EXT: now also J4.6, J6.18; no longer J6.23
- net BRAKE_PRESSURE_R_EXT: now also J4.7, J6.19; no longer J6.24
- net CANH_1: now also J10.6, J6.27; no longer J6.12
- net CANH_2: now also J10.4, J6.31; no longer J6.8
- net CANH_3: now also J10.2, J12.4, J6.21; no longer J6.4
- net CANL_1: now also J10.5, J6.25; no longer J6.10
- net CANL_2: now also J10.3, J6.29; no longer J6.6
- net CANL_3: now also J10.1, J12.3, J6.23; no longer J6.2
- net CURRENT_EXT: now also J10.7, J6.6; no longer J6.19
- net ECU_CLK: now also R1.2
- net ECU_SDI: now also J7.9, R2.2; no longer J7.14
- net ECU_SDO: now also J7.11, R3.2; no longer J7.15
- net GND: now also J1.8, J10.16, J11.12, J11.18, J11.3, J11.4, J11.5, J12.8, J4.8, J6.20, J6.24, J6.28, J6.30, J6.32, R14.2, R15.2; no longer J6.1, J6.11, J6.13, J6.14, J6.17, J6.18, J6.21, J6.3, J6.5, J6.7, J6.9, J7.16, J7.17, J7.26, J7.27, J7.3, J7.35, J7.36, J7.37, J7.39, J7.4, J7.7, J7.8
- net INVERTER_24V_EN: now also J7.19; no longer J7.10
- net INVERTER_24V_EN_BOOSTED: now also J10.11
- net INVERTER_EN: now also J7.17; no longer J7.11
- net INVERTER_EN_BOOSTED: now also J10.12
- net LATCH_BTN: now also J10.14, J7.25, J7.26; no longer J7.5, J7.6
- net LOAD_FL_EXT: now also J6.13; no longer J6.39
- net LOAD_FR_EXT: now also J6.14; no longer J6.40
- net LOAD_RL_EXT: now also J11.7, J6.8; no longer J6.37
- net LOAD_RR_EXT: now also J11.14, J6.12; no longer J6.38
- net OKHS_IN: now also J10.9, J7.32; no longer J7.33
- net REFERENCE_EXT: now also J10.8, J6.7; no longer J6.20
- net SHDN_B: now also J12.5, J7.33, J7.34; no longer J6.15, J6.16
- net SHDN_H: now also J7.3
- net SHDN_I: now also J11.10, J7.4
- net SHDN_K: now also J11.17, J7.6
- net SHDN_L: now also J12.6, J7.7
- net SHDN_M: now also J10.13, J12.2
- net SPN_POT_1_EXT: now also J6.15; no longer J6.35
- net SPN_POT_2_EXT: now also J6.16; no longer J6.36
- net SPN_POT_3_EXT: now also J6.17; no longer J6.33
- net SPN_POT_4_EXT: now also J11.8, J6.9; no longer J6.34
- net SPN_POT_5_EXT: now also J11.9, J6.10; no longer J6.31
- net SPN_POT_6_EXT: now also J11.15, J6.11; no longer J6.32
- net STEERING_1_EXT: now also J1.7, J6.5; no longer J6.25, R13.1

Commit message: finished routing. passed DRC
Parts:
- J4: value CONNECTOR-8_μF_T_V_BLACK -> CONNECTOR-10_MF_T_V_; device HyTechDevices:CONNECTOR-8_μF_T_V_BLACK -> HyTechDevices:CONNECTOR-10_MF_T_V_
Connections:
- net CANH_1: now also J10.3; no longer J10.6
- net CANH_2: now also J10.1; no longer J10.4
- net CANH_3: now also J10.6; no longer J10.2
- net CANL_1: now also J10.4; no longer J10.5
- net CANL_2: now also J10.2; no longer J10.3
- net CANL_3: now also J10.5; no longer J10.1
- net CURRENT_EXT: now also J10.8; no longer J10.7
- net LOAD_RL_EXT: now also J11.9; no longer J11.7
- net REFERENCE_EXT: now also J10.7; no longer J10.8
- net SHDN_H: now also J3.8; no longer J3.5
- net SPN_POT_5_EXT: now also J11.7; no longer J11.9
Other:
- moved on the sheet: J12, J5, J8, J9
