File: EAGLE Board Designs/Tractive System Board/Tractive System Board Rev6.brd (EAGLE design)
At the start: 209.3 x 74 mm, 135 parts, among them J1 CONNECTOR-5_MICRO_V7S_, J2 CONNECTOR-5_MICRO_V6S_, J3 CONNECTOR-8_μF_T_V_BLACK, K1 RELAY_SPST_NO_D_24, Q1 TRANSISTOR_N_MOS_POWERFLAT5X6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, Q2 TRANSISTOR_N_MOS__PMV15ENEA, T1 TRANSFORMER(3W), U1 VOLTAGE_REGULATOR_SOT-223_10V, U10 LTC6994-2, U2 LT8316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

Commit message: tsb-update
Replaced 24-to-5V linear regulator to DC-DC converter
Parts:
- removed U6: VOLTAGE_REGULATOR_SOT-23-5_5V, HyTechDevices:SOT-23-5
- added A1: VOLTAGE_REGULATOR_MODULE_OKI-78SR_5V, HyTechDevices:OKI-78SR
- C24: value CAPACITOR_0603_10V_4.7UF -> CAPACITOR_0603_25V_10UF
- C27: value CAPACITOR_0603_50V_1UF -> CAPACITOR_0603_50V_10NF
- moved C24 7.62 mm to (56.1, -62.2)
- moved C25 7.62 mm to (57.9, -62.2)
- moved C27 0.76 mm to (74.7, -62.2)
Connections:
- net +24V: now also A1.1; no longer U6.2
- net +5V: now also A1.3; no longer U6.3
- net GND: now also A1.2; no longer U6.1
Routing:
- net GND: track 112.6 -> 123.4 mm
- net +5V: track 138.1 -> 146.3 mm
- net +24V: track 74.6 -> 78.5 mm
- net PRECHARGE_OK: track 77.6 -> 79.3 mm
