File: ESF Schematics/2024/BSPD System Schematic.sch (EAGLE design)
At the start: 47 parts, among them Q1 MOSFET_N-CHANNEL, Q2 MOSFET_P-CHANNEL, U1 OPAMP, U10 LOGICGATE_NOR, U11 OPAMP, U12 LOGICGATE_OR, U13 LOGICGATE_OR, U14 OPAMP, U2 OPAMP, U3 OPAMP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

Commit message: Update BSPD System Schematic.sch
Parts:
- A2: value BSE9360 -> BSEEURO-XPD-2838-806-214-911-00; device HyTechSymbols:BSE9360 -> HyTechSymbols:BSEEURO-XPD-2838-806-214-911-00
Connections:
- net 0.5V renamed 0.9V
- net 4.45V renamed 4.4V
Changed lines of the file:
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@@
 <part name="P15" library="HyTechSupplies" deviceset="GND" device=""/>
 <part name="P16" library="HyTechSupplies" deviceset="+5V" device=""/>
-<part name="A2" library="HyTechSymbols" deviceset="BSE" device="" technology="9360" value="BSE9360"/>
+<part name="A2" library="HyTechSymbols" deviceset="BSE" device="" technology="EURO-XPD-2838-806-214-911-00" value="BSEEURO-XPD-2838-806-214-911-00"/>
 <part name="LATCHING_BUTTON" library="HyTechSymbolsTemp" deviceset="BUTTON_NO_*" device="" technology="LP9"/>
 <part name="U1" library="HyTechSymbols" deviceset="OPAMP" device=""/>
@@
 </segment>
 </net>
-<net name="4.45V" class="0">
+<net name="4.4V" class="0">
 <segment>
 <pinref part="U7" gate="G$1" pin="VIN-"/>
@@
 </segment>
 </net>
-<net name="0.5V" class="0">
+<net name="0.9V" class="0">
 <segment>
 <pinref part="U14" gate="G$1" pin="VIN+"/>

Commit message: num num
Connections:
- net 0.9V renamed 0.5V
- net 4.4V renamed 4.5V
Changed lines of the file:
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@@
 </segment>
 </net>
-<net name="4.4V" class="0">
+<net name="4.5V" class="0">
 <segment>
 <pinref part="U7" gate="G$1" pin="VIN-"/>
@@
 </segment>
 </net>
-<net name="0.9V" class="0">
+<net name="0.5V" class="0">
 <segment>
 <pinref part="U14" gate="G$1" pin="VIN+"/>

Commit message: fixing broken stuff
Parts:
- removed U$6: FILTER_ACTIVE606.3HZ, HyTechSymbols:FILTER_ACTIVE606.3HZ
- U$1, U$2: value FILTER_ACTIVE606.3HZ -> FILTER_ACTIVE; device HyTechSymbols:FILTER_ACTIVE606.3HZ -> HyTechSymbols:FILTER_ACTIVE1KHZ
Connections:
- net 0.5V renamed 0.3V
- net 4.5V renamed 2.7V
- net +5V: no longer R1.2, U$6.VDD
- net GND: now also R1.1; no longer U$6.GND
- net SIGNAL_BRAKE: now also R1.2; no longer R1.1, U$6.IN, U$6.OUT
Other:
- moved on the sheet: R1
Changed lines of the file:
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@@
 <part name="R9" library="HyTechSymbols" deviceset="RESISTOR" device="" value="10.5K"/>
 <part name="P11" library="HyTechSupplies" deviceset="GND" device=""/>
-<part name="U$1" library="HyTechSymbols" deviceset="FILTER_ACTIVE" device="" technology="606.3HZ" value="FILTER_ACTIVE606.3HZ"/>
+<part name="U$1" library="HyTechSymbols" deviceset="FILTER_ACTIVE" device="" technology="1KHZ" value="FILTER_ACTIVE"/>
 <part name="P14" library="HyTechSupplies" deviceset="GND" device=""/>
 <part name="P17" library="HyTechSupplies" deviceset="+5V" device=""/>
 <part name="P18" library="HyTechSupplies" deviceset="GND" device=""/>
-<part name="U$2" library="HyTechSymbols" deviceset="FILTER_ACTIVE" device="" technology="606.3HZ" value="FILTER_ACTIVE606.3HZ"/>
+<part name="U$2" library="HyTechSymbols" deviceset="FILTER_ACTIVE" device="" technology="1KHZ" value="FILTER_ACTIVE"/>
 <part name="P19" library="HyTechSupplies" deviceset="GND" device=""/>
 <part name="P20" library="HyTechSupplies" deviceset="+5V" device=""/>
@@
 <part name="U6" library="HyTechSymbols" deviceset="OPAMP" device=""/>
 <part name="U7" library="HyTechSymbols" deviceset="OPAMP" device=""/>
-<part name="U$6" library="HyTechSymbols" deviceset="FILTER_ACTIVE" device="" technology="606.3HZ" value="FILTER_ACTIVE606.3HZ"/>
 <part name="P3" library="HyTechSupplies" deviceset="GND" device=""/>
-<part name="P25" library="HyTechSupplies" deviceset="+5V" device=""/>
 <part name="R1" library="HyTechSymbols" deviceset="RESISTOR" device="" value="100K"/>
-<part name="P2" library="HyTechSupplies" deviceset="+5V" device=""/>
 <part name="U8" library="HyTechSymbols" deviceset="LOGICGATE_OR" device=""/>
 <part name="U9" library="HyTechSymbols" deviceset="LOGICGATE_AND" device=""/>
@@
 <instance part="U6" gate="G$1" x="175.26" y="147.32" smashed="yes"/>
 <instance part="U7" gate="G$1" x="149.86" y="180.34" smashed="yes"/>
-<instance part="U$6" gate="G$1" x="124.46" y="116.84" smashed="yes">
-<attribute name="MANUFACTURER" x="124.46" y="118.11" size="1.778" layer="97"/>
-<attribute name="MPN" x="124.46" y="93.98" size="1.778" layer="97"/>
-<attribute name="FREQ" x="124.46" y="91.44" size="1.778" layer="97"/>
-</instance>
 <instance part="P3" gate="1" x="119.38" y="88.9" smashed="yes">
 <attribute name="VALUE" x="119.38" y="87.63" size="1.27" layer="96" align="top-center"/>
 </instance>
-<instance part="P25" gate="1" x="149.86" y="119.38" smashed="yes">
-<attribute name="VALUE" x="149.86" y="121.92" size="1.27" layer="96" align="bottom-center"/>
-</instance>
-<instance part="R1" gate="G$1" x="119.38" y="111.76" smashed="yes" rot="R90">
-<attribute name="NAME" x="118.11" y="110.49" size="1.27" layer="95" rot="R90" align="bottom-center"/>
-<attribute name="VALUE" x="120.65" y="110.49" size="1.27" layer="96" rot="R90" align="top-center"/>
-</instance>
-<instance part="P2" gate="1" x="119.38" y="119.38" smashed="yes">
-<attribute name="VALUE" x="119.38" y="121.92" size="1.27" layer="96" align="bottom-center"/>
+<instance part="R1" gate="G$1" x="111.76" y="99.06" smashed="yes" rot="R90">
+<attribute name="NAME" x="110.49" y="97.79" size="1.27" layer="95" rot="R90" align="bottom-center"/>
+<attribute name="VALUE" x="113.03" y="97.79" size="1.27" layer="96" rot="R90" align="top-center"/>
 </instance>
 <instance part="U8" gate="G$1" x="208.28" y="177.8" smashed="yes"/>
@@
 <segment>
 <pinref part="P3" gate="1" pin="GND"/>
-<pinref part="U$6" gate="G$1" pin="GND"/>
 <wire x1="119.38" y1="91.44" x2="119.38" y2="99.06" width="0.0762" layer="91"/>
 <wire x1="119.38" y1="99.06" x2="121.92" y2="99.06" width="0.0762" layer="91"/>
+<pinref part="R1" gate="G$1" pin="1"/>
+<wire x1="111.76" y1="93.98" x2="111.76" y2="91.44" width="0.0762" layer="91"/>
+<wire x1="111.76" y1="91.44" x2="119.38" y2="91.44" width="0.0762" layer="91"/>
+<junction x="119.38" y="91.44"/>
 </segment>
 <segment>
@@
 </segment>
 <segment>
-<pinref part="U$6" gate="G$1" pin="VDD"/>
-<pinref part="P25" gate="1" pin="+5V"/>
-<wire x1="147.32" y1="114.3" x2="149.86" y2="114.3" width="0.0762" layer="91"/>
-<wire x1="149.86" y1="114.3" x2="149.86" y2="116.84" width="0.0762" layer="91"/>
-</segment>
-<segment>
-<pinref part="P2" gate="1" pin="+5V"/>
-<pinref part="R1" gate="G$1" pin="2"/>
-<wire x1="119.38" y1="116.84" x2="119.38" y2="114.3" width="0.1524" layer="91"/>
-</segment>
-<segment>
 <pinref part="A2" gate="G$1" pin="VDD"/>
 <pinref part="P16" gate="1" pin="+5V"/>
@@
 <wire x1="160.02" y1="83.82" x2="160.02" y2="104.14" width="0.0762" layer="91"/>
 <junction x="160.02" y="104.14"/>
-<pinref part="U$6" gate="G$1" pin="OUT"/>
 <wire x1="147.32" y1="104.14" x2="160.02" y2="104.14" width="0.0762" layer="91"/>
 <pinref part="U11" gate="G$1" pin="VIN-"/>
@@
 </segment>
 <segment>
-<pinref part="U$6" gate="G$1" pin="IN"/>
-<wire x1="121.92" y1="104.14" x2="119.38" y2="104.14" width="0.0762" layer="91"/>
-<pinref part="R1" gate="G$1" pin="1"/>
-<wire x1="119.38" y1="106.68" x2="119.38" y2="104.14" width="0.0762" layer="91"/>
-<wire x1="119.38" y1="104.14" x2="104.14" y2="104.14" width="0.0762" layer="91"/>
-<junction x="119.38" y="104.14"/>
+<wire x1="121.92" y1="104.14" x2="111.76" y2="104.14" width="0.0762" layer="91"/>
 <pinref part="S1" gate="SPST" pin="O"/>
+<wire x1="111.76" y1="104.14" x2="104.14" y2="104.14" width="0.0762" layer="91"/>
 <wire x1="104.14" y1="104.14" x2="104.14" y2="106.68" width="0.0762" layer="91"/>
+<pinref part="R1" gate="G$1" pin="2"/>
+<wire x1="111.76" y1="104.14" x2="111.76" y2="101.6" width="0.0762" layer="91"/>
+<junction x="111.76" y="104.14"/>
 </segment>
 <segment>
@@
 </segment>
 </net>
-<net name="4.5V" class="0">
+<net name="2.7V" class="0">
 <segment>
 <pinref part="U7" gate="G$1" pin="VIN-"/>
@@
 </segment>
 </net>
-<net name="0.5V" class="0">
+<net name="0.3V" class="0">
 <segment>
 <pinref part="U14" gate="G$1" pin="VIN+"/>

Commit message: Update BSPD System Schematic.sch
Parts:
- added R11: RESISTOR_0603_15K, HyTechDevices:RESISTOR_0603_15K
- added U$3: FILTER_ACTIVE, HyTechSymbols:FILTER_ACTIVE
- R1: value 100K -> RESISTOR_0603_10K; device HyTechSymbols:RESISTOR -> HyTechDevices:RESISTOR_0603_10K
Connections:
- new net +3V3: U$3.VDD
- new net 0.5V: U14.VIN+
- new net 4.5V: U7.VIN-
- new net N$6: R1.2, R11.2, U$3.IN
- new net N$9: R1.1, S1.O
- net 0.3V: no longer U14.VIN+
- net 2.7V: no longer U7.VIN-
- net GND: now also R11.1, U$3.GND; no longer R1.1
- net SIGNAL_BRAKE: now also U$3.OUT; no longer R1.2, S1.O
Other:
- note added: "0.6x Voltage divider 5->3V"
- note added: "Eric Galluzzi"
- note added: "Shayan N. & Mikhail Allen"
- moved on the sheet: R1
Changed lines of the file:
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@@
 <layer number="56" name="wert" color="7" fill="1" visible="no" active="no"/>
 <layer number="57" name="tCAD" color="7" fill="1" visible="no" active="no"/>
+<layer number="58" name="bCAD" color="7" fill="1" visible="no" active="no"/>
 <layer number="59" name="tCarbon" color="7" fill="1" visible="no" active="no"/>
 <layer number="60" name="bCarbon" color="7" fill="1" visible="no" active="no"/>
@@
 <layer number="156" name="HIGH_CURRENT_PATH" color="12" fill="1" visible="yes" active="yes"/>
 <layer number="157" name="HIGH_VOLTAGE_WIRES" color="2" fill="1" visible="yes" active="yes"/>
+<layer number="166" name="AntennaArea" color="7" fill="1" visible="no" active="no"/>
+<layer number="168" name="4mmHeightArea" color="7" fill="1" visible="no" active="no"/>
 <layer number="191" name="mNets" color="7" fill="1" visible="yes" active="yes"/>
 <layer number="192" name="mBusses" color="7" fill="1" visible="yes" active="yes"/>
@@
 <part name="U7" library="HyTechSymbols" deviceset="OPAMP" device=""/>
 <part name="P3" library="HyTechSupplies" deviceset="GND" device=""/>
-<part name="R1" library="HyTechSymbols" deviceset="RESISTOR" device="" value="100K"/>
 <part name="U8" library="HyTechSymbols" deviceset="LOGICGATE_OR" device=""/>
 <part name="U9" library="HyTechSymbols" deviceset="LOGICGATE_AND" device=""/>
@@
 <part name="U13" library="HyTechSymbols" deviceset="LOGICGATE_OR" device=""/>
 <part name="U14" library="HyTechSymbols" deviceset="OPAMP" device=""/>
+<part name="U$3" library="HyTechSymbols" deviceset="FILTER_ACTIVE" device=""/>
+<part name="R1" library="HyTechDevices" deviceset="RESISTOR_?_*" device="0603" technology="10K"/>
+<part name="R11" library="HyTechDevices" deviceset="RESISTOR_?_*" device="0603" technology="15K"/>
+<part name="P2" library="HyTechSupplies" deviceset="+3V3" device=""/>
 </parts>
 <sheets>
@@
 24.16-&gt;4.891V</text>
 <text x="99.06" y="97.536" size="1.27" layer="97" align="top-center">BSE Testing Switch</text>
-<text x="111.76" y="106.68" size="1.27" layer="97" align="top-center">PCB Trace</text>
-<text x="134.62" y="22.86" size="2.54" layer="95">Shayan Noorani</text>
+<text x="116.84" y="106.68" size="1.27" layer="97" align="top-center">PCB Trace</text>
+<text x="130.556" y="22.606" size="2.54" layer="95">Shayan N. &amp; Mikhail Allen</text>
 <text x="180.34" y="30.48" size="2.54" layer="95">Shayan Noorani</text>
+<text x="99.06" y="111.76" size="1.27" layer="97">0.6x Voltage divider
+5-&gt;3V</text>
+<text x="233.68" y="30.48" size="2.54" layer="95">Eric Galluzzi</text>
 </plain>
 <instances>
@@
 <instance part="P3" gate="1" x="119.38" y="88.9" smashed="yes">
 <attribute name="VALUE" x="119.38" y="87.63" size="1.27" layer="96" align="top-center"/>
-</instance>
-<instance part="R1" gate="G$1" x="111.76" y="99.06" smashed="yes" rot="R90">
-<attribute name="NAME" x="110.49" y="97.79" size="1.27" layer="95" rot="R90" align="bottom-center"/>
-<attribute name="VALUE" x="113.03" y="97.79" size="1.27" layer="96" rot="R90" align="top-center"/>
 </instance>
 <instance part="U8" gate="G$1" x="208.28" y="177.8" smashed="yes"/>
@@
 <attribute name="VALUE" x="165.1" y="156.21" size="1.27" layer="96" align="top-center"/>
 </instance>
-<instance part="S1" gate="SPST" x="99.06" y="104.14" smashed="yes">
-<attribute name="MANUFACTURER" x="99.06" y="107.442" size="1.27" layer="96" align="bottom-center"/>
-<attribute name="MPN" x="99.06" y="100.838" size="1.27" layer="96" align="top-center"/>
+<instance part="S1" gate="SPST" x="96.52" y="104.14" smashed="yes">
+<attribute name="MANUFACTURER" x="96.52" y="107.442" size="1.27" layer="96" align="bottom-center"/>
+<attribute name="MPN" x="96.52" y="100.838" size="1.27" layer="96" align="top-center"/>
 </instance>
 <instance part="U11" gate="G$1" x="172.72" y="114.3" smashed="yes"/>
@@
 <instance part="U13" gate="G$1" x="195.58" y="172.72" smashed="yes"/>
 <instance part="U14" gate="G$1" x="149.86" y="193.04" smashed="yes"/>
+<instance part="U$3" gate="G$1" x="124.46" y="116.84" smashed="yes">
+<attribute name="MANUFACTURER" x="124.46" y="118.11" size="1.778" layer="97"/>
+<attribute name="MPN" x="124.46" y="93.98" size="1.778" layer="97"/>
+<attribute name="FREQ" x="124.46" y="91.44" size="1.778" layer="97"/>
+</instance>
+<instance part="R1" gate="G$1" x="106.68" y="104.14" smashed="yes">
+<attribute name="NAME" x="105.41" y="105.41" size="1.27" layer="95" align="bottom-center"/>
+<attribute name="RESISTANCE" x="105.41" y="102.87" size="1.27" layer="96" align="top-center"/>
+</instance>
+<instance part="R11" gate="G$1" x="111.76" y="99.06" smashed="yes" rot="R90">
+<attribute name="NAME" x="110.49" y="97.79" size="1.27" layer="95" rot="R90" align="bottom-center"/>
+<attribute name="RESISTANCE" x="113.03" y="97.79" size="1.27" layer="96" rot="R90" align="top-center"/>
+</instance>
+<instance part="P2" gate="G$1" x="149.86" y="121.92" smashed="yes">
+<attribute name="VALUE" x="149.86" y="123.19" size="1.27" layer="96" align="bottom-center"/>
+</instance>
 </instances>
 <busses>
@@
 <wire x1="119.38" y1="91.44" x2="119.38" y2="99.06" width="0.0762" layer="91"/>
 <wire x1="119.38" y1="99.06" x2="121.92" y2="99.06" width="0.0762" layer="91"/>
-<pinref part="R1" gate="G$1" pin="1"/>
 <wire x1="111.76" y1="93.98" x2="111.76" y2="91.44" width="0.0762" layer="91"/>
 <wire x1="111.76" y1="91.44" x2="119.38" y2="91.44" width="0.0762" layer="91"/>
 <junction x="119.38" y="91.44"/>
+<pinref part="U$3" gate="G$1" pin="GND"/>
+<pinref part="R11" gate="G$1" pin="1"/>
 </segment>
 <segment>
@@
 <wire x1="170.18" y1="111.76" x2="160.02" y2="111.76" width="0.0762" layer="91"/>
 <wire x1="160.02" y1="111.76" x2="160.02" y2="104.14" width="0.0762" layer="91"/>
-</segment>
-<segment>
-<wire x1="121.92" y1="104.14" x2="111.76" y2="104.14" width="0.0762" layer="91"/>
-<pinref part="S1" gate="SPST" pin="O"/>
-<wire x1="111.76" y1="104.14" x2="104.14" y2="104.14" width="0.0762" layer="91"/>
-<wire x1="104.14" y1="104.14" x2="104.14" y2="106.68" width="0.0762" layer="91"/>
-<pinref part="R1" gate="G$1" pin="2"/>
-<wire x1="111.76" y1="104.14" x2="111.76" y2="101.6" width="0.0762" layer="91"/>
-<junction x="111.76" y="104.14"/>
+<pinref part="U$3" gate="G$1" pin="OUT"/>
 </segment>
 <segment>
 <pinref part="S1" gate="SPST" pin="P"/>
-<wire x1="93.98" y1="104.14" x2="88.9" y2="104.14" width="0.0762" layer="91"/>
+<wire x1="91.44" y1="104.14" x2="88.9" y2="104.14" width="0.0762" layer="91"/>
 <label x="88.9" y="104.14" size="1.27" layer="95" rot="R180" xref="yes"/>
 </segment>
@@
 <net name="2.7V" class="0">
 <segment>
-<pinref part="U7" gate="G$1" pin="VIN-"/>
-<wire x1="147.32" y1="177.8" x2="144.78" y2="177.8" width="0.0762" layer="91"/>
-<label x="144.78" y="177.8" size="1.27" layer="95" rot="R180" xref="yes"/>
-</segment>
-<segment>
 <pinref part="U1" gate="G$1" pin="VIN-"/>
 <wire x1="170.18" y1="99.06" x2="167.64" y2="99.06" width="0.0762" layer="91"/>
@@
 <net name="0.3V" class="0">
 <segment>
-<pinref part="U14" gate="G$1" pin="VIN+"/>
-<wire x1="147.32" y1="195.58" x2="144.78" y2="195.58" width="0.0762" layer="91"/>
-<label x="144.78" y="195.58" size="1.27" layer="95" rot="R180" xref="yes"/>
-</segment>
-<segment>
 <pinref part="U11" gate="G$1" pin="VIN+"/>
 <wire x1="170.18" y1="116.84" x2="167.64" y2="116.84" width="0.0762" layer="91"/>
@@
 </segment>
 </net>
+<net name="N$9" class="0">
+<segment>
+<pinref part="S1" gate="SPST" pin="O"/>
+<wire x1="101.6" y1="104.14" x2="101.6" y2="106.68" width="0.0762" layer="91"/>
+<pinref part="R1" gate="G$1" pin="1"/>
+</segment>
+</net>
+<net name="N$6" class="0">
+<segment>
+<pinref part="R1" gate="G$1" pin="2"/>
+<pinref part="U$3" gate="G$1" pin="IN"/>
+<wire x1="121.92" y1="104.14" x2="111.76" y2="104.14" width="0.0762" layer="91"/>
+<pinref part="R11" gate="G$1" pin="2"/>
+<wire x1="111.76" y1="104.14" x2="109.22" y2="104.14" width="0.0762" layer="91"/>
+<wire x1="111.76" y1="101.6" x2="111.76" y2="104.14" width="0.0762" layer="91"/>
+<junction x="111.76" y="104.14"/>
+</segment>
+</net>
+<net name="+3V3" class="0">
+<segment>
+<pinref part="U$3" gate="G$1" pin="VDD"/>
+<wire x1="147.32" y1="114.3" x2="149.86" y2="114.3" width="0.1524" layer="91"/>
+<wire x1="149.86" y1="114.3" x2="149.86" y2="119.38" width="0.1524" layer="91"/>
+<pinref part="P2" gate="G$1" pin="+3V3"/>
+</segment>
+</net>
+<net name="0.5V" class="0">
+<segment>
+<pinref part="U14" gate="G$1" pin="VIN+"/>
+<wire x1="147.32" y1="195.58" x2="144.78" y2="195.58" width="0.1524" layer="91"/>
+<label x="144.78" y="195.58" size="1.27" layer="95" rot="R180" xref="yes"/>
+</segment>
+</net>
+<net name="4.5V" class="0">
+<segment>
+<pinref part="U7" gate="G$1" pin="VIN-"/>
+<wire x1="147.32" y1="177.8" x2="144.78" y2="177.8" width="0.1524" layer="91"/>
+<label x="144.78" y="177.8" size="1.27" layer="95" rot="R180" xref="yes"/>
+</segment>
+</net>

Commit message: changes after review
Parts:
- BSPD_RELAY: value RELAY_DPDT_ -> RELAY_DPDT_3-1462039-7; device HyTechSymbols:RELAY_DPDT_ -> HyTechSymbols:RELAY_DPDT_3-1462039-7; MPN RT424024 -> (none)
Changed lines of the file:
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@@
 </classes>
 <parts>
-<part name="BSPD_RELAY" library="HyTechSymbols" deviceset="RELAY_DPDT_?*" device="" value="RELAY_DPDT_">
-<attribute name="MPN" value="RT424024"/>
-</part>
 <part name="D4" library="HyTechSymbolsTemp" deviceset="DIODE" device=""/>
 <part name="D5" library="HyTechSymbolsTemp" deviceset="DIODE" device=""/>
@@
 <part name="R11" library="HyTechDevices" deviceset="RESISTOR_?_*" device="0603" technology="15K"/>
 <part name="P2" library="HyTechSupplies" deviceset="+3V3" device=""/>
+<part name="BSPD_RELAY" library="HyTechSymbols" deviceset="RELAY_DPDT_?*" device="" technology="3-1462039-7"/>
 </parts>
 <sheets>
@@
 </plain>
 <instances>
-<instance part="BSPD_RELAY" gate="G$1" x="238.76" y="86.36" smashed="yes">
-<attribute name="MPN" x="238.76" y="52.578" size="1.27" layer="96" align="top-left"/>
-<attribute name="NAME" x="238.76" y="87.122" size="1.27" layer="95"/>
-</instance>
 <instance part="D4" gate="G$1" x="228.6" y="78.74" smashed="yes" rot="R180">
 <attribute name="NAME" x="229.87" y="76.835" size="1.27" layer="95" rot="R180" align="bottom-center"/>
@@
 <attribute name="VALUE" x="149.86" y="123.19" size="1.27" layer="96" align="bottom-center"/>
 </instance>
+<instance part="BSPD_RELAY" gate="G$1" x="238.76" y="86.36" smashed="yes">
+<attribute name="MPN" x="238.76" y="52.578" size="1.27" layer="96" align="top-left"/>
+<attribute name="NAME" x="238.76" y="87.122" size="1.27" layer="96"/>
+</instance>
 </instances>
 <busses>
@@
 <net name="GND" class="0">
 <segment>
-<pinref part="BSPD_RELAY" gate="G$1" pin="4"/>
 <wire x1="251.46" y1="71.12" x2="256.54" y2="71.12" width="0.0762" layer="91"/>
 <wire x1="256.54" y1="71.12" x2="256.54" y2="68.58" width="0.0762" layer="91"/>
 <pinref part="P12" gate="1" pin="GND"/>
+<pinref part="BSPD_RELAY" gate="G$1" pin="4"/>
 </segment>
 <segment>
@@
 <net name="N$14" class="0">
 <segment>
-<pinref part="BSPD_RELAY" gate="G$1" pin="COIL-"/>
 <pinref part="D4" gate="G$1" pin="A"/>
 <wire x1="236.22" y1="78.74" x2="233.68" y2="78.74" width="0.0762" layer="91"/>
@@
 <wire x1="236.22" y1="93.98" x2="241.3" y2="93.98" width="0.0762" layer="91"/>
 <junction x="236.22" y="78.74"/>
+<wire x1="236.22" y1="68.58" x2="236.22" y2="68.58" width="0.0762" layer="91"/>
 <pinref part="BSPD_RELAY" gate="G$1" pin="3"/>
-<wire x1="236.22" y1="78.74" x2="236.22" y2="68.58" width="0.0762" layer="91"/>
+<pinref part="BSPD_RELAY" gate="G$1" pin="COIL-"/>
 </segment>
 </net>
 <net name="BSPD_OK" class="0">
 <segment>
-<pinref part="BSPD_RELAY" gate="G$1" pin="COIL+"/>
 <wire x1="251.46" y1="78.74" x2="256.54" y2="78.74" width="0.0762" layer="91"/>
 <pinref part="D5" gate="G$1" pin="C"/>
@@
 <wire x1="266.7" y1="119.38" x2="266.7" y2="93.98" width="0.0762" layer="91"/>
 <wire x1="266.7" y1="93.98" x2="256.54" y2="93.98" width="0.0762" layer="91"/>
+<pinref part="BSPD_RELAY" gate="G$1" pin="COIL+"/>
 </segment>
 <segment>
@@
 <net name="SHUTDOWN_D" class="0">
 <segment>
-<pinref part="BSPD_RELAY" gate="G$1" pin="6"/>
 <wire x1="236.22" y1="58.42" x2="233.68" y2="58.42" width="0.0762" layer="91"/>
 <label x="233.68" y="58.42" size="1.27" layer="95" rot="R180" xref="yes"/>
+<pinref part="BSPD_RELAY" gate="G$1" pin="6"/>
 </segment>
 </net>
@@
 <net name="SHUTDOWN_E" class="0">
 <segment>
-<pinref part="BSPD_RELAY" gate="G$1" pin="5"/>
 <wire x1="251.46" y1="60.96" x2="254" y2="60.96" width="0.0762" layer="91"/>
 <label x="254" y="60.96" size="1.27" layer="95" xref="yes"/>
-</segment>
-</net>
+<pinref part="BSPD_RELAY" gate="G$1" pin="5"/>
+</segment>
+</net>
