File: ESF Schematics/2024/Shutdown Circuit Schematic.sch (EAGLE design)
At the start: 77 parts, among them J1 CONNECTOR-2_HVP800, Q1 MOSFET_N-CHANNEL, Q2 MOSFET_N-CHANNEL, U1 LOGICGATE_INVERTER, U2 LOGICGATE_INVERTER

Commit message: changes after review
Parts:
- AMS_RELAY, BOTS_SENSE_RELAY, BSPD_RELAY, IMD_RELAY, SOFTWARE_SHDN_RELAY: value RELAY_DPDT_RT424024 -> RELAY_DPDT_3-1462039-7; device HyTechSymbols:RELAY_DPDT_RT424024 -> HyTechSymbols:RELAY_DPDT_3-1462039-7
Connections:
- removed net N$13: S5.O, S7.P
- new net N$30: S5.O, S8.P
- net N$21: no longer S8.P
- net SHDN: now also S7.P
Changed lines of the file:
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@@
 </classes>
 <parts>
-<part name="IMD_RELAY" library="HyTechSymbols" deviceset="RELAY_DPDT_?*" device="" technology="RT424024" value="RELAY_DPDT_RT424024"/>
-<part name="AMS_RELAY" library="HyTechSymbols" deviceset="RELAY_DPDT_?*" device="" technology="RT424024" value="RELAY_DPDT_RT424024"/>
-<part name="SOFTWARE_SHDN_RELAY" library="HyTechSymbols" deviceset="RELAY_DPDT_?*" device="" technology="RT424024" value="RELAY_DPDT_RT424024"/>
+<part name="IMD_RELAY" library="HyTechSymbols" deviceset="RELAY_DPDT_?*" device="" technology="3-1462039-7" value="RELAY_DPDT_3-1462039-7"/>
+<part name="AMS_RELAY" library="HyTechSymbols" deviceset="RELAY_DPDT_?*" device="" technology="3-1462039-7" value="RELAY_DPDT_3-1462039-7"/>
+<part name="SOFTWARE_SHDN_RELAY" library="HyTechSymbols" deviceset="RELAY_DPDT_?*" device="" technology="3-1462039-7" value="RELAY_DPDT_3-1462039-7"/>
 <part name="P1" library="HyTechSupplies" deviceset="GND" device=""/>
 <part name="P2" library="HyTechSupplies" deviceset="GND" device=""/>
 <part name="P4" library="HyTechSupplies" deviceset="GND" device=""/>
 <part name="P3" library="HyTechSupplies" deviceset="GND" device=""/>
-<part name="BSPD_RELAY" library="HyTechSymbols" deviceset="RELAY_DPDT_?*" device="" technology="RT424024" value="RELAY_DPDT_RT424024"/>
+<part name="BSPD_RELAY" library="HyTechSymbols" deviceset="RELAY_DPDT_?*" device="" technology="3-1462039-7" value="RELAY_DPDT_3-1462039-7"/>
 <part name="F1" library="HyTechSymbols" deviceset="FUSE" device="" value="15A"/>
 <part name="F3" library="HyTechSymbolsTemp" deviceset="FUSE" device="" value="3A"/>
@@
 <part name="Q2" library="HyTechSymbolsTemp" deviceset="MOSFET_N-CHANNEL" device=""/>
 <part name="P9" library="HyTechSupplies" deviceset="GND" device=""/>
-<part name="BOTS_SENSE_RELAY" library="HyTechSymbols" deviceset="RELAY_DPDT_?*" device="" technology="RT424024" value="RELAY_DPDT_RT424024"/>
+<part name="BOTS_SENSE_RELAY" library="HyTechSymbols" deviceset="RELAY_DPDT_?*" device="" technology="3-1462039-7" value="RELAY_DPDT_3-1462039-7"/>
 <part name="P6" library="HyTechSupplies" deviceset="GND" device=""/>
 <part name="D1" library="HyTechSymbolsTemp" deviceset="DIODE" device=""/>
@@
 <text x="68.58" y="208.28" size="1.27" layer="97" align="top-left">PCB Trace</text>
 <text x="96.52" y="165.1" size="1.27" layer="97" align="top-left">PCB Trace</text>
-<text x="76.2" y="142.24" size="1.27" layer="97" align="top-left">22AWG</text>
+<text x="110.49" y="142.494" size="1.27" layer="97" align="top-left">22AWG</text>
 <text x="208.28" y="208.28" size="1.27" layer="97" align="top-left">PCB Trace</text>
 <text x="218.44" y="142.24" size="1.27" layer="97" align="top-left">22AWG</text>
@@
 <text x="205.74" y="106.68" size="1.27" layer="97" align="top-left">22AWG</text>
 <text x="30.48" y="170.18" size="1.27" layer="97" align="bottom-center">GLVMS</text>
-<text x="68.58" y="144.78" size="1.27" layer="97" align="bottom-center">TSMS</text>
+<text x="104.14" y="144.78" size="1.27" layer="97" align="bottom-center">TSMS</text>
 <text x="124.46" y="144.78" size="1.27" layer="97" align="bottom-center">Right BRB</text>
 <text x="142.24" y="144.78" size="1.27" layer="97" align="bottom-center">Left BRB</text>
@@
 <text x="213.36" y="144.78" size="1.27" layer="97" align="bottom-center">Inertia Switch</text>
 <text x="17.78" y="170.18" size="1.27" layer="97" align="top-left">16AWG</text>
-<text x="91.44" y="142.24" size="1.27" layer="97" align="top-left">22AWG</text>
+<text x="68.58" y="142.24" size="1.27" layer="97" align="top-left">22AWG</text>
 <text x="127" y="142.24" size="1.27" layer="97" align="top-left">22AWG</text>
 <text x="147.32" y="142.24" size="1.27" layer="97" align="top-left">22AWG</text>
-<text x="109.22" y="142.24" size="1.27" layer="97" align="top-left">22AWG</text>
+<text x="91.44" y="142.24" size="1.27" layer="97" align="top-left">22AWG</text>
 <text x="200.66" y="142.24" size="1.27" layer="97" align="top-left">22AWG</text>
 <text x="60.96" y="160.02" size="1.27" layer="97" rot="R180" align="top-left">22AWG</text>
@@
 <wire x1="93.98" y1="78.74" x2="114.3" y2="78.74" width="0.1524" layer="94"/>
 <wire x1="114.3" y1="78.74" x2="114.3" y2="71.12" width="0.1524" layer="94"/>
-<wire x1="106.68" y1="50.8" x2="111.76" y2="50.8" width="0.1524" layer="94"/>
-<wire x1="111.76" y1="50.8" x2="111.76" y2="53.34" width="0.1524" layer="94"/>
+<wire x1="106.68" y1="50.8" x2="119.38" y2="50.8" width="0.1524" layer="94"/>
+<wire x1="119.38" y1="50.8" x2="119.38" y2="53.34" width="0.1524" layer="94"/>
 <wire x1="22.86" y1="182.88" x2="33.02" y2="182.88" width="0.1524" layer="94"/>
 <text x="7.62" y="182.88" size="1.778" layer="97" align="top-left">Direct
@@
 <instance part="MAIN_FUSE" gate="G$1" x="116.84" y="53.34" smashed="yes">
 <attribute name="NAME" x="118.11" y="54.61" size="1.27" layer="95" align="bottom-center"/>
-<attribute name="VALUE" x="115.57" y="52.07" size="1.27" layer="96" align="top-center"/>
+<attribute name="VALUE" x="116.84" y="52.324" size="1.27" layer="96" align="top-center"/>
 </instance>
 <instance part="U$17" gate="G$1" x="91.44" y="116.84" smashed="yes"/>
@@
 <attribute name="MPN" x="124.46" y="136.398" size="1.27" layer="96" rot="MR0" align="top-center"/>
 </instance>
-<instance part="S6" gate="SPST" x="88.9" y="139.7" smashed="yes" rot="MR0">
-<attribute name="MANUFACTURER" x="88.9" y="143.002" size="1.27" layer="96" rot="MR0" align="bottom-center"/>
-<attribute name="MPN" x="88.9" y="136.398" size="1.27" layer="96" rot="MR0" align="top-center"/>
-</instance>
-<instance part="S7" gate="SPST" x="106.68" y="139.7" smashed="yes" rot="MR0">
-<attribute name="MANUFACTURER" x="106.68" y="143.002" size="1.27" layer="96" rot="MR0" align="bottom-center"/>
-<attribute name="MPN" x="106.68" y="136.398" size="1.27" layer="96" rot="MR0" align="top-center"/>
-</instance>
-<instance part="S8" gate="SPST" x="68.58" y="139.7" smashed="yes" rot="MR0">
-<attribute name="MANUFACTURER" x="68.58" y="143.002" size="1.27" layer="96" rot="MR0" align="bottom-center"/>
-<attribute name="MPN" x="68.58" y="136.398" size="1.27" layer="96" rot="MR0" align="top-center"/>
+<instance part="S6" gate="SPST" x="66.04" y="139.7" smashed="yes" rot="MR0">
+<attribute name="MANUFACTURER" x="66.04" y="143.002" size="1.27" layer="96" rot="MR0" align="bottom-center"/>
+<attribute name="MPN" x="66.04" y="136.398" size="1.27" layer="96" rot="MR0" align="top-center"/>
+</instance>
+<instance part="S7" gate="SPST" x="83.82" y="139.7" smashed="yes" rot="MR0">
+<attribute name="MANUFACTURER" x="83.82" y="143.002" size="1.27" layer="96" rot="MR0" align="bottom-center"/>
+<attribute name="MPN" x="83.82" y="136.398" size="1.27" layer="96" rot="MR0" align="top-center"/>
+</instance>
+<instance part="S8" gate="SPST" x="104.14" y="139.7" smashed="yes" rot="MR0">
+<attribute name="MANUFACTURER" x="104.14" y="143.002" size="1.27" layer="96" rot="MR0" align="bottom-center"/>
+<attribute name="MPN" x="104.14" y="136.398" size="1.27" layer="96" rot="MR0" align="top-center"/>
 </instance>
 <instance part="S9" gate="SPST" x="30.48" y="165.1" smashed="yes">
@@
 </segment>
 </net>
-<net name="N$13" class="0">
-<segment>
-<pinref part="S5" gate="SPST" pin="O"/>
-<wire x1="119.38" y1="142.24" x2="119.38" y2="139.7" width="0.1524" layer="91"/>
-<pinref part="S7" gate="SPST" pin="P"/>
-<wire x1="119.38" y1="139.7" x2="111.76" y2="139.7" width="0.1524" layer="91"/>
-</segment>
-</net>
 <net name="GLV_SYSTEMS" class="0">
 <segment>
@@
 </segment>
 <segment>
-<wire x1="63.5" y1="139.7" x2="55.88" y2="139.7" width="0.1524" layer="91"/>
 <label x="55.88" y="139.7" size="1.27" layer="95" rot="R180" xref="yes"/>
 <pinref part="S8" gate="SPST" pin="S"/>
-<wire x1="63.5" y1="139.7" x2="63.5" y2="137.16" width="0.1524" layer="91"/>
+<wire x1="99.06" y1="139.7" x2="99.06" y2="137.16" width="0.1524" layer="91"/>
+<pinref part="S7" gate="SPST" pin="P"/>
+<wire x1="88.9" y1="139.7" x2="99.06" y2="139.7" width="0.1524" layer="91"/>
 </segment>
 <segment>
@@
 <segment>
 <pinref part="S6" gate="SPST" pin="S"/>
-<wire x1="83.82" y1="139.7" x2="83.82" y2="137.16" width="0.1524" layer="91"/>
-<pinref part="S8" gate="SPST" pin="P"/>
-<wire x1="83.82" y1="139.7" x2="73.66" y2="139.7" width="0.1524" layer="91"/>
+<wire x1="60.96" y1="139.7" x2="60.96" y2="137.16" width="0.1524" layer="91"/>
+<wire x1="60.96" y1="139.7" x2="55.88" y2="139.7" width="0.1524" layer="91"/>
 </segment>
 </net>
@@
 <segment>
 <pinref part="S7" gate="SPST" pin="S"/>
-<wire x1="101.6" y1="139.7" x2="101.6" y2="137.16" width="0.1524" layer="91"/>
+<wire x1="78.74" y1="139.7" x2="78.74" y2="137.16" width="0.1524" layer="91"/>
 <pinref part="S6" gate="SPST" pin="P"/>
-<wire x1="101.6" y1="139.7" x2="93.98" y2="139.7" width="0.1524" layer="91"/>
+<wire x1="78.74" y1="139.7" x2="71.12" y2="139.7" width="0.1524" layer="91"/>
 </segment>
 </net>
@@
 </segment>
 </net>
+<net name="N$30" class="0">
+<segment>
+<pinref part="S8" gate="SPST" pin="P"/>
+<pinref part="S5" gate="SPST" pin="O"/>
+<wire x1="119.38" y1="142.24" x2="119.38" y2="139.7" width="0.1524" layer="91"/>
+<wire x1="109.22" y1="139.7" x2="119.38" y2="139.7" width="0.1524" layer="91"/>
+</segment>
+</net>

Commit message: updates on things that are wrong
Parts:
- removed U2: LOGICGATE_INVERTER, HyTechSymbolsTemp:LOGICGATE_INVERTER
- added S14: SWITCH_SPST_, HyTechSymbols:SWITCH_SPST_
- DISCHARGE_RES, DISCHARGE_RES1, DISCHARGE_RES2: value 15k -> 20k
- PRECHARGE_RES, PRECHARGE_RES1: value 1.5k -> 3k
- S7: SPICEPREFIX (none) -> J
Connections:
- removed net N$25: U$17.PRECHARGE_OK, U2.IN
- removed net N$51: S6.P, S7.S
- new net N$13: S6.S, S7.P
- net N$21: now also S7.S; no longer S6.S
- net N$52: now also U$17.PRECHARGE_OK; no longer U2.!IN
- net SHDN: no longer S7.P
