File: ESF Schematics/2024/TSAL Schematic.sch (EAGLE design)
At the start: 25 parts, among them Q3 TRANSISTOR_N_MOS__PMV15ENEA, Q4 TRANSISTOR_N_MOS__PMV15ENEA, U1 ADG1423, U4 LM555

Commit message: Update TSAL Schematic.sch
Parts:
- removed U$1: 60V_THRESHOLD, HyTechSymbolsTemp:60V_THRESHOLD
- added R10, R9: 365k, HyTechSymbols:RESISTOR
- added R11: 3.3k, HyTechSymbols:RESISTOR
- added R12, R13, R14, R15, R7: (no value), HyTechSymbols:RESISTOR
- added R8: 1M, HyTechSymbols:RESISTOR
- added U2: ISO_224BDWVR, HyTechSymbols:ISO_224BDWVR
- added U3, U5: OPAMP, HyTechSymbols:OPAMP
Connections:
- removed net PACK+FUSED: U$1.PACK+
- new net N$10: R8.1, R9.2
- new net N$8: R10.1, R11.2, U2.IN
- new net N$9: R10.2, R9.1
- net +12V: no longer U$1.VDD
- net 60V_THRESHOLD: now also R7.2, U5.VOUT; no longer U$1.60V_THRESHOLD
- net GND: now also R7.1; no longer U$1.GND
- net TS+: now also R8.2; no longer U$1.TS+
- net TS-UNFUSED: now also R11.1; no longer U$1.TS-
Other:
- note removed: "22AWG"

Commit message: Update TSAL Schematic.sch
Parts:
- added R16: 10k, HyTechSymbols:RESISTOR
- added R17: 37.2k, HyTechSymbols:RESISTOR
- added R18: 1M, HyTechSymbols:RESISTOR
- added R19: 8.66k, HyTechSymbols:RESISTOR
- R12, R13: value (none) -> 18.7k
- R14, R15: value (none) -> 43k
- R7: value (none) -> 10k
Connections:
- new net +5V: R17.2
- new net ISO_TS+: R14.1, R16.2, U3.VOUT, U5.VIN+
- new net N$11: R13.1, R15.2, U3.VIN+
- new net N$12: R13.2, U2.OUTP
- new net N$13: R12.2, U2.OUTN
- new net N$14: R12.1, R14.2, U3.VIN-
- new net N$15: R17.1, R18.2, R19.2, U5.VIN-
- net GND: now also R15.1, R16.1, R18.1, R19.1
Other:
- note added: ".525V_DIV"
- note added: "22AWG"
- note added: "550V corresponds to 4.816V on ISO_TS+"
- note added: "Trips at 59.95V"
- moved on the sheet: R12, R13, R15, R7
