File: ESF Schematics/2024/Tractive System Schematic.sch (EAGLE design)
At the start: 38 parts, among them J1 CONNECTOR-1_CT2242-2, J10 CONNECTOR-3_1-2371113-2, J11 CONNECTOR-3_1-2371113-2, J12 CONNECTOR-1_LCAX2-14F-E, J13 CONNECTOR-3_1-2371113-2, J14 RING_TERMINAL_10MM2, J15 CONNECTOR-5_436500513, J16 CONNECTOR-2_HIROSE, J17 CONNECTOR-2_HIROSE, J18 RING_TERMINAL_10MM2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

Commit message: Update Tractive System Schematic.sch
Parts:
- DISCHARGE_RES, DISCHARGE_RES1, DISCHARGE_RES2: value 15k -> 20k
Changed lines of the file:
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@@
 <part name="J2" library="HyTechSymbolsTemp" deviceset="CONNECTOR-1_*" device="" technology="LCAX2-14F-E"/>
 <part name="U$4" library="HyTechFrames" deviceset="FRAME_SCHEMATIC_ONLY" device="">
-<attribute name="DESCRIPTION_1" value="ESF compliant representation of the HT07 "/>
+<attribute name="DESCRIPTION_1" value="ESF compliant representation of the HT08 "/>
 <attribute name="DESCRIPTION_2" value="tractive system."/>
 <attribute name="DESIGNER_SCHEMATIC" value="Liwei Sun"/>
-<attribute name="ENGINEER" value="Liwei Sun"/>
+<attribute name="ENGINEER" value="Shayan Noorani &amp; Liwei Sun"/>
 <attribute name="REVIEWER_SCHEMATIC" value="Zekun Li"/>
 </part>
@@
 <part name="DISCHARGE" library="HyTechSymbols" deviceset="RELAY_SPST_NC_?*" device="" technology="DBR72410" value="RELAY_SPST_NC_DBR72410"/>
 <part name="P13" library="HyTechSupplies" deviceset="GND" device=""/>
-<part name="DISCHARGE_RES" library="HyTechSymbolsTemp" deviceset="RESISTOR" device="" value="15k"/>
-<part name="DISCHARGE_RES1" library="HyTechSymbolsTemp" deviceset="RESISTOR" device="" value="15k"/>
-<part name="DISCHARGE_RES2" library="HyTechSymbolsTemp" deviceset="RESISTOR" device="" value="15k"/>
+<part name="DISCHARGE_RES" library="HyTechSymbolsTemp" deviceset="RESISTOR" device="" value="20k"/>
+<part name="DISCHARGE_RES1" library="HyTechSymbolsTemp" deviceset="RESISTOR" device="" value="20k"/>
+<part name="DISCHARGE_RES2" library="HyTechSymbolsTemp" deviceset="RESISTOR" device="" value="20k"/>
 <part name="J19" library="HyTechSymbols" deviceset="RING_TERMINAL_*" device="" technology="10MM2"/>
 <part name="J20" library="HyTechSymbols" deviceset="RING_TERMINAL_*" device="" technology="10MM2"/>
@@
 <attribute name="DRAWING_NAME" x="207.01" y="22.86" size="2.54" layer="95"/>
 <attribute name="SHEET" x="259.08" y="2.54" size="2.54" layer="95"/>
-<attribute name="ENGINEER" x="134.62" y="22.86" size="2.54" layer="95"/>
+<attribute name="ENGINEER" x="129.54" y="22.86" size="2.54" layer="96"/>
 <attribute name="DESIGNER_SCHEMATIC" x="179.07" y="30.48" size="2.54" layer="95"/>
 <attribute name="REVIEWER_SCHEMATIC" x="227.33" y="30.48" size="2.54" layer="95"/>

Commit message: More changes for ESF
Connections:
- removed net TS-UNFUSED: J15.1, J25.P$2
- new net N$16: J25.P$2
- new net N$3: J15.1
Changed lines of the file:
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@@
 <part name="R2" library="HyTechSymbols" deviceset="RESISTOR" device="" value="15k"/>
 <part name="P1" library="HyTechSupplies" deviceset="TS+UNFUSED" device=""/>
-<part name="P2" library="HyTechSupplies" deviceset="TS-UNFUSED" device=""/>
+<part name="P4" library="HyTechSupplies" deviceset="TS+UNFUSED" device=""/>
 <part name="P3" library="HyTechSupplies" deviceset="TS-UNFUSED" device=""/>
-<part name="P4" library="HyTechSupplies" deviceset="TS+UNFUSED" device=""/>
 </parts>
 <sheets>
@@
 <text x="236.22" y="81.28" size="1.27" layer="97" align="top-left">PCB Trace</text>
 <text x="223.52" y="101.6" size="1.27" layer="97" align="top-left">PCB Trace</text>
-<text x="124.46" y="96.52" size="1.27" layer="97" rot="R180" align="top-left">22AWG</text>
 <text x="116.84" y="119.38" size="1.27" layer="97" align="top-left">22AWG</text>
 <text x="147.32" y="147.32" size="1.27" layer="97">10mm^2</text>
 <text x="114.3" y="127" size="1.27" layer="97">10mm^2</text>
 <text x="144.78" y="66.04" size="1.27" layer="97" align="top-left">16AWG</text>
-<text x="119.38" y="83.82" size="1.27" layer="97">10mm^2</text>
+<text x="118.618" y="81.534" size="1.27" layer="97">10mm^2</text>
 <text x="198.12" y="91.44" size="1.27" layer="97" align="top-left">PCB Trace</text>
 <wire x1="180.34" y1="71.12" x2="180.34" y2="111.76" width="0.508" layer="97" style="shortdash"/>
@@
 <text x="147.32" y="198.12" size="1.27" layer="97">10mm^2</text>
 <text x="198.12" y="96.52" size="1.27" layer="97" align="top-left">PCB Trace</text>
-<text x="106.68" y="88.9" size="1.27" layer="97">10mm^2</text>
+<text x="104.14" y="86.36" size="1.27" layer="97">10mm^2</text>
 <text x="124.46" y="111.76" size="1.27" layer="97">10mm^2</text>
 <text x="129.54" y="71.12" size="1.27" layer="97">10mm^2</text>
@@
 <wire x1="101.6" y1="121.92" x2="101.6" y2="114.3" width="0.1524" layer="94"/>
 <wire x1="101.6" y1="114.3" x2="104.14" y2="114.3" width="0.1524" layer="94"/>
-<wire x1="111.76" y1="81.28" x2="111.76" y2="73.66" width="0.1524" layer="94"/>
+<wire x1="111.76" y1="88.9" x2="111.76" y2="73.66" width="0.1524" layer="94"/>
 <wire x1="111.76" y1="73.66" x2="99.06" y2="73.66" width="0.1524" layer="94"/>
 <wire x1="99.06" y1="76.2" x2="104.14" y2="76.2" width="0.1524" layer="94"/>
 <wire x1="99.06" y1="101.6" x2="104.14" y2="101.6" width="0.1524" layer="94"/>
-<wire x1="104.14" y1="101.6" x2="106.68" y2="101.6" width="0.1524" layer="94"/>
 <wire x1="104.14" y1="101.6" x2="104.14" y2="99.06" width="0.1524" layer="94"/>
 <wire x1="104.14" y1="81.28" x2="104.14" y2="76.2" width="0.1524" layer="94"/>
@@
 <text x="166.624" y="72.39" size="1.27" layer="97" rot="R90">130mm</text>
 <text x="197.104" y="14.986" size="2.54" layer="95">ESF compliant representation of the HT08</text>
+<wire x1="104.14" y1="101.6" x2="114.3" y2="101.6" width="0.1524" layer="94"/>
+<text x="124.46" y="89.154" size="1.27" layer="97" rot="R180" align="top-left">22AWG</text>
 </plain>
 <instances>
@@
 <attribute name="MPN" x="104.14" y="120.142" size="1.27" layer="96" align="top-left"/>
 </instance>
-<instance part="J25" gate="G$1" x="109.22" y="101.6" smashed="yes">
-<attribute name="MANUFACTURER" x="106.68" y="103.378" size="1.27" layer="96"/>
-<attribute name="MPN" x="106.68" y="99.822" size="1.27" layer="96" align="top-left"/>
+<instance part="J25" gate="G$1" x="114.3" y="88.9" smashed="yes">
+<attribute name="MANUFACTURER" x="111.76" y="90.678" size="1.27" layer="96"/>
+<attribute name="MPN" x="111.76" y="87.122" size="1.27" layer="96" align="top-left"/>
 </instance>
 <instance part="J26" gate="G$1" x="182.88" y="76.2" smashed="yes" rot="MR180">
@@
 <attribute name="VALUE" x="134.62" y="129.54" size="1.27" layer="96" align="bottom-center"/>
 </instance>
-<instance part="P2" gate="G$1" x="134.62" y="99.06" smashed="yes">
-<attribute name="VALUE" x="134.62" y="96.52" size="1.27" layer="96" align="top-center"/>
-</instance>
-<instance part="P3" gate="G$1" x="167.64" y="68.58" smashed="yes">
-<attribute name="VALUE" x="167.64" y="66.04" size="1.27" layer="96" align="top-center"/>
-</instance>
 <instance part="P4" gate="G$1" x="152.4" y="91.44" smashed="yes">
 <attribute name="VALUE" x="152.4" y="96.52" size="1.27" layer="96" align="bottom-center"/>
+</instance>
+<instance part="P3" gate="G$1" x="114.3" y="99.06" smashed="yes">
+<attribute name="VALUE" x="114.3" y="96.52" size="1.27" layer="96" align="top-center"/>
 </instance>
 </instances>
@@
 <pinref part="P4" gate="G$1" pin="TS+UNFUSED"/>
 <wire x1="167.64" y1="88.9" x2="152.4" y2="88.9" width="0.1524" layer="91"/>
-</segment>
-</net>
-<net name="TS-UNFUSED" class="0">
-<segment>
-<pinref part="J25" gate="G$1" pin="P$2"/>
-<pinref part="P2" gate="G$1" pin="TS-UNFUSED"/>
-<wire x1="111.76" y1="101.6" x2="134.62" y2="101.6" width="0.1524" layer="91"/>
-</segment>
-<segment>
-<pinref part="J15" gate="G$1" pin="1"/>
-<pinref part="P3" gate="G$1" pin="TS-UNFUSED"/>
-<wire x1="167.64" y1="78.74" x2="167.64" y2="71.12" width="0.1524" layer="91"/>
 </segment>
 </net>
@@
 <wire x1="116.84" y1="81.28" x2="127" y2="81.28" width="0.508" layer="91"/>
 <label x="127" y="81.28" size="1.27" layer="95" xref="yes"/>
+<label x="127" y="88.9" size="1.27" layer="95" xref="yes"/>
+<label x="167.64" y="71.12" size="1.27" layer="95" rot="R270" xref="yes"/>
 </segment>
 </net>
@@
 </segment>
 </net>
+<net name="N$3" class="0">
+<segment>
+<pinref part="J15" gate="G$1" pin="1"/>
+<wire x1="167.64" y1="78.74" x2="167.64" y2="71.12" width="0.1524" layer="91"/>
+</segment>
+</net>
+<net name="N$16" class="0">
+<segment>
+<pinref part="J25" gate="G$1" pin="P$2"/>
+<wire x1="116.84" y1="88.9" x2="127" y2="88.9" width="0.1524" layer="91"/>
+</segment>
+</net>
