File: EAGLE Board Designs/Accumulator Control Unit/Accumulator Control Unit rev6.sch (EAGLE design)
At the start: 263 parts, among them J1 CONNECTOR-12_MF_T_V_, J2 CONNECTOR-6_μF_T_V_BLACK, J3 CONNECTOR-4_μF_T_V_BLACK, J4 CONNECTOR-2_MF_T_V_, J5 CONNECTOR-8_μF_T_V_BLACK, J6 CONNECTOR-14_MF_T_V_, J7 JUMPER__1X02, J8 JUMPER__1X02, J9 CONNECTOR-2_MF_T_V_, Q1 TRANSISTOR_N_MOS__PMV15ENEA, Q2 TRANSISTOR_N_MOS__PMV15ENEA, Q3 TRANSISTOR_N_MOS__PMV15ENEA, Q4 TRANSISTOR_N_MOS__PMV15ENEA, T1 TRANSFORMER_HM2112ZNLT_AIRGAP, U1 VOLTAGE_REGULATOR_SOT-223_3.3V, U10 TCAN1051HQV-Q1, U11 OPAMP_1_CHANNEL_OPA991, U12 OPAMP_1_CHANNEL_OPA991, U13 OPAMP_1_CHANNEL_OPA991, U14 RELAY_SOLIDSTATE_NO_DIP-4, U15 LM555, U16 OPAMP_1_CHANNEL_OPA991, U17 MAX7404, U18 OPAMP_1_CHANNEL_OPA991, U19 MAX7404, U2 RELAY_SOLIDSTATE_NO_DIP-4, U20 LOGICGATE_BUFFER, U21 ADM8316WBX30, U22 OPAMP_1_CHANNEL_OPA991, U23 LOGICGATE_AND_DCK3, U24 LOGICGATE_AND_DCK3, U25 LOGICGATE_AND_DCK3, U26 OPAMP_1_CHANNEL_OPA991, U27 ADG1423, U28 OPAMP_1_CHANNEL_OPA991, U29 MAX7404, U3 RELAY_SOLIDSTATE_NO_DIP-4, U30 OPAMP_1_CHANNEL_OPA991, U31 MAX7404, U32 LTC6820, U33 OPAMP_1_CHANNEL_OPA991, U4 OPAMP_1_CHANNEL_OPA991, U5 OPAMP_1_CHANNEL_OPA991, U6 TCAN1051HQV-Q1, U7 LTC6820, U8 OPAMP_1_CHANNEL_OPA991, U9 OPAMP_1_CHANNEL_OPA991

Commit message: yum
Parts:
- removed J7, J8: JUMPER__1X02, HyTechDevices:JUMPER__1X02
Connections:
- removed net CANH/1.3B: J7.2, R27.2
- removed net N$35: J8.2, R51.2
- net CANH: now also R27.2; no longer J7.1
- net EM_CANH: now also R51.2; no longer J8.1
Other:
- moved on the sheet: R51
Changed lines of the file:
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@@
 <part name="P108" library="HyTechSupplies" deviceset="GND" device=""/>
 <part name="C12" library="HyTechDevices" deviceset="CAPACITOR_?_*" device="0603" technology="10V_4.7NF"/>
-<part name="J7" library="HyTechDevices" deviceset="JUMPER_?_*" device="" technology="1X02" value="JUMPER__1X02"/>
 <part name="F2" library="HyTechDevices" deviceset="FUSE_?_*" device="0603" technology=".75A"/>
 <part name="F1" library="HyTechDevices" deviceset="FUSE_?_*" device="0603" technology=".75A"/>
@@
 <part name="P119" library="HyTechSupplies" deviceset="GND" device=""/>
 <part name="C21" library="HyTechDevices" deviceset="CAPACITOR_?_*" device="0603" technology="10V_4.7NF"/>
-<part name="J8" library="HyTechDevices" deviceset="JUMPER_?_*" device="" technology="1X02" value="JUMPER__1X02"/>
 <part name="P120" library="HyTechSupplies" deviceset="+3V3" device=""/>
 <part name="C20" library="HyTechDevices" deviceset="CAPACITOR_?_*" device="0603" technology="10V_0.1UF"/>
@@
 <attribute name="CAPACITANCE" x="104.902" y="102.87" size="1.27" layer="96" rot="R270" align="top-center"/>
 </instance>
-<instance part="J7" gate="G$1" x="119.38" y="119.38" smashed="yes" rot="R270">
-<attribute name="NAME" x="116.84" y="116.84" size="1.27" layer="95" rot="R270" align="bottom-center"/>
-<attribute name="MPN" x="123.698" y="119.38" size="1.27" layer="96" rot="R270" align="top-left"/>
-</instance>
 <instance part="U20" gate="A" x="246.38" y="88.9" smashed="yes">
 <attribute name="NAME" x="248.793" y="91.948" size="1.27" layer="95"/>
@@
 <attribute name="RESISTANCE" x="128.27" y="59.69" size="1.27" layer="96" rot="R90" align="top-center"/>
 </instance>
-<instance part="R51" gate="G$1" x="137.16" y="60.96" smashed="yes" rot="R90">
-<attribute name="NAME" x="135.89" y="59.69" size="1.27" layer="95" rot="R90" align="bottom-center"/>
-<attribute name="RESISTANCE" x="138.43" y="59.69" size="1.27" layer="96" rot="R90" align="top-center"/>
+<instance part="R51" gate="G$1" x="142.24" y="60.96" smashed="yes" rot="R90">
+<attribute name="NAME" x="140.97" y="59.69" size="1.27" layer="95" rot="R90" align="bottom-center"/>
+<attribute name="RESISTANCE" x="143.51" y="59.69" size="1.27" layer="96" rot="R90" align="top-center"/>
 </instance>
 <instance part="P119" gate="1" x="132.08" y="43.18" smashed="yes">
@@
 <attribute name="CAPACITANCE" x="127.762" y="52.07" size="1.27" layer="96" rot="R270" align="top-center"/>
 </instance>
-<instance part="J8" gate="G$1" x="144.78" y="68.58" smashed="yes" rot="R270">
-<attribute name="NAME" x="142.24" y="66.04" size="1.27" layer="95" rot="R270" align="bottom-center"/>
-<attribute name="MPN" x="149.098" y="68.58" size="1.27" layer="96" rot="R270" align="top-left"/>
-</instance>
 <instance part="P120" gate="G$1" x="144.78" y="91.44" smashed="yes">
 <attribute name="VALUE" x="144.78" y="92.71" size="1.27" layer="96" align="bottom-center"/>
@@
 </segment>
 </net>
-<net name="CANH/1.3B" class="0">
-<segment>
-<pinref part="R27" gate="G$1" pin="2"/>
-<pinref part="J7" gate="G$1" pin="2"/>
-</segment>
-</net>
 <net name="N$21" class="0">
 <segment>
@@
 <segment>
 <pinref part="U6" gate="G$1" pin="CANH"/>
-<pinref part="J7" gate="G$1" pin="1"/>
 <label x="127" y="121.92" size="1.27" layer="95" xref="yes"/>
 <wire x1="101.6" y1="121.92" x2="116.84" y2="121.92" width="0.1524" layer="91"/>
-<wire x1="116.84" y1="121.92" x2="116.84" y2="119.38" width="0.1524" layer="91"/>
 <wire x1="116.84" y1="121.92" x2="127" y2="121.92" width="0.1524" layer="91"/>
 <junction x="116.84" y="121.92"/>
+<pinref part="R27" gate="G$1" pin="2"/>
+<wire x1="116.84" y1="114.3" x2="116.84" y2="121.92" width="0.1524" layer="91"/>
 </segment>
 </net>
@@
 <pinref part="R51" gate="G$1" pin="1"/>
 <pinref part="C21" gate="G$1" pin="2"/>
-<wire x1="132.08" y1="55.88" x2="137.16" y2="55.88" width="0.1524" layer="91"/>
+<wire x1="132.08" y1="55.88" x2="142.24" y2="55.88" width="0.1524" layer="91"/>
 <junction x="132.08" y="55.88"/>
 </segment>
 </net>
-<net name="N$35" class="0">
-<segment>
-<pinref part="R51" gate="G$1" pin="2"/>
-<pinref part="J8" gate="G$1" pin="2"/>
-<wire x1="142.24" y1="63.5" x2="137.16" y2="63.5" width="0.1524" layer="91"/>
-</segment>
-</net>
 <net name="EM_CANH" class="0">
 <segment>
 <pinref part="U10" gate="G$1" pin="CANH"/>
 <wire x1="121.92" y1="76.2" x2="142.24" y2="76.2" width="0.1524" layer="91"/>
-<pinref part="J8" gate="G$1" pin="1"/>
-<wire x1="142.24" y1="76.2" x2="142.24" y2="68.58" width="0.1524" layer="91"/>
+<wire x1="142.24" y1="76.2" x2="142.24" y2="63.5" width="0.1524" layer="91"/>
 <label x="142.24" y="76.2" size="1.27" layer="95" xref="yes"/>
+<pinref part="R51" gate="G$1" pin="2"/>
 </segment>
 </net>

Commit message: Replaced iso_TS and iso_Pack processing resistors
Parts:
- R33, R34, R37, R38: value RESISTOR_0603_10.5K -> RESISTOR_0603_18.7K_LT; device HyTechDevices:RESISTOR_0603_10.5K -> HyTechDevices:RESISTOR_0603_18.7K_LT
- R35, R36, R39, R40: value RESISTOR_0603_13K -> RESISTOR_0603_43K_LT; device HyTechDevices:RESISTOR_0603_13K -> HyTechDevices:RESISTOR_0603_43K_LT
Changed lines of the file:
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@@
 <part name="P114" library="HyTechSupplies" deviceset="GND" device=""/>
 <part name="C37" library="HyTechDevices" deviceset="CAPACITOR_?_*" device="0603" technology="10V_0.1UF"/>
-<part name="R39" library="HyTechDevices" deviceset="RESISTOR_?_*" device="0603" technology="13K"/>
-<part name="R40" library="HyTechDevices" deviceset="RESISTOR_?_*" device="0603" technology="13K"/>
-<part name="R37" library="HyTechDevices" deviceset="RESISTOR_?_*" device="0603" technology="10.5K"/>
-<part name="R38" library="HyTechDevices" deviceset="RESISTOR_?_*" device="0603" technology="10.5K"/>
-<part name="R36" library="HyTechDevices" deviceset="RESISTOR_?_*" device="0603" technology="13K"/>
-<part name="R35" library="HyTechDevices" deviceset="RESISTOR_?_*" device="0603" technology="13K"/>
-<part name="R33" library="HyTechDevices" deviceset="RESISTOR_?_*" device="0603" technology="10.5K"/>
-<part name="R34" library="HyTechDevices" deviceset="RESISTOR_?_*" device="0603" technology="10.5K"/>
+<part name="R39" library="HyTechDevices" deviceset="RESISTOR_?_*" device="0603" technology="43K_LT" value="RESISTOR_0603_43K_LT"/>
+<part name="R40" library="HyTechDevices" deviceset="RESISTOR_?_*" device="0603" technology="43K_LT" value="RESISTOR_0603_43K_LT"/>
+<part name="R37" library="HyTechDevices" deviceset="RESISTOR_?_*" device="0603" technology="18.7K_LT" value="RESISTOR_0603_18.7K_LT"/>
+<part name="R38" library="HyTechDevices" deviceset="RESISTOR_?_*" device="0603" technology="18.7K_LT" value="RESISTOR_0603_18.7K_LT"/>
+<part name="R36" library="HyTechDevices" deviceset="RESISTOR_?_*" device="0603" technology="43K_LT" value="RESISTOR_0603_43K_LT"/>
+<part name="R35" library="HyTechDevices" deviceset="RESISTOR_?_*" device="0603" technology="43K_LT" value="RESISTOR_0603_43K_LT"/>
+<part name="R33" library="HyTechDevices" deviceset="RESISTOR_?_*" device="0603" technology="18.7K_LT" value="RESISTOR_0603_18.7K_LT"/>
+<part name="R34" library="HyTechDevices" deviceset="RESISTOR_?_*" device="0603" technology="18.7K_LT" value="RESISTOR_0603_18.7K_LT"/>
 <part name="P115" library="HyTechSupplies" deviceset="GND" device=""/>
 <part name="U10" library="HyTechDevices" deviceset="TCAN1051*V-Q1" device="" technology="HQ"/>

Commit message: changed pins to have a can in and out
Parts:
- J6: value CONNECTOR-14_MF_T_V_ -> CONNECTOR-16_MF_T_V_; device HyTechDevices:CONNECTOR-14_MF_T_V_ -> HyTechDevices:CONNECTOR-16_MF_T_V_
Connections:
- net BSPD_CURRENT: now also J6.14; no longer J6.10
- net BSPD_CURRENT_REF: now also J6.13; no longer J6.11
- net CANH: now also J6.11, J6.3; no longer J6.9
- net CANL: now also J6.12, J6.4; no longer J6.8
- net CHASSIS_GND: now also J6.16; no longer J6.13
- net GND: now also J6.15; no longer J6.12
- net N$28: now also J6.10; no longer J6.3
- net N$31: now also J6.9; no longer J6.4
Other:
- moved on the sheet: F1, F2
Changed lines of the file:
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@@
 <part name="D1" library="HyTechDevices" deviceset="TVS_?_*" device="" technology="8V"/>
 <part name="P5" library="HyTechSupplies" deviceset="GND" device=""/>
-<part name="J6" library="HyTechDevices" deviceset="CONNECTOR-14_?_*" device="MF_T_V"/>
+<part name="J6" library="HyTechDevices" deviceset="CONNECTOR-16_?_*" device="MF_T_V"/>
 <part name="R3" library="HyTechDevices" deviceset="RESISTOR_?_*" device="0603" technology="20K" value="RESISTOR_0603_20K"/>
 <part name="GND5" library="supply1" deviceset="GND" device=""/>
@@
 <attribute name="MPN" x="129.54" y="189.738" size="1.27" layer="96" align="top-center"/>
 </instance>
-<instance part="F2" gate="G$1" x="76.2" y="180.34" smashed="yes">
-<attribute name="NAME" x="74.93" y="181.61" size="1.27" layer="95" align="bottom-center"/>
-<attribute name="CURRENT" x="74.93" y="179.07" size="1.27" layer="96" align="top-center"/>
-</instance>
-<instance part="F1" gate="G$1" x="83.82" y="177.8" smashed="yes">
-<attribute name="NAME" x="82.55" y="179.07" size="1.27" layer="95" align="bottom-center"/>
-<attribute name="CURRENT" x="82.55" y="176.53" size="1.27" layer="96" align="top-center"/>
+<instance part="F2" gate="G$1" x="76.2" y="162.56" smashed="yes">
+<attribute name="NAME" x="74.93" y="163.83" size="1.27" layer="95" align="bottom-center"/>
+<attribute name="CURRENT" x="74.93" y="161.29" size="1.27" layer="96" align="top-center"/>
+</instance>
+<instance part="F1" gate="G$1" x="76.2" y="165.1" smashed="yes">
+<attribute name="NAME" x="74.93" y="166.37" size="1.27" layer="95" align="bottom-center"/>
+<attribute name="CURRENT" x="74.93" y="163.83" size="1.27" layer="96" align="top-center"/>
 </instance>
 <instance part="A1" gate="G$1" x="109.22" y="160.02" smashed="yes">
@@
 <attribute name="VALUE" x="43.18" y="121.92" size="1.27" layer="96" align="bottom-center"/>
 </instance>
-<instance part="P115" gate="1" x="93.98" y="154.94" smashed="yes">
-<attribute name="VALUE" x="93.98" y="153.67" size="1.27" layer="96" align="top-center"/>
+<instance part="P115" gate="1" x="94.996" y="146.05" smashed="yes">
+<attribute name="VALUE" x="94.996" y="144.78" size="1.27" layer="96" align="top-center"/>
 </instance>
 <instance part="J3" gate="G$1" x="12.7" y="195.58" smashed="yes">
@@
 <net name="CANH" class="0">
 <segment>
-<wire x1="68.58" y1="165.1" x2="71.12" y2="165.1" width="0.1524" layer="91"/>
-<label x="71.12" y="165.1" size="1.27" layer="95" xref="yes"/>
-<pinref part="J6" gate="G$1" pin="9"/>
+<pinref part="J6" gate="G$1" pin="11"/>
+<wire x1="68.58" y1="160.02" x2="71.12" y2="160.02" width="0.1524" layer="91"/>
+<label x="71.12" y="160.02" size="1.27" layer="95" xref="yes"/>
+</segment>
+<segment>
+<pinref part="J6" gate="G$1" pin="3"/>
+<wire x1="68.58" y1="180.34" x2="70.866" y2="180.34" width="0.1524" layer="91"/>
+<label x="71.12" y="180.34" size="1.27" layer="95" xref="yes"/>
 </segment>
 </net>
 <net name="CANL" class="0">
 <segment>
-<wire x1="68.58" y1="167.64" x2="71.12" y2="167.64" width="0.1524" layer="91"/>
-<label x="71.12" y="167.64" size="1.27" layer="95" xref="yes"/>
-<pinref part="J6" gate="G$1" pin="8"/>
+<pinref part="J6" gate="G$1" pin="4"/>
+<wire x1="68.58" y1="177.8" x2="71.12" y2="177.8" width="0.1524" layer="91"/>
+<label x="71.12" y="177.8" size="1.27" layer="95" xref="yes"/>
+</segment>
+<segment>
+<pinref part="J6" gate="G$1" pin="12"/>
+<wire x1="68.58" y1="157.48" x2="71.12" y2="157.48" width="0.1524" layer="91"/>
+<label x="71.12" y="157.48" size="1.27" layer="95" xref="yes"/>
 </segment>
 </net>
@@
 </segment>
 <segment>
-<pinref part="J6" gate="G$1" pin="12"/>
-<pinref part="P115" gate="1" pin="GND"/>
-<wire x1="68.58" y1="157.48" x2="93.98" y2="157.48" width="0.1524" layer="91"/>
-</segment>
-<segment>
 <pinref part="CURRENT_SHUNT" gate="G$1" pin="4"/>
 <wire x1="17.78" y1="15.24" x2="22.86" y2="15.24" width="0.1524" layer="91"/>
 <pinref part="P131" gate="1" pin="GND"/>
 <wire x1="22.86" y1="15.24" x2="22.86" y2="12.7" width="0.1524" layer="91"/>
+</segment>
+<segment>
+<pinref part="J6" gate="G$1" pin="15"/>
+<wire x1="68.58" y1="149.86" x2="94.996" y2="149.86" width="0.1524" layer="91"/>
+<pinref part="P115" gate="1" pin="GND"/>
+<wire x1="94.996" y1="149.86" x2="94.996" y2="148.59" width="0.1524" layer="91"/>
 </segment>
 </net>
@@
 <net name="BSPD_CURRENT" class="0">
 <segment>
-<wire x1="68.58" y1="162.56" x2="71.12" y2="162.56" width="0.1524" layer="91"/>
-<label x="71.12" y="162.56" size="1.27" layer="95" xref="yes"/>
-<pinref part="J6" gate="G$1" pin="10"/>
+<label x="71.12" y="152.4" size="1.27" layer="95" xref="yes"/>
+<pinref part="J6" gate="G$1" pin="14"/>
+<wire x1="68.58" y1="152.4" x2="71.12" y2="152.4" width="0.1524" layer="91"/>
 </segment>
 </net>
@@
 <segment>
 <pinref part="F1" gate="G$1" pin="2"/>
-<wire x1="86.36" y1="177.8" x2="88.9" y2="177.8" width="0.1524" layer="91"/>
-<label x="88.9" y="177.8" size="1.27" layer="95" xref="yes"/>
+<wire x1="78.74" y1="165.1" x2="86.36" y2="165.1" width="0.1524" layer="91"/>
+<label x="86.36" y="165.1" size="1.27" layer="95" xref="yes"/>
 </segment>
 </net>
@@
 <segment>
 <pinref part="F2" gate="G$1" pin="2"/>
-<wire x1="78.74" y1="180.34" x2="88.9" y2="180.34" width="0.1524" layer="91"/>
-<label x="88.9" y="180.34" size="1.27" layer="95" xref="yes"/>
+<wire x1="78.74" y1="162.56" x2="86.36" y2="162.56" width="0.1524" layer="91"/>
+<label x="86.36" y="162.56" size="1.27" layer="95" xref="yes"/>
 </segment>
 </net>
@@
 </segment>
 <segment>
-<pinref part="J6" gate="G$1" pin="13"/>
-<wire x1="68.58" y1="154.94" x2="76.2" y2="154.94" width="0.1524" layer="91"/>
-<label x="76.2" y="154.94" size="1.27" layer="95" xref="yes"/>
+<label x="76.2" y="147.32" size="1.27" layer="95" xref="yes"/>
+<pinref part="J6" gate="G$1" pin="16"/>
+<wire x1="68.58" y1="147.32" x2="76.2" y2="147.32" width="0.1524" layer="91"/>
 </segment>
 </net>
@@
 </segment>
 </net>
-<net name="N$28" class="0">
-<segment>
-<pinref part="J6" gate="G$1" pin="3"/>
-<wire x1="68.58" y1="180.34" x2="71.12" y2="180.34" width="0.1524" layer="91"/>
-<pinref part="F2" gate="G$1" pin="1"/>
-</segment>
-</net>
-<net name="N$31" class="0">
-<segment>
-<pinref part="J6" gate="G$1" pin="4"/>
-<wire x1="68.58" y1="177.8" x2="78.74" y2="177.8" width="0.1524" layer="91"/>
-<pinref part="F1" gate="G$1" pin="1"/>
-</segment>
-</net>
 <net name="+24V" class="0">
 <segment>
@@
 <net name="BSPD_CURRENT_REF" class="0">
 <segment>
-<pinref part="J6" gate="G$1" pin="11"/>
-<wire x1="68.58" y1="160.02" x2="71.12" y2="160.02" width="0.1524" layer="91"/>
-<label x="71.12" y="160.02" size="1.27" layer="95" xref="yes"/>
+<label x="71.12" y="154.94" size="1.27" layer="95" xref="yes"/>
+<pinref part="J6" gate="G$1" pin="13"/>
+<wire x1="68.58" y1="154.94" x2="71.12" y2="154.94" width="0.1524" layer="91"/>
 </segment>
 </net>
@@
 </segment>
 </net>
+<net name="N$28" class="0">
+<segment>
+<pinref part="J6" gate="G$1" pin="10"/>
+<pinref part="F2" gate="G$1" pin="1"/>
+<wire x1="68.58" y1="162.56" x2="71.12" y2="162.56" width="0.1524" layer="91"/>
+</segment>
+</net>
+<net name="N$31" class="0">
+<segment>
+<pinref part="J6" gate="G$1" pin="9"/>
+<pinref part="F1" gate="G$1" pin="1"/>
+<wire x1="68.58" y1="165.1" x2="71.12" y2="165.1" width="0.1524" layer="91"/>
+</segment>
+</net>

Commit message: changed some stuff to make it look better
Connections:
- net N$28: now also F1.1; no longer F2.1
- net N$31: now also F2.1; no longer F1.1
Other:
- moved on the sheet: A1, C1, C2, F1, F2, J6

Commit message: num num num
Connections:
- net PRECHARGE_OK_TEENSY: now also A3.D4; no longer A3.D2
Other:
- moved on the sheet: WATCHDOG_INPUT
Changed lines of the file:
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@@
 <attribute name="CAPACITANCE" x="135.89" y="198.882" size="1.27" layer="96" align="top-center"/>
 </instance>
-<instance part="WATCHDOG_INPUT" gate="G$1" x="81.28" y="167.64" smashed="yes" rot="R180">
-<attribute name="NAME" x="83.82" y="166.878" size="1.27" layer="95"/>
-<attribute name="MPN" x="78.74" y="166.878" size="1.27" layer="95" rot="R180" align="top-left"/>
+<instance part="WATCHDOG_INPUT" gate="G$1" x="86.36" y="170.18" smashed="yes" rot="R180">
+<attribute name="NAME" x="88.9" y="169.418" size="1.27" layer="95"/>
+<attribute name="MPN" x="83.82" y="169.418" size="1.27" layer="95" rot="R180" align="top-left"/>
 </instance>
 <instance part="WATCHDOG" gate="LED" x="185.42" y="66.04" smashed="yes">
@@
 </segment>
 <segment>
-<pinref part="A3" gate="G$1" pin="D2"/>
-<wire x1="68.58" y1="162.56" x2="71.12" y2="162.56" width="0.1524" layer="91"/>
-<label x="71.12" y="162.56" size="1.27" layer="95" xref="yes"/>
+<label x="71.12" y="167.64" size="1.27" layer="95" xref="yes"/>
+<pinref part="A3" gate="G$1" pin="D4"/>
+<wire x1="68.58" y1="167.64" x2="71.12" y2="167.64" width="0.1524" layer="91"/>
 </segment>
 </net>
@@
 </segment>
 <segment>
-<label x="83.82" y="170.18" size="1.27" layer="95" xref="yes"/>
+<label x="106.68" y="170.18" size="1.27" layer="95" xref="yes"/>
 <pinref part="WATCHDOG_INPUT" gate="G$1" pin="P$1"/>
 <wire x1="78.74" y1="170.18" x2="83.82" y2="170.18" width="0.1524" layer="91"/>
-<wire x1="78.74" y1="170.18" x2="78.74" y2="167.64" width="0.1524" layer="91"/>
 <pinref part="A3" gate="G$1" pin="D5"/>
 <wire x1="68.58" y1="170.18" x2="78.74" y2="170.18" width="0.1524" layer="91"/>
