File: EAGLE Board Designs/Sensor Acquisition Board/Sensor Acquisition Board Rev5.sch (EAGLE design)
At the start: 123 parts, among them J1 CONNECTOR-8_μF_T_V_BLACK, J10 CONNECTOR-10_MF_T_V_, J11 CONNECTOR-2_MICROFIT_SMD_RIGH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, J12 CONNECTOR-6_μF_T_V_BLACK, J13 CONNECTOR-4_μF_T_V_BLACK, J14 CONNECTOR-8_μF_T_V_BLACK, J15 CONNECTOR-4_μF_T_V_BLACK, J16 CONNECTOR-8_μF_T_V_BLACK, J2 CONNECTOR-4_μF_T_V_BLACK, J3 CONNECTOR-4_μF_T_V_BLACK, J4 CONNECTOR-4_μF_S_RA_, J5 CONNECTOR-4_μF_S_RA_, J6 CONNECTOR-8_μF_T_V_BLACK, J7 CONNECTOR-4_μF_T_V_BLACK, J8 CONNECTOR-2_μF_T_V_BLACK, J9 CONNECTOR-4_μF_S_RA_, T1 78613/3C_78613/3C, T2 78613/3C_78613/3C, U1 VOLTAGE_REGULATOR_SOT-223_3.3V, U10 MAX3227, U11 LTC6820, U12 LTC6820, U13 TCAN1051HQV-Q1, U14 MAX3075, U15 MCP3208

Commit message: some schematic changes and routes
Parts:
- removed D5: SCHOTTKY_1206_40V, HyTechDevices:SCHOTTKY_1206_40V
Connections:
- removed net N$44: D5.C, D6.C, XF1.1
- net +24V: now also J16.4; no longer J16.1
- net +5V: now also J16.3; no longer J16.2
- net 24VIN: now also D6.C, XF1.1; no longer D5.A
- net GND: now also J16.1; no longer J16.4
- net RR_EXT_N: now also J16.6; no longer J16.8
- net RR_EXT_P: now also J16.5; no longer J16.7
- net SHDN_K: now also J16.7; no longer J16.5
- net SHDN_L: now also J16.8; no longer J16.6
- net THERM1: now also J6.8; no longer J1.7
- net THERM2: now also J6.7; no longer J1.6
- net THERM3: now also J6.6; no longer J1.5
- net THERM4: now also J6.5; no longer J1.8
- net THERM5: now also J1.8; no longer J6.7
- net THERM6: now also J1.7; no longer J6.6
- net THERM7: now also J1.6; no longer J6.5
- net THERM8: now also J1.5; no longer J6.8

Commit message: final change
Connections:
- net SHDN_L: now also J16.2; no longer J16.8
Changed lines of the file:
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@@
 </segment>
 <segment>
-<pinref part="J16" gate="G$1" pin="8"/>
-<wire x1="246.38" y1="78.74" x2="256.54" y2="78.74" width="0.1524" layer="91"/>
+<pinref part="J16" gate="G$1" pin="2"/>
+<wire x1="246.38" y1="93.98" x2="248.92" y2="93.98" width="0.1524" layer="91"/>
+<wire x1="248.92" y1="93.98" x2="248.92" y2="78.74" width="0.1524" layer="91"/>
+<wire x1="248.92" y1="78.74" x2="256.54" y2="78.74" width="0.1524" layer="91"/>
 <label x="256.54" y="78.74" size="1.27" layer="95" xref="yes"/>
 </segment>

Commit message: review changes
Connections:
- removed net SHDN_J: J12.4, J14.7
- new net SHDN_M: J12.5, J16.2
- net SHDN_K: now also J12.4, J14.7; no longer J14.8, J16.7
- net SHDN_L: now also J14.8, J16.7; no longer J12.5, J16.2
Changed lines of the file:
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@@
 <net name="SHDN_K" class="0">
-<segment>
-<pinref part="J14" gate="G$1" pin="8"/>
-<wire x1="198.12" y1="78.74" x2="208.28" y2="78.74" width="0.1524" layer="91"/>
-<label x="208.28" y="78.74" size="1.27" layer="95" xref="yes"/>
-</segment>
-<segment>
-<pinref part="J16" gate="G$1" pin="7"/>
-<wire x1="246.38" y1="81.28" x2="256.54" y2="81.28" width="0.1524" layer="91"/>
-<label x="256.54" y="81.28" size="1.27" layer="95" xref="yes"/>
-</segment>
-</net>
-<net name="SHDN_J" class="0">
 <segment>
 <pinref part="J12" gate="G$1" pin="4"/>
@@
 </segment>
 </net>
-<net name="SHDN_L" class="0">
+<net name="SHDN_M" class="0">
 <segment>
 <pinref part="J12" gate="G$1" pin="5"/>
@@
 </segment>
 </net>
+<net name="SHDN_L" class="0">
+<segment>
+<pinref part="J14" gate="G$1" pin="8"/>
+<wire x1="198.12" y1="78.74" x2="208.28" y2="78.74" width="0.1524" layer="91"/>
+<label x="208.28" y="78.74" size="1.27" layer="95" xref="yes"/>
+</segment>
+<segment>
+<pinref part="J16" gate="G$1" pin="7"/>
+<wire x1="246.38" y1="81.28" x2="256.54" y2="81.28" width="0.1524" layer="91"/>
+<label x="256.54" y="81.28" size="1.27" layer="95" xref="yes"/>
+</segment>
+</net>

Commit message: swapped rs232 and rs485 caps for higher voltage ratings
Parts:
- C48, C49, C50, C51, C52: value CAPACITOR_0603_25V_0.1UF -> CAPACITOR_0603_35V_0.1UF; device HyTechDevices:CAPACITOR_0603_25V_0.1UF -> HyTechDevices:CAPACITOR_0603_35V_0.1UF
- C53, C64: value CAPACITOR_0603_10V_1UF -> CAPACITOR_0603_35V_1UF; device HyTechDevices:CAPACITOR_0603_10V_1UF -> HyTechDevices:CAPACITOR_0603_35V_1UF
- C62: value CAPACITOR_0603_10V_0.1UF -> CAPACITOR_0603_35V_0.1UF; device HyTechDevices:CAPACITOR_0603_10V_0.1UF -> HyTechDevices:CAPACITOR_0603_35V_0.1UF
Changed lines of the file:
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@@
 <part name="P112" library="HyTechSupplies" deviceset="GND" device=""/>
 <part name="P115" library="HyTechSupplies" deviceset="GND" device=""/>
-<part name="C62" library="HyTechDevices" deviceset="CAPACITOR_?_*" device="0603" technology="10V_0.1UF"/>
-<part name="C64" library="HyTechDevices" deviceset="CAPACITOR_?_*" device="0603" technology="10V_1UF"/>
+<part name="C62" library="HyTechDevices" deviceset="CAPACITOR_?_*" device="0603" technology="35V_0.1UF" value="CAPACITOR_0603_35V_0.1UF"/>
+<part name="C64" library="HyTechDevices" deviceset="CAPACITOR_?_*" device="0603" technology="35V_1UF" value="CAPACITOR_0603_35V_1UF"/>
 <part name="R21" library="HyTechDevices" deviceset="RESISTOR_?_*" device="0603" technology="60.4"/>
 <part name="R22" library="HyTechDevices" deviceset="RESISTOR_?_*" device="0603" technology="60.4"/>
@@
 <part name="P1" library="HyTechSupplies" deviceset="GND" device=""/>
 <part name="P14" library="HyTechSupplies" deviceset="+3V3" device=""/>
-<part name="C48" library="HyTechDevices" deviceset="CAPACITOR_?_*" device="0603" technology="25V_0.1UF"/>
-<part name="C49" library="HyTechDevices" deviceset="CAPACITOR_?_*" device="0603" technology="25V_0.1UF"/>
-<part name="C50" library="HyTechDevices" deviceset="CAPACITOR_?_*" device="0603" technology="25V_0.1UF"/>
-<part name="C51" library="HyTechDevices" deviceset="CAPACITOR_?_*" device="0603" technology="25V_0.1UF"/>
+<part name="C48" library="HyTechDevices" deviceset="CAPACITOR_?_*" device="0603" technology="35V_0.1UF" value="CAPACITOR_0603_35V_0.1UF"/>
+<part name="C49" library="HyTechDevices" deviceset="CAPACITOR_?_*" device="0603" technology="35V_0.1UF" value="CAPACITOR_0603_35V_0.1UF"/>
+<part name="C50" library="HyTechDevices" deviceset="CAPACITOR_?_*" device="0603" technology="35V_0.1UF" value="CAPACITOR_0603_35V_0.1UF"/>
+<part name="C51" library="HyTechDevices" deviceset="CAPACITOR_?_*" device="0603" technology="35V_0.1UF" value="CAPACITOR_0603_35V_0.1UF"/>
 <part name="P15" library="HyTechSupplies" deviceset="+3V3" device=""/>
 <part name="P24" library="HyTechSupplies" deviceset="GND" device=""/>
 <part name="P26" library="HyTechSupplies" deviceset="+3V3" device=""/>
-<part name="C52" library="HyTechDevices" deviceset="CAPACITOR_?_*" device="0603" technology="25V_0.1UF"/>
+<part name="C52" library="HyTechDevices" deviceset="CAPACITOR_?_*" device="0603" technology="35V_0.1UF" value="CAPACITOR_0603_35V_0.1UF"/>
 <part name="P27" library="HyTechSupplies" deviceset="GND" device=""/>
-<part name="C53" library="HyTechDevices" deviceset="CAPACITOR_?_*" device="0603" technology="10V_1UF"/>
+<part name="C53" library="HyTechDevices" deviceset="CAPACITOR_?_*" device="0603" technology="35V_1UF" value="CAPACITOR_0603_35V_1UF"/>
 <part name="U15" library="HyTechDevices" deviceset="MCP3208" device=""/>
 <part name="P93" library="HyTechSupplies" deviceset="+3V3" device=""/>
